File: GPIO.kicad_sch (KiCad schematic)
At the start: 0 parts

Commit message: Updated pinouts and added protection circuitry for signals
Parts:
- added CR1 (x3): D5V0P4UR6SO-7, UTSVT_ICs:SOT26_DIO, symbol utsvt-chips:D5V0P4UR6SO-7
Connections:
- new net GND: CR1.2, CR1.2, CR1.2
- new net GPIO1: CR1.1
- new net GPIO10: CR1.3
- new net GPIO11: CR1.6
- new net GPIO12: CR1.4
- new net GPIO2: CR1.3
- new net GPIO3: CR1.6
- new net GPIO4: CR1.4
- new net GPIO5: CR1.1
- new net GPIO6: CR1.3
- new net GPIO7: CR1.6
- new net GPIO8: CR1.4
- new net GPIO9: CR1.1
- no-connect marks 0 -> 3
