File: UART.kicad_sch (KiCad schematic)
At the start: 0 parts

Commit message: Updated UART
Parts:
- added CR1: D5V0P4UR6SO-7, UTSVT_ICs:SOT26_DIO, symbol utsvt-chips:D5V0P4UR6SO-7
- added J5: UART1, Connector_PinHeader_2.54mm:PinHeader_1x04_P2.54mm_Vertical, symbol Connector_Generic:Conn_01x04
- added J6: UART2, Connector_PinHeader_2.54mm:PinHeader_1x04_P2.54mm_Vertical, symbol Connector_Generic:Conn_01x04
Connections:
- new net +3.3V: J5.1 (Pin_1), J6.1 (Pin_1)
- new net GND: CR1.2, J5.4 (Pin_4), J6.4 (Pin_4)
- new net UART1_RX: CR1.1, J5.2 (Pin_2)
- new net UART1_TX: CR1.3, J5.3 (Pin_3)
- new net UART2_RX: CR1.6, J6.2 (Pin_2)
- new net UART2_TX: CR1.4, J6.3 (Pin_3)
- no-connect marks 0 -> 1

Commit message: Updated pin assignments
Changed lines of the file:
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@@
     (stroke (width 0) (type default))
   )
-  (label "UART2_RX" (at 187.325 107.95 180) (fields_autoplaced)
-    (effects (font (size 1.27 1.27)) (justify right bottom))
+  (hierarchical_label "UART1_TX" (shape input) (at 187.325 86.36 180) (fields_autoplaced)
+    (effects (font (size 1.27 1.27)) (justify right))
   )
-  (label "UART1_TX" (at 111.76 100.965 180) (fields_autoplaced)
-    (effects (font (size 1.27 1.27)) (justify right bottom))
+  (hierarchical_label "UART1_RX" (shape output) (at 187.325 83.82 180) (fields_autoplaced)
+    (effects (font (size 1.27 1.27)) (justify right))
   )
-  (label "UART2_TX" (at 187.325 110.49 180) (fields_autoplaced)
-    (effects (font (size 1.27 1.27)) (justify right bottom))
+  (hierarchical_label "UART2_RX" (shape output) (at 187.325 107.95 180) (fields_autoplaced)
+    (effects (font (size 1.27 1.27)) (justify right))
   )
-  (label "UART2_TX" (at 152.4 100.965 0) (fields_autoplaced)
-    (effects (font (size 1.27 1.27)) (justify left bottom))
+  (hierarchical_label "UART2_TX" (shape input) (at 152.4 100.965 0) (fields_autoplaced)
+    (effects (font (size 1.27 1.27)) (justify left))
   )
-  (label "UART2_RX" (at 152.4 95.885 0) (fields_autoplaced)
-    (effects (font (size 1.27 1.27)) (justify left bottom))
+  (hierarchical_label "UART2_TX" (shape input) (at 187.325 110.49 180) (fields_autoplaced)
+    (effects (font (size 1.27 1.27)) (justify right))
   )
-  (label "UART1_RX" (at 187.325 83.82 180) (fields_autoplaced)
-    (effects (font (size 1.27 1.27)) (justify right bottom))
+  (hierarchical_label "UART2_RX" (shape output) (at 152.4 95.885 0) (fields_autoplaced)
+    (effects (font (size 1.27 1.27)) (justify left))
   )
-  (label "UART1_RX" (at 111.76 95.885 180) (fields_autoplaced)
-    (effects (font (size 1.27 1.27)) (justify right bottom))
+  (hierarchical_label "UART1_RX" (shape output) (at 111.76 95.885 180) (fields_autoplaced)
+    (effects (font (size 1.27 1.27)) (justify right))
   )
-  (label "UART1_TX" (at 187.325 86.36 180) (fields_autoplaced)
-    (effects (font (size 1.27 1.27)) (justify right bottom))
+  (hierarchical_label "UART1_TX" (shape input) (at 111.76 100.965 180) (fields_autoplaced)
+    (effects (font (size 1.27 1.27)) (justify right))
   )
   (symbol (lib_id "Connector_Generic:Conn_01x04") (at 192.405 107.95 0) (unit 1)

Commit message: Updated pinouts and added protection circuitry for signals
Parts:
- removed J5: UART1, Connector_PinHeader_2.54mm:PinHeader_1x04_P2.54mm_Vertical, symbol Connector_Generic:Conn_01x04
- removed J6: UART2, Connector_PinHeader_2.54mm:PinHeader_1x04_P2.54mm_Vertical, symbol Connector_Generic:Conn_01x04
Other:
- moved on the sheet: CR1
