File: InternalCAN.kicad_sch (KiCad schematic)
At the start: 6 parts, among them J11 CAN_1, U4 ISO1044BD, U5 CDSOT23-T24CAN

Commit message: Updated datasheets
Parts:
- J11: footprint (none) -> UTSVT_Connectors:Molex_MicroFit3.0_1x4xP3.00mm_PolarizingPeg_Vertical
Changed lines of the file:
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@@
       (effects (font (size 1.524 1.524)))
     )
-    (property "Footprint" "" (at 109.855 108.585 0)
+    (property "Footprint" "UTSVT_Connectors:Molex_MicroFit3.0_1x4xP3.00mm_PolarizingPeg_Vertical" (at 109.855 108.585 0)
       (effects (font (size 1.524 1.524)) hide)
     )
-    (property "Datasheet" "" (at 109.855 108.585 0)
+    (property "Datasheet" "https://www.mouser.com/ProductDetail/Molex/43650-0244?qs=XoD1gVtqLQuEe6RJ38AzJQ%3D%3D" (at 109.855 108.585 0)
       (effects (font (size 1.524 1.524)) hide)
     )

Commit message: Updated power dist and CAN circuitry
Parts:
- added PS3: RS6-0505S, RS60505S, symbol utsvt-power-regulators:RS6-0505S
Connections:
- net +5V: now also PS3.2 (+VIN), PS3.3 (CTRL); no longer C10.1, J11.1 (5V), U4.8 (VCC2)
- net GND: now also PS3.1 (-VIN); no longer C10.2, J11.2 (GND), U4.7 (GND2), U5.3 (GND)
- new net +V_CAN1: C10.1, J11.1 (5V), PS3.6 (+VOUT), U4.8 (VCC2)
- new net -V_CAN1: C10.2, J11.2 (GND), PS3.7 (-VOUT), U4.7 (GND2), U5.3 (GND)
- no-connect marks 0 -> 1
Other:
- note removed: "Connect the jumper (JP1) to make this the terminating end"
- note removed: "GND1 != GND GND1 = CAN GND = GND_ISO_In/Out"
- moved on the sheet: J11

Commit message: a
Parts:
- added C12: 22uF, Capacitor_SMD:C_0805_2012Metric, symbol Device:C_Small
- added L1: 1uH, Inductor_SMD:L_0805_2012Metric, symbol Device:L_Small
- J11: value CAN_1 -> CAN_Int
- PS3: footprint RS60505S -> UTSVT_Power:RS60505S
Connections:
- net +5V: now also C12.1, L1.1; no longer PS3.2 (+VIN), PS3.3 (CTRL)
- net GND: now also C12.2
- new net: L1.2, PS3.2 (+VIN)
- no-connect marks 1 -> 2
Other:
- note added: "Power Delivery for Periphery Boards 600mA Max"
- moved on the sheet: C10, C9, J11, PS3, R10, U4, U5

Commit message: updated pin assignments
Changed lines of the file:
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@@
     (effects (font (size 1.27 1.27)) (justify right))
-  )
-  (symbol (lib_id "power:+3.3V") (at 75.565 58.42 0) (unit 1)
-    (in_bom yes) (on_board yes) (dnp no)
-    (property "Reference" "#PWR082" (at 75.565 62.23 0)
-      (effects (font (size 1.27 1.27)) hide)
-    )
-    (property "Value" "+3.3V" (at 75.946 54.0258 0)
-      (effects (font (size 1.27 1.27)))
-    )
-    (property "Footprint" "" (at 75.565 58.42 0)
-      (effects (font (size 1.27 1.27)) hide)
-    )
-    (property "Datasheet" "" (at 75.565 58.42 0)
-      (effects (font (size 1.27 1.27)) hide)
-    )
-    (pin "1")
-    (instances
-      (project "LeaderSOM"
-        (path "/192d0c36-944e-4927-949b-263b8c85a7ca/3c3cb7b2-3464-4424-b8df-3064a68eb04d"
-          (reference "#PWR082") (unit 1)
-        )
-      )
-      (project "Dashboard"
-        (path "/66218487-e316-4467-9eba-79d4626ab24e/00000000-0000-0000-0000-00005f547b94"
-          (reference "#PWR0100") (unit 1)
-        )
-      )
-      (project "BPS-PeripheralSOM"
-        (path "/d5ebd247-5a7c-47c2-8aee-beabaef72d6d/1d0c269d-60cf-499b-bfd2-5087981d6678"
-          (reference "#PWR036") (unit 1)
-        )
-      )
-    )
   )
   (symbol (lib_id "power:GND") (at 86.995 139.7 0) (unit 1)
@@
         )
       )
+    )
+  )
+  (symbol (lib_id "power:+3.3V") (at 75.565 58.42 0) (unit 1)
+    (in_bom yes) (on_board yes) (dnp no) (fields_autoplaced)
+    (property "Reference" "#PWR025" (at 75.565 62.23 0)
+      (effects (font (size 1.27 1.27)) hide)
+    )
+    (property "Value" "+3.3V" (at 75.565 54.61 0)
+      (effects (font (size 1.27 1.27)))
+    )
+    (property "Footprint" "" (at 75.565 58.42 0)
+      (effects (font (size 1.27 1.27)) hide)
+    )
+    (property "Datasheet" "" (at 75.565 58.42 0)
+      (effects (font (size 1.27 1.27)) hide)
+    )
+    (pin "1")
+    (instances
+      (project "LeaderSOM"
+        (path "/192d0c36-944e-4927-949b-263b8c85a7ca"
+          (reference "#PWR025") (unit 1)
+        )
+        (path "/192d0c36-944e-4927-949b-263b8c85a7ca/07cef2e6-f2f4-4f04-bcaf-7b98b53ab0fe"
+          (reference "#PWR025") (unit 1)
+        )
+        (path "/192d0c36-944e-4927-949b-263b8c85a7ca/3c3cb7b2-3464-4424-b8df-3064a68eb04d"
+          (reference "#PWR058") (unit 1)
+        )
+      )
+      (project "BPS-PeripheralSOM"
+        (path "/d5ebd247-5a7c-47c2-8aee-beabaef72d6d"
+          (reference "#PWR02") (unit 1)
+        )
+      )

Commit message: 👹
Parts:
- added D2: V_CAN1, LED_SMD:LED_0805_2012Metric, symbol Device:LED
- added F1: 1.8A, Fuse:Fuse_1206_3216Metric, symbol Device:Polyfuse_Small
- added R1: 5.1k, Resistor_SMD:R_0805_2012Metric, symbol Device:R
Connections:
- net +V_CAN1: now also F1.2, R1.1; no longer PS3.6 (+VOUT)
- net -V_CAN1: now also D2.1 (K)
- new net: F1.1, PS3.6 (+VOUT)
- new net: D2.2 (A), R1.2
Other:
- note added: "PTC Hold Current is 1A"
- note added: "Power Delivery for Periphery Boards 1.2A Max"
- note removed: "Power Delivery for Periphery Boards 600mA Max"

Commit message: fix power dist, update to kicad 8
Parts:
- renumbered D2 to D5, R1 to R34

Commit message: Updated schem for redesign
Parts:
- removed C12: 22uF, Capacitor_SMD:C_0805_2012Metric, symbol Device:C_Small
- removed D5: V_CAN1, LED_SMD:LED_0805_2012Metric, symbol Device:LED
- removed F1: 1.8A, Fuse:Fuse_1206_3216Metric, symbol Device:Polyfuse_Small
- removed J11: CAN_Int, UTSVT_Connectors:Molex_MicroFit3.0_1x4xP3.00mm_PolarizingPeg_Vertical, symbol utsvt-connectors:CANConnector
- removed L1: 1uH, Inductor_SMD:L_0805_2012Metric, symbol Device:L_Small
- removed PS3: RS6-0505S, UTSVT_Power:RS60505S, symbol utsvt-power-regulators:RS6-0505S
- removed R34: 5.1k, Resistor_SMD:R_0805_2012Metric, symbol Device:R
Connections:
- net +V_CAN1 is gone; now on net +3.3V: C10.1, U4.8 (VCC2)
- net -V_CAN1 is gone; now on net GND: C10.2, U4.7 (GND2), U5.3 (GND)
- net CAN_H renamed IntCAN_H
- net CAN_L renamed IntCAN_L
- no-connect marks 2 -> 0
Other:
- note added: "Internal CAN Bus unisolated from LeaderSOM Power"
- note added: "Note: +3.3V is not sent with CAN. +12V gets sent with CAN to each PSOM and each PSOM individually bucks down to +3.3V for the bus side"
- note added: "UNISOLATED"
- note removed: "CAN GND (Different from Power GND)"
- note removed: "ISOLATED"
- note removed: "Local (Primary Board) GND"
- note removed: "PTC Hold Current is 1A"
- note removed: "Power Delivery for Periphery Boards 1.2A Max"
- moved on the sheet: C10, C9, R10, U4, U5
