File: InternalCAN.kicad_sch (KiCad schematic)
At the start: 5 parts, among them U4 ISO1044BD, U5 CDSOT23-T24CAN

Commit message: laid things out but still need to fix things :(
Parts:
- removed C10, C9: 100nF, Capacitor_SMD:C_0805_2012Metric, symbol Device:C_Small
- removed U4: ISO1044BD, Package_SO:SSOP-8_3.9x5.05mm_P1.27mm, symbol utsvt-chips:ISO1044BD
- removed U5: CDSOT23-T24CAN, Package_TO_SOT_SMD:SOT-23W, symbol utsvt-chips:CDSOT23-T24CAN
- added D8: LED, LED_SMD:LED_0805_2012Metric, symbol Device:LED
- added IC3: TCAN337DCNR, UTSVT_ICs:SOT65P280X145-8N, symbol utsvt-chips:TCAN337DCNR
- added R22: 2.2k, Resistor_SMD:R_0805_2012Metric, symbol Device:R
- added U4: CDSOT23-T24CAN, Package_TO_SOT_SMD:SOT-23W, symbol utsvt-chips:CDSOT23-T24CAN
Connections:
- net +3.3V: now also IC3.3 (VCC)
- net CAN_RX: now also IC3.4 (RXD)
- net CAN_TX: now also IC3.1 (TXD)
- net GND: now also D8.1 (K), IC3.2 (GND), U4.3 (GND)
- net IntCAN_H: now also R10.1, IC3.7 (CANH), U4.2 (CAN_L); no longer R10.2
- net IntCAN_L: now also R10.2, IC3.6 (CANL), U4.1 (CAN_H); no longer R10.1
- new net: D8.2 (A), R22.2
- new net Fault: IC3.5 (FAULT), R22.1
- no-connect marks 0 -> 1
Other:
- note removed: "Internal CAN Bus unisolated from LeaderSOM Power"
- note removed: "Note: +3.3V is not sent with CAN. +12V gets sent with CAN to each PSOM and each PSOM individually bucks down to +3.3V for the bus side"
- note removed: "UNISOLATED"

Commit message: fixed can stuff
Parts:
- added C11, C18: 100nF, Capacitor_SMD:C_0805_2012Metric, symbol Device:C
- added R11: 10k, Resistor_SMD:R_0805_2012Metric, symbol Device:R
- renumbered D8 to IC_FLT1
Connections:
- net +3.3V: now also C11.1, C18.1, R11.1
- net Fault: now also R11.2
- net GND: now also C11.2, C18.2
Other:
- note added: "Decoupling Caps"
- moved on the sheet: IC3, IC_FLT1, R10, R22, U4

Commit message: MCU pins, PSON power distribution, KiCad-Sharepoint, and 7 seg
Parts:
- C18: value 100nF -> 1u
- IC3: footprint UTSVT_ICs:SOT65P280X145-8N -> UTSVT_ICs:TCAN337DCNR; symbol utsvt-chips:TCAN337DCNR -> UTSVT-ICs:TCAN337; P/N (none) -> TCAN337DCNR
Connections:
- net IntCAN_H: now also R10.2, U4.1 (CAN_H); no longer R10.1, U4.2 (CAN_L)
- net IntCAN_L: now also R10.1, U4.2 (CAN_L); no longer R10.2, U4.1 (CAN_H)
Other:
- note added: "CAN Bus Termination"
- note added: "CAN Transceiver"
- moved on the sheet: C11, C18, IC3, IC_FLT1, R10, R11, R22, U4

Commit message: net class fixes and ERC
Connections:
- net +3.3V renamed +3V3
Changed lines of the file:
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@@
+	)
+	(symbol
+		(lib_id "power:+3.3V")
+		(at 109.22 73.025 0)
+		(unit 1)
+		(exclude_from_sim no)
+		(in_bom yes)
+		(on_board yes)
+		(dnp no)
+		(property "Reference" "#PWR0125"
+			(at 109.22 76.835 0)
+			(effects
+				(font
+					(size 1.27 1.27)
+				)
+				(hide yes)
+			)
+		)
+		(property "Value" "+3V3"
+			(at 109.601 68.6308 0)
+			(effects
+				(font
+					(size 1.27 1.27)
+				)
+			)
+		)
+		(property "Footprint" ""
+			(at 109.22 73.025 0)
+			(effects
+				(font
+					(size 1.27 1.27)
+				)
+				(hide yes)
+			)
+		)
+		(property "Datasheet" ""
+			(at 109.22 73.025 0)
+			(effects
+				(font
+					(size 1.27 1.27)
+				)
+				(hide yes)
+			)
+		)
+		(property "Description" "Power symbol creates a global label with name \"+3.3V\""
+			(at 109.22 73.025 0)
+			(effects
+				(font
+					(size 1.27 1.27)
+				)
+				(hide yes)
+			)
+		)
+		(pin "1"
+		)
+		(instances
+			(project "LeaderSOM"
+				(path "/192d0c36-944e-4927-949b-263b8c85a7ca/3c3cb7b2-3464-4424-b8df-3064a68eb04d"
+					(reference "#PWR0125")
+					(unit 1)
+				)
+			)
+		)
 	)
 	(symbol
@@
 	)
 	(symbol
-		(lib_id "power:+3.3V")
-		(at 81.915 76.2 0)
-		(unit 1)
-		(exclude_from_sim no)
-		(in_bom yes)
-		(on_board yes)
-		(dnp no)
-		(property "Reference" "#PWR043"
-			(at 81.915 80.01 0)
-			(effects
-				(font
-					(size 1.27 1.27)
-				)
-				(hide yes)
-			)
-		)
-		(property "Value" "+3.3V"
-			(at 82.296 71.8058 0)
-			(effects
-				(font
-					(size 1.27 1.27)
-				)
-			)
-		)
-		(property "Footprint" ""
-			(at 81.915 76.2 0)
-			(effects
-				(font
-					(size 1.27 1.27)
-				)
-				(hide yes)
-			)
-		)
-		(property "Datasheet" ""
-			(at 81.915 76.2 0)
-			(effects
-				(font
-					(size 1.27 1.27)
-				)
-				(hide yes)
-			)
-		)
-		(property "Description" "Power symbol creates a global label with name \"+3.3V\""
-			(at 81.915 76.2 0)
-			(effects
-				(font
-					(size 1.27 1.27)
-				)
-				(hide yes)
-			)
-		)
-		(pin "1"
-		)
-		(instances
-			(project "LeaderSOM"
-				(path "/192d0c36-944e-4927-949b-263b8c85a7ca/3c3cb7b2-3464-4424-b8df-3064a68eb04d"
-					(reference "#PWR043")
-					(unit 1)
-				)
-			)
-		)
-	)
-	(symbol
 		(lib_id "power:GND")
 		(at 109.22 93.345 0)
@@
 	(symbol
 		(lib_id "power:+3.3V")
+		(at 81.915 76.2 0)
+		(unit 1)
+		(exclude_from_sim no)
+		(in_bom yes)
+		(on_board yes)
+		(dnp no)
+		(property "Reference" "#PWR0124"
+			(at 81.915 80.01 0)
+			(effects
+				(font
+					(size 1.27 1.27)
+				)
+				(hide yes)
+			)
+		)
+		(property "Value" "+3V3"
+			(at 82.296 71.8058 0)
+			(effects
+				(font
+					(size 1.27 1.27)
+				)
+			)
+		)
+		(property "Footprint" ""
+			(at 81.915 76.2 0)
+			(effects
+				(font
+					(size 1.27 1.27)
+				)
+				(hide yes)
+			)
+		)
+		(property "Datasheet" ""
+			(at 81.915 76.2 0)
+			(effects
+				(font
+					(size 1.27 1.27)
+				)
+				(hide yes)
+			)
+		)
+		(property "Description" "Power symbol creates a global label with name \"+3.3V\""
+			(at 81.915 76.2 0)
+			(effects
+				(font
+					(size 1.27 1.27)
+				)
+				(hide yes)
+			)
+		)
+		(pin "1"
+		)
+		(instances
+			(project "LeaderSOM"
+				(path "/192d0c36-944e-4927-949b-263b8c85a7ca/3c3cb7b2-3464-4424-b8df-3064a68eb04d"
+					(reference "#PWR0124")
+					(unit 1)
+				)
+			)
+		)
+	)
+	(symbol
+		(lib_id "power:+3.3V")
 		(at 189.23 85.09 0)
 		(unit 1)
@@
 		(on_board yes)
 		(dnp no)
-		(property "Reference" "#PWR064"
+		(property "Reference" "#PWR0126"
 			(at 189.23 88.9 0)
 			(effects
@@
 			)
 		)
-		(property "Value" "+3.3V"
+		(property "Value" "+3V3"
 			(at 189.611 80.6958 0)
 			(effects
@@
 			(project "LeaderSOM"
 				(path "/192d0c36-944e-4927-949b-263b8c85a7ca/3c3cb7b2-3464-4424-b8df-3064a68eb04d"
-					(reference "#PWR064")
+					(reference "#PWR0126")
 					(unit 1)
 				)
@@
 					(unit 1)
 				)
-			)
-		)
-	)
-	(symbol
-		(lib_id "power:+3.3V")
-		(at 109.22 73.025 0)
-		(unit 1)
-		(exclude_from_sim no)
-		(in_bom yes)
-		(on_board yes)
-		(dnp no)
-		(property "Reference" "#PWR07"
-			(at 109.22 76.835 0)
-			(effects
-				(font
-					(size 1.27 1.27)
-				)
-				(hide yes)
-			)
-		)
-		(property "Value" "+3.3V"
-			(at 109.601 68.6308 0)
-			(effects
-				(font
-					(size 1.27 1.27)
-				)
-			)
-		)
-		(property "Footprint" ""
-			(at 109.22 73.025 0)
-			(effects
-				(font
-					(size 1.27 1.27)
-				)
-				(hide yes)
-			)
-		)
-		(property "Datasheet" ""
-			(at 109.22 73.025 0)
-			(effects
-				(font
-					(size 1.27 1.27)
-				)
-				(hide yes)
-			)
-		)
-		(property "Description" "Power symbol creates a global label with name \"+3.3V\""
-			(at 109.22 73.025 0)
-			(effects
-				(font
-					(size 1.27 1.27)
-				)
-				(hide yes)
-			)
-		)
-		(pin "1"
-		)
-		(instances
-			(project "LeaderSOM"
-				(path "/192d0c36-944e-4927-949b-263b8c85a7ca/3c3cb7b2-3464-4424-b8df-3064a68eb04d"
-					(reference "#PWR07")
-					(unit 1)
-				)

Commit message: workday for review
Parts:
- U4: footprint Package_TO_SOT_SMD:SOT-23W -> UTSVT_ICs:CDSOT23-T24CAN; symbol utsvt-chips:CDSOT23-T24CAN -> UTSVT-ICs:CDSOT23-T24CAN; P/N (none) -> CDSOT23-T24CAN
Connections:
- net Fault renamed ICAN_Fault
Changed lines of the file:
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@@
 		)
 	)
-	(label "Fault"
+	(label "ICAN_Fault"
 		(at 172.72 76.2 0)
 		(effects
@@
 		)
 	)
-	(label "Fault"
-		(at 88.9 85.725 0)
+	(label "ICAN_Fault"
+		(at 84.455 85.725 0)
 		(effects
 			(font
@@
 			)
 		)
+		(property "Sim.Pins" "1=K 2=A"
+			(at 172.72 92.075 0)
+			(effects
+				(font
+					(size 1.27 1.27)
+				)
+				(hide yes)
+			)
+		)
 		(pin "1"
 		)
@@
 	)
 	(symbol
-		(lib_id "utsvt-chips:CDSOT23-T24CAN")
+		(lib_id "UTSVT-ICs:CDSOT23-T24CAN")
 		(at 151.765 94.615 0)
 		(unit 1)
@@
 			)
 		)
-		(property "Footprint" "Package_TO_SOT_SMD:SOT-23W"
+		(property "Footprint" "UTSVT_ICs:CDSOT23-T24CAN"
 			(at 151.765 103.505 0)
 			(effects
@@
 			(at 151.765 94.615 0)
 			(effects
+				(font
+					(size 1.27 1.27)
+				)
+				(hide yes)
+			)
+		)
+		(property "P/N" "CDSOT23-T24CAN"
+			(at 151.765 94.615 0)
+			(effects

Commit message: review council
Parts:
- added CC_Term2: Jumper_2_Open, Connector_PinHeader_2.54mm:PinHeader_1x02_P2.54mm_Vertical, symbol Jumper:Jumper_2_Open
Connections:
- net IntCAN_L: now also CC_Term2.2 (B); no longer R10.1
- new net: CC_Term2.1 (A), R10.1
Changed lines of the file:
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@@
-		)
-	)
-	(wire
-		(pts
-			(xy 156.21 127) (xy 158.115 127)
-		)
-		(stroke
-			(width 0)
-			(type default)
 		)
 	)
@@
 	(hierarchical_label "IntCAN_L"
 		(shape input)
-		(at 158.115 127 0)
+		(at 166.37 127 0)
 		(effects
 			(font
@@
 					(unit 1)
 				)
+			)
+		)
+	)
+	(symbol
+		(lib_id "Jumper:Jumper_2_Open")
+		(at 161.29 127 0)
+		(unit 1)
+		(exclude_from_sim no)
+		(in_bom yes)
+		(on_board yes)
+		(dnp no)
+		(property "Reference" "CC_Term2"
+			(at 161.163 129.032 0)
+			(effects
+				(font
+					(size 1.27 1.27)
+				)
+			)
+		)
+		(property "Value" "Jumper_2_Open"
+			(at 161.163 131.572 0)
+			(effects
+				(font
+					(size 1.27 1.27)
+				)
+			)
+		)
+		(property "Footprint" "Connector_PinHeader_2.54mm:PinHeader_1x02_P2.54mm_Vertical"
+			(at 161.29 127 0)
+			(effects
+				(font
+					(size 1.27 1.27)
+				)
+				(hide yes)
+			)
+		)
+		(property "Datasheet" "~"
+			(at 161.29 127 0)
+			(effects
+				(font
+					(size 1.27 1.27)
+				)
+				(hide yes)
+			)
+		)
+		(property "Description" "Jumper, 2-pole, open"
+			(at 161.29 127 0)
+			(effects
+				(font
+					(size 1.27 1.27)
+				)
+				(hide yes)
+			)
+		)
+		(property "PN" ""
+			(at 161.29 127 0)
+			(effects
+				(font
+					(size 1.27 1.27)
+				)
+				(hide yes)
+			)
+		)
+		(property "p/n" ""
+			(at 161.29 127 0)
+			(effects
+				(font
+					(size 1.27 1.27)
+				)
+				(hide yes)
+			)
+		)
+		(pin "2"
+		)
+		(pin "1"
+		)
+		(instances
+			(project "LeaderSOM"
+				(path "/192d0c36-944e-4927-949b-263b8c85a7ca/3c3cb7b2-3464-4424-b8df-3064a68eb04d"
+					(reference "CC_Term2")
+					(unit 1)
+				)
