File: CarCAN.kicad_sch (KiCad schematic)
At the start: 10 parts, among them J11 CAN_In2, J12 CAN_Out2, U4 ISO1044BD, U5 CDSOT23-T24CAN

Commit message: -Changed C1 TMK212BBJ106MGHT to C0805C106M3PAC7210 because C0805 is on the standardized components and TMK2 is NRND. -Changed C5 & C6 0805YC106KAT2A to C0805C105K5PACTU because C0805 is on the standardized components. -Changed C17 PN from C0805C104K5RAC7411 to GRM219R6YA475KA73D. C0805 is 0.1u for some reason when the specified value for 17 is 4.7u. -Updated C21 & C22 to C0805C120K5HACTU from standardized parts list when they previously had no PN listed. -Updated J5,J6,J11 to 43650-0428 when no PN was assigned before. Standardized parts list has 43650-0244, which is currently non-stocked on Mouser. 43650-0428 looks like the same shape and series, just now in stock. Variations on Mouser include different finishes (eg tin, gold plating of different thicknesses) so the choice to use 0428 was arbitrary since it was cheapest. -Updated J7 to 43650-0215 when no PN was assigned before. 43650-0215 is from the standardized parts list and is in stock on Mouser. -Updated L1 to IHHP0805ZHER1R0M01 when no PN was assigned before. IHHP0805ZHER1R0M01 indicates supporting a max of 3.5A whereas the schematic specifies that 1.2A must be supported by the component. -Changed R1 to 22.1kOhms from 20kOhms because there are 22.1kOhm resistors in inventory, and the change will hardly impact function. R1 is for a 12V power indicator LED (reference D2), so precise resistance is not critical. CRCW080522K1FKEA was also assigned from the standardized parts list. -Updated R2 to ERA-6VRW1202V. This resistor is used to set the operating status of U1 and should be a precision resistor. -Changed R3 from 100 to 105. The exact value is not too critical since the capacitance multiplier filter shouldn't be too affected by a small change like this. 105 resistors are also in inventory and easier to find instead of 100. Changed PN to CRCW0805105RFKEA from standardized parts list from CRCW08051K00FKEAC which itself is 1k and the completely wrong value. -Changed R4 and R7 from CRCW08054K70FKEA (a 4.7kOhm resis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
Parts:
- C10, C9: Inventory (none) -> Y; Mouser Price/Stock (none) -> https://www.mouser.com/ProductDetail/KEMET/C0805C104M5RACTU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
- D2: Inventory (none) -> Y; Mouser Price/Stock (none) -> https://www.mouser.com/ProductDetail/Kingbright/APTD2012LCG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
- J11, J12: Mouser Part Number (none) -> 538-43650-0428; Mouser Price/Stock (none) -> https://www.mouser.com/ProductDetail/Molex/43650-0428?qs=zh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; P/N (none) -> 43650-0428
- R1: Inventory (none) -> Y; Mouser Part Number Inventory -> 603-RT0805FRE135K1L; Mouser Price/Stock (none) -> https://www.mouser.com/ProductDetail/YAGEO/RT0805FRE135K1L?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; P/N Inventory -> RT0805FRE135K1L
- R10: Inventory (none) -> Y; Mouser Price/Stock (none) -> https://www.mouser.com/ProductDetail/Vishay-Dale/CRCW080559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
- U4: Mouser Part Number (none) -> 595-ISO1044BD; Mouser Price/Stock (none) -> https://www.mouser.com/ProductDetail/Texas-Instruments/ISO1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; P/N (none) -> ISO1044BD
- U5: Mouser Part Number (none) -> 652-CDSOT23-T24CAN; Mouser Price/Stock (none) -> https://www.mouser.com/ProductDetail/Bourns/CDSOT23-T24CAN?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; P/N (none) -> CDSOT23-T24CAN
Changed lines of the file:
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@@
+      (effects (font (size 1.27 1.27)) hide)
+    )
+    (property "Inventory" "Y" (at 156.21 88.9 0)
+      (effects (font (size 1.27 1.27)) hide)
+    )
+    (property "Mouser Price/Stock" "https://www.mouser.com/ProductDetail/KEMET/C0805C104M5RACTU?qs=VOOUd%252Bza08qHu13WgNByHQ%3D%3D" (at 156.21 88.9 0)
       (effects (font (size 1.27 1.27)) hide)
     )
@@
       (effects (font (size 1.27 1.27)) hide)
     )
+    (property "Inventory" "Y" (at 209.55 139.7 0)
+      (effects (font (size 1.27 1.27)) hide)
+    )
+    (property "Mouser Price/Stock" "https://www.mouser.com/ProductDetail/Kingbright/APTD2012LCGCK?qs=AQlKX63v8RvNHN%2F9EGvNTg%3D%3D" (at 209.55 139.7 0)
+      (effects (font (size 1.27 1.27)) hide)
+    )
     (pin "1")
     (pin "2")
@@
     )
     (property "Datasheet" "https://www.mouser.com/ProductDetail/Texas-Instruments/ISO1044BDR?qs=DuoOggApuK9UGD9QQWYeTA%3D%3D" (at 119.38 93.98 0)
+      (effects (font (size 1.27 1.27)) hide)
+    )
+    (property "Inventory" "" (at 119.38 92.71 0)
+      (effects (font (size 1.27 1.27)) hide)
+    )
+    (property "Mouser Part Number" "595-ISO1044BD" (at 119.38 92.71 0)
+      (effects (font (size 1.27 1.27)) hide)
+    )
+    (property "Mouser Price/Stock" "https://www.mouser.com/ProductDetail/Texas-Instruments/ISO1044BD?qs=W%2FMpXkg%252BdQ6CUu0TGf8UTA%3D%3D" (at 119.38 92.71 0)
+      (effects (font (size 1.27 1.27)) hide)
+    )
+    (property "P/N" "ISO1044BD" (at 119.38 92.71 0)
       (effects (font (size 1.27 1.27)) hide)
     )
@@
       (effects (font (size 1.524 1.524)) hide)
     )
+    (property "Inventory" "" (at 118.11 137.16 0)
+      (effects (font (size 1.27 1.27)) hide)
+    )
+    (property "Mouser Part Number" "538-43650-0428" (at 118.11 137.16 0)
+      (effects (font (size 1.27 1.27)) hide)
+    )
+    (property "Mouser Price/Stock" "https://www.mouser.com/ProductDetail/Molex/43650-0428?qs=zhePCb1yaFNxbtO8xFE5bw%3D%3D" (at 118.11 137.16 0)
+      (effects (font (size 1.27 1.27)) hide)
+    )
+    (property "P/N" "43650-0428" (at 118.11 137.16 0)
+      (effects (font (size 1.27 1.27)) hide)
+    )
     (pin "1")
     (pin "2")
@@
     )
     (property "P/N" "CRCW080559R0FKEA" (at 141.605 102.87 0)
+      (effects (font (size 1.27 1.27)) hide)
+    )
+    (property "Inventory" "Y" (at 141.605 102.87 0)
+      (effects (font (size 1.27 1.27)) hide)
+    )
+    (property "Mouser Price/Stock" "https://www.mouser.com/ProductDetail/Vishay-Dale/CRCW080559R0FKEA?qs=8UjxRNpjuUJYxxQ6CUGOZA%3D%3D" (at 141.605 102.87 0)
       (effects (font (size 1.27 1.27)) hide)
     )
@@
       (effects (font (size 1.27 1.27)) hide)
     )
+    (property "Inventory" "Y" (at 90.805 93.98 0)
+      (effects (font (size 1.27 1.27)) hide)
+    )
+    (property "Mouser Price/Stock" "https://www.mouser.com/ProductDetail/KEMET/C0805C104M5RACTU?qs=VOOUd%252Bza08qHu13WgNByHQ%3D%3D" (at 90.805 93.98 0)
+      (effects (font (size 1.27 1.27)) hide)
+    )
     (pin "1")
     (pin "2")
@@
       (effects (font (size 1.27 1.27)) hide)
     )
-    (property "P/N" "Inventory" (at 209.55 130.81 0)
-      (effects (font (size 1.27 1.27)) hide)
-    )
-    (property "Mouser Part Number" "Inventory" (at 209.55 130.81 0)
+    (property "P/N" "RT0805FRE135K1L" (at 209.55 130.81 0)
+      (effects (font (size 1.27 1.27)) hide)
+    )
+    (property "Mouser Part Number" "603-RT0805FRE135K1L" (at 209.55 130.81 0)
+      (effects (font (size 1.27 1.27)) hide)
+    )
+    (property "Inventory" "Y" (at 209.55 130.81 0)
+      (effects (font (size 1.27 1.27)) hide)
+    )
+    (property "Mouser Price/Stock" "https://www.mouser.com/ProductDetail/YAGEO/RT0805FRE135K1L?qs=sGAEpiMZZMtlubZbdhIBIMaxnMKvEBNd0yD7ShRalSo%3D" (at 209.55 130.81 0)
       (effects (font (size 1.27 1.27)) hide)
     )
@@
       (effects (font (size 1.524 1.524)) hide)
     )
+    (property "Inventory" "" (at 155.575 137.16 0)
+      (effects (font (size 1.27 1.27)) hide)
+    )
+    (property "Mouser Part Number" "538-43650-0428" (at 155.575 137.16 0)
+      (effects (font (size 1.27 1.27)) hide)
+    )
+    (property "Mouser Price/Stock" "https://www.mouser.com/ProductDetail/Molex/43650-0428?qs=zhePCb1yaFNxbtO8xFE5bw%3D%3D" (at 155.575 137.16 0)
+      (effects (font (size 1.27 1.27)) hide)
+    )
+    (property "P/N" "43650-0428" (at 155.575 137.16 0)
+      (effects (font (size 1.27 1.27)) hide)
+    )
     (pin "1")
     (pin "2")
@@
     )
     (property "Datasheet" "~" (at 136.525 110.49 0)
+      (effects (font (size 1.27 1.27)) hide)
+    )
+    (property "Inventory" "" (at 136.525 110.49 0)
       (effects (font (size 1.27 1.27)) hide)
     )
@@
       (effects (font (size 1.524 1.524)) hide)
     )
-    (pin "1")
+    (property "Inventory" "" (at 160.655 108.585 0)
+      (effects (font (size 1.27 1.27)) hide)
+    )
+    (property "Mouser Part Number" "652-CDSOT23-T24CAN" (at 160.655 108.585 0)
+      (effects (font (size 1.27 1.27)) hide)
+    )
+    (property "Mouser Price/Stock" "https://www.mouser.com/ProductDetail/Bourns/CDSOT23-T24CAN?qs=Z7P4xsdcg2LuAOb%2FzQ7xoQ%3D%3D" (at 160.655 108.585 0)
+      (effects (font (size 1.27 1.27)) hide)
+    )
+    (property "P/N" "CDSOT23-T24CAN" (at 160.655 108.585 0)
+      (effects (font (size 1.27 1.27)) hide)
+    )
+    (pin "1")
