File: Power_Distribution.kicad_sch (KiCad schematic)
At the start: 24 parts, among them IC1 TLV74033PDBVR, J7 CarPowerConnector, Q1 PBSS4330X,135, Q3 SI7149ADP-T1-GE3, U2 RI3-1205S

Commit message: Updated power dist and CAN circuitry
Parts:
- removed IC1: TLV74033PDBVR, SOT95P280X145-5N, symbol UTSVT_LeaderSOM:TLV74033PDBVR
- removed U2: RI3-1205S, UTSVT_ICs:RI3_DC_Converter, symbol utsvt-power-regulators:RI3-1205S
- added IC3: LP5912-3.3DRVR, SON65P200X200X80-7N, symbol UTSVT_LeaderSOM:LP5912-3.3DRVR
- added PS2: MYLSM00502ERPL, MYLSM00502ERPL, symbol utsvt-power-regulators:MYLSM00502ERPL
- added R11: 10k, Resistor_SMD:R_0805_2012Metric, symbol Device:R
- added R35: 1k, Resistor_SMD:R_0805_2012Metric, symbol Device:R
- added R36: 47, Resistor_SMD:R_0805_2012Metric, symbol Device:R
- C2: value 100uF -> 47u
- C5, C6: value 10uF -> 1uF
Connections:
- net GNDPWR is gone; now on net GND: C1.2, D2.1 (K), D3.1 (A1), J7.2 (GND), R2.2, TP2.1
- net +12V: now also C1.1, Q3.2 (S), TP1.1, PS2.4 (VIN), PS2.5 (EN); no longer FB3.1, J7.1 (+12V)
- net +3.3V: now also IC3.1 (OUT), R11.1
- net +5V: now also PS2.7 (VO)
- net GND: now also IC3.5 (GND), IC3.7 (EP), PS2.2 (GND_1), PS2.3 (GND_2), PS2.6 (GND_3), PS2.8 (GND_4), PS2.9 (G-PAD), R36.2
- net at C6.1, Q1.1 (E): now also IC3.4 (EN), IC3.6 (IN)
- new net: IC3.3 (PG), R11.2
- new net: PS2.1 (VAR), R35.1
- new net: R35.2, R36.1
- new net 12V_In: FB3.1, J7.1 (+12V)
Other:
- note added: "+12V (unisolated) to +5V (unisolated)"
- note removed: "+5V (unisolated) to +5V (isolated)"
- note removed: "ISOLATED"
- note removed: "Local GND (Internal)"
- note removed: "Power GND (External)"
- moved on the sheet: C2, C5, C6, TP1, TP4

Commit message: a
Parts:
- removed D4: PowerLED, LED_SMD:LED_0805_2012Metric, symbol Device:LED
- removed FB3: FerriteBead, Inductor_SMD:L_0805_2012Metric, symbol Device:FerriteBead
- removed Q3: SI7149ADP-T1-GE3, Package_TO_SOT_SMD:SOT-23, symbol Transistor_FET:AO3401A
- removed R11: 10k, Resistor_SMD:R_0805_2012Metric, symbol Device:R
- removed R4: 1.5k, Resistor_SMD:R_0805_2012Metric, symbol Device:R
- removed TP1: +12V_TP, TestPoint:TestPoint_Keystone_5005-5009_Compact, symbol Connector:TestPoint
- removed TP2: GNDPWR_TP, TestPoint:TestPoint_Keystone_5005-5009_Compact, symbol Connector:TestPoint
- added Q2: SI7149ADP-T1-GE3, POWERPAKSO-8, symbol utsvt-chips:SI7149ADP-T1-GE3
- C1: footprint UTSVT_Passive:C_2220_5750Metric -> Capacitor_SMD:C_0805_2012Metric; Mouser Part Number 581-22201C106KAT2A -> 963-TMK212BBJ106MGHT; P/N 22201C106KAT2A -> TMK212BBJ106MGHT
- C2: footprint UTSVT_Passive:C_2220_5750Metric -> Capacitor_SMD:C_0805_2012Metric; Mouser Part Number 581-22201C106KAT2A -> 81-GRM21B80J476ME01K; P/N 22201C106KAT2A -> GRM21BC80J476ME01K
- C4: footprint Capacitor_SMD:C_0805_2012Metric -> Capacitor_SMD:C_1206_3216Metric; Mouser Part Number (none) -> 187-CL31A107MPKNNWE; P/N (none) -> CL31A107MPKNNWE
- PS2: footprint MYLSM00502ERPL -> UTSVT_Power:MYLSM00502ERPL
- Q1: footprint Package_TO_SOT_THT:TO-39-3 -> Package_TO_SOT_SMD:SOT-89-3
Connections:
- net +12V: now also Q2.1 (S_1), Q2.2 (S_2), Q2.3 (S_3)
- net 12V_In: now also D3.2 (A2), Q2.5 (D_1), Q2.6 (D_2), Q2.7 (D_3), Q2.8 (D_4)
- net at R2.1: now also Q2.4 (G)
- no-connect marks 0 -> 1
Other:
- note added: "UNISOLATED DC-DC Converter for +12V power to +5V"
- note removed: "D"
- note removed: "G"
- note removed: "Isolated DC-DC Converter for +12V power to an isolated +5V. The input gnd (Power GND) is different from the output gnd (Local GND)"
- note removed: "Need to review ferrite bead"
- note removed: "S"
- moved on the sheet: C1, C2, C4, C5, C6, D2, D3, D5, IC3, J7, PS2, Q1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

Commit message: updated pin assignments
Parts:
- removed IC3: LP5912-3.3DRVR, SON65P200X200X80-7N, symbol UTSVT_LeaderSOM:LP5912-3.3DRVR
- added C25: 100nF, Capacitor_SMD:C_0805_2012Metric, symbol Device:C
- added FB2: FerriteBead, Inductor_SMD:L_0805_2012Metric, symbol Device:FerriteBead
- added IC1: LP5912-3.3DRVR, SON65P200X200X80-7N, symbol utsvt-power-regulators:LP5912-3.3DRVR
- Q1: footprint Package_TO_SOT_SMD:SOT-89-3 -> Package_TO_SOT_THT:TO-39-3
Connections:
- net +3.3V: now also FB2.1, IC1.1 (OUT)
- net GND: now also C25.2, IC1.5 (GND), IC1.7 (EP)
- net at C6.1, Q1.1 (E): now also IC1.4 (EN), IC1.6 (IN)
- new net +3.3VA: C25.1, FB2.2
Other:
- note added: "VDDA Separation"
- moved on the sheet: C1, C2, C4, C5, C6, D2, D3, D5, J7, PS2, Q1, Q2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

Commit message: 👹
Parts:
- removed D5: PowerLED, LED_SMD:LED_0805_2012Metric, symbol Device:LED
- added D4: 3V3, LED_SMD:LED_0805_2012Metric, symbol Device:LED
- added Q3: SI7149ADP-T1-GE3, UTSVT_ICs:POWERPAKSO-8, symbol utsvt-chips:SI7149ADP-T1-GE3
- added R15: 138k, Resistor_SMD:R_0805_2012Metric, symbol Device:R
- added U1: MAX16914AUB/V+T, UTSVT_ICs:21-0061L_MXM, symbol utsvt-chips:MAX16914AUB_V+T
- D2: value PowerLED -> 12V
- IC1: footprint SON65P200X200X80-7N -> UTSVT_Power:SON65P200X200X80-7N
- Q1: footprint Package_TO_SOT_THT:TO-39-3 -> Package_TO_SOT_SMD:SOT-89-3
- Q2: footprint POWERPAKSO-8 -> UTSVT_ICs:POWERPAKSO-8
- R1: value 5.1k -> 20k; Mouser Part Number 71-CRCW0805-21.5K-E3 -> Inventory; P/N CRCW080521K5FKEA -> Inventory
- R2: value 1k -> 12k; Mouser Part Number 71-CRCW08051K00FKEAC -> (none); P/N CRCW08051K00FKEAC -> (none)
- R9: value 1k -> 2.2k; Mouser Part Number 71-CRCW0805-21.5K-E3 -> Inventory; P/N CRCW080521K5FKEA -> Inventory
Connections:
- net +12V: now also Q3.5 (D_1), Q3.6 (D_2), Q3.7 (D_3), Q3.8 (D_4), U1.9 (SENSEOUT); no longer Q2.1 (S_1), Q2.2 (S_2), Q2.3 (S_3)
- net 12V_In: now also U1.3 (SENSEIN)
- net GND: now also D4.1 (K), R15.2, U1.6 (GND); no longer R2.2
- net at Q2.4 (G): now also U1.2 (GATE1); no longer R2.1
- net at R9.2: now also D4.2 (A)
- new net: Q2.1 (S_1), Q2.2 (S_2), Q2.3 (S_3), Q3.1 (S_1), Q3.2 (S_2), Q3.3 (S_3), U1.1 (VCC), U1.4 (*SHDN)
- new net: Q3.4 (G), U1.10 (GATE2)
- new net: R15.1, R2.2, U1.7 (SET)
- new net: R2.1, U1.8 (TERM)
- no-connect marks 1 -> 2
Other:
- note added: "Capacitance Multiplier Circuit for DC/DC output ripple"
- note added: "DC/DC is rated for max Vin = 17V. Overvoltage limit set to 15V."
- moved on the sheet: C1, C2, C25, C4, C5, C6, FB2, IC1, PS2, Q1, R3, R35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

Commit message: ahahaha ahehehe ahohohoho
Parts:
- added C25: 100nF, Capacitor_SMD:C_0805_2012Metric, symbol Device:C
- Q1: symbol Transistor_BJT:2N2219 -> Transistor_BJT:2SC1815
Connections:
- net +5V: now also Q1.2 (C); no longer Q1.3 (C)
- net GND: now also C25.2
- net at Q2.1 (S_1), Q2.2 (S_2), Q2.3 (S_3)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: now also C25.1
- net at C4.1, R3.2: now also Q1.3 (B); no longer Q1.2 (B)
Changed lines of the file:
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@@
   (junction (at 189.865 70.485) (diameter 0) (color 0 0 0 0)
+  )
+  (junction (at 174.625 44.45) (diameter 0) (color 0 0 0 0)
   )
   (junction (at 139.7 44.45) (diameter 0) (color 0 0 0 0)
@@
     (stroke (width 0) (type default))
   )
+  (wire (pts (xy 174.625 55.245) (xy 174.625 54.61))
+    (stroke (width 0) (type default))
+  )
   (wire (pts (xy 256.54 125.095) (xy 255.27 125.095))
     (stroke (width 0) (type default))
@@
     (stroke (width 0) (type default))
   )
-  (wire (pts (xy 139.7 44.45) (xy 179.705 44.45))
+  (wire (pts (xy 139.7 44.45) (xy 174.625 44.45))
     (stroke (width 0) (type default))
   )
@@
   )
   (wire (pts (xy 169.545 136.525) (xy 188.595 136.525))
+    (stroke (width 0) (type default))
+  )
+  (wire (pts (xy 174.625 46.99) (xy 174.625 44.45))
     (stroke (width 0) (type default))
   )
@@
   )
   (wire (pts (xy 106.045 142.875) (xy 106.045 149.225))
+    (stroke (width 0) (type default))
+  )
+  (wire (pts (xy 174.625 44.45) (xy 179.705 44.45))
     (stroke (width 0) (type default))
   )
@@
         (path "/192d0c36-944e-4927-949b-263b8c85a7ca/07cef2e6-f2f4-4f04-bcaf-7b98b53ab0fe"
           (reference "J7") (unit 1)
+        )
+      )
+    )
+  )
+  (symbol (lib_id "power:GND") (at 174.625 55.245 0) (unit 1)
+    (in_bom yes) (on_board yes) (dnp no)
+    (property "Reference" "#PWR075" (at 174.625 61.595 0)
+      (effects (font (size 1.27 1.27)) hide)
+    )
+    (property "Value" "GND" (at 174.752 59.6392 0)
+      (effects (font (size 1.27 1.27)))
+    )
+    (property "Footprint" "" (at 174.625 55.245 0)
+      (effects (font (size 1.27 1.27)) hide)
+    )
+    (property "Datasheet" "" (at 174.625 55.245 0)
+      (effects (font (size 1.27 1.27)) hide)
+    )
+    (pin "1")
+    (instances
+      (project "LeaderSOM"
+        (path "/192d0c36-944e-4927-949b-263b8c85a7ca/07cef2e6-f2f4-4f04-bcaf-7b98b53ab0fe"
+          (reference "#PWR075") (unit 1)
+        )
+      )
+      (project "Telemetry-Primary"
+        (path "/7f2a449b-14af-42b3-8d38-5f0f8a5ee7ce/00000000-0000-0000-0000-00005f6cdfd6"
+          (reference "#PWR0127") (unit 1)
+        )
+      )
+      (project "BPS-PeripheralSOM"
+        (path "/d5ebd247-5a7c-47c2-8aee-beabaef72d6d/60a4ab70-544e-48ed-aa76-f39bfcac39df"
+          (reference "#PWR026") (unit 1)
         )
       )
@@
     )
   )
-  (symbol (lib_id "Transistor_BJT:2N2219") (at 154.94 116.205 90) (unit 1)
+  (symbol (lib_id "Transistor_BJT:2SC1815") (at 154.94 116.205 90) (unit 1)
     (in_bom yes) (on_board yes) (dnp no) (fields_autoplaced)
     (property "Reference" "Q1" (at 154.94 108.585 90)
@@
       (effects (font (size 1.27 1.27) italic) (justify left) hide)
     )
-    (property "Datasheet" "http://www.onsemi.com/pub_link/Collateral/2N2219-D.PDF" (at 154.94 116.205 0)
+    (property "Datasheet" "https://media.digikey.com/pdf/Data%20Sheets/Toshiba%20PDFs/2SC1815.pdf" (at 154.94 116.205 0)
       (effects (font (size 1.27 1.27)) (justify left) hide)
     )
@@
         )
       )
+    )
+  )
+  (symbol (lib_id "Device:C") (at 174.625 50.8 0) (unit 1)
+    (in_bom yes) (on_board yes) (dnp no) (fields_autoplaced)
+    (property "Reference" "C25" (at 178.435 50.165 0)
+      (effects (font (size 1.27 1.27)) (justify left))
+    )
+    (property "Value" "100nF" (at 178.435 52.705 0)
+      (effects (font (size 1.27 1.27)) (justify left))
+    )
+    (property "Footprint" "Capacitor_SMD:C_0805_2012Metric" (at 175.5902 54.61 0)
+      (effects (font (size 1.27 1.27)) hide)
+    )
+    (property "Datasheet" "~" (at 174.625 50.8 0)
+      (effects (font (size 1.27 1.27)) hide)
+    )
+    (property "Mouser Part Number" "80-C0805C104M5R" (at 174.625 50.8 0)
+      (effects (font (size 1.27 1.27)) hide)
+    )
+    (property "P/N" "C0805C104M5RACTU" (at 174.625 50.8 0)
+      (effects (font (size 1.27 1.27)) hide)
+    )
+    (pin "1")
+    (pin "2")
+    (instances
+      (project "LeaderSOM"
+        (path "/192d0c36-944e-4927-949b-263b8c85a7ca"
+          (reference "C25") (unit 1)
+        )
+        (path "/192d0c36-944e-4927-949b-263b8c85a7ca/07cef2e6-f2f4-4f04-bcaf-7b98b53ab0fe"
+          (reference "C16") (unit 1)
+        )
+      )
+      (project "BPS-PeripheralSOM"
+        (path "/d5ebd247-5a7c-47c2-8aee-beabaef72d6d"
+          (reference "C7") (unit 1)
+        )
+      )

Commit message: hi lakshay
Parts:
- added TP1: +12V_TP, UTSVT_Special:TestPoint_HEX_3mmID, symbol Connector:TestPoint
- added TP2: +3V3_TP, UTSVT_Special:TestPoint_HEX_3mmID, symbol Connector:TestPoint
- added TP6: GND_TP, UTSVT_Special:TestPoint_HEX_3mmID, symbol Connector:TestPoint
- TP3, TP4: footprint TestPoint:TestPoint_Keystone_5005-5009_Compact -> UTSVT_Special:TestPoint_HEX_3mmID; Mouser Part Number 534-5005 -> (none); P/N 5005 -> (none)
Connections:
- net +12V: now also TP1.1
- net +3.3V: now also TP2.1
- net GND: now also TP6.1
Other:
- note added: "One per side on PCB Front/Back"
- moved on the sheet: C5, C6, J7, TP3
