File: Power_Distribution.kicad_sch (KiCad schematic)
At the start: 32 parts, among them U4 LT1963AEST-3.3#TRPBF, U5 TPS2115ADRBR, U6 TPS5405DR

Commit message: ahahahahsaofiwqihfwqof
Parts:
- 3.3V1, 5V1: now left out of the parts list

Commit message: bom
Parts:
- C10, C13, C14, C20, C21, C22: Mouser Part Number (none) -> GRM21BR61H106KE43K
- C11, C12, C19: Mouser Part Number (none) -> MLASH168SB7104KTNA01
- C15, C18: Mouser Part Number (none) -> MLASU168SB5105KTNA01
- C16: Mouser Part Number (none) -> MSASH168SB5103KTNA01
- C17: Mouser Part Number (none) -> 06035C332K4T2A
- D3: Mouser Part Number (none) -> MP01EA06
- D4, D5, D6, D7: Mouser Part Number (none) -> XL-1608UBC-06A
- L1: Mouser Part Number (none) -> MSS1246-104MLC
- R14: Mouser Part Number (none) -> CRCW0603332RFKEAHP
- R15: Mouser Part Number (none) -> CRCW060316K0FKEA
- R17: Mouser Part Number (none) -> CRCW060310K0FKEI
- R18, R20: Mouser Part Number (none) -> CRCW06034K30FKTA
- R19: Mouser Part Number (none) -> CRCW0603120RFKEC
- R21: Mouser Part Number (none) -> CRCW0603768RFKEA
- U4: Mouser Part Number (none) -> LT1963AEST-3.3#TRPBF
- U5: Mouser Part Number (none) -> TPS2115ADRBR
- U6: Mouser Part Number (none) -> TPS5405DR

Commit message: revB for assembly stuff
Parts:
- added D19: USB, LED_SMD:LED_0603_1608Metric_Pad1.05x0.95mm_HandSolder, symbol Device:LED
- added D20: BUCK, LED_SMD:LED_0603_1608Metric_Pad1.05x0.95mm_HandSolder, symbol Device:LED
- added R28, R34: 768, Resistor_SMD:R_0603_1608Metric_Pad0.98x0.95mm_HandSolder, symbol Device:R
- D7: value BUCK -> 5V
Connections:
- net +5V_BUCK: now also R34.1
- net GND: now also D19.1 (K), D20.1 (K)
- net VBUS: now also R28.1
- new net: D19.2 (A), R28.2
- new net: D20.2 (A), R34.2

Commit message: the emptiness machine - linkin park
Other:
- sheet Power Protection ports: added none; removed IMON_OUT
Changed lines of the file:
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@@
 	(wire
 		(pts
-			(xy 208.788 103.632) (xy 211.582 103.632)
-		)
-		(stroke
-			(width 0)
-			(type default)
-		)
-	)
-	(wire
-		(pts
 			(xy 116.84 52.07) (xy 127 52.07)
 		)
@@
 		)
 	)
-	(hierarchical_label "IMON_OUT"
-		(shape output)
-		(at 208.788 103.632 180)
-		(effects
-			(font
-				(size 1.27 1.27)
-			)
-			(justify right)
-		)
-	)
 	(hierarchical_label "24V_In"
 		(shape input)
@@
 			(effects
 				(font
-					(size 1.27 1.27)
-				)
-				(justify left)
-			)
-		)
-		(pin "IMON_OUT" output
-			(at 211.582 103.632 180)
-			(effects
-				(font

Commit message: qol changes
Parts:
- added D18: D_Schottky, Diode_SMD:D_SOD-123, symbol Device:D_Schottky
Connections:
- net +3V3: now also D18.1 (K); no longer C14.1, U4.3 (OUT)
- new net: C14.1, D18.2 (A), U4.3 (OUT)
Other:
- moved on the sheet: 3.3V1
Changed lines of the file:
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@@
 	(rectangle
 		(start 14.605 157.48)
-		(end 69.85 188.595)
+		(end 93.345 188.595)
 		(stroke
 			(width 0)
@@
 	)
 	(junction
-		(at 59.69 170.18)
+		(at 148.59 69.85)
 		(diameter 0)
 		(color 0 0 0 0)
 	)
 	(junction
-		(at 148.59 69.85)
+		(at 62.23 46.99)
 		(diameter 0)
 		(color 0 0 0 0)
 	)
 	(junction
-		(at 62.23 46.99)
+		(at 71.12 170.18)
 		(diameter 0)
 		(color 0 0 0 0)
@@
 	)
 	(junction
-		(at 54.61 170.18)
+		(at 59.69 170.18)
+		(diameter 0)
+		(color 0 0 0 0)
+	)
+	(junction
+		(at 67.31 170.18)
 		(diameter 0)
 		(color 0 0 0 0)
@@
 	(wire
 		(pts
-			(xy 220.98 46.99) (xy 220.98 52.07)
+			(xy 67.31 170.18) (xy 71.12 170.18)
 		)
 		(stroke
@@
 	(wire
 		(pts
-			(xy 74.93 52.07) (xy 76.2 52.07)
+			(xy 220.98 46.99) (xy 220.98 52.07)
 		)
 		(stroke
@@
 	(wire
 		(pts
-			(xy 52.07 46.99) (xy 62.23 46.99)
+			(xy 74.93 52.07) (xy 76.2 52.07)
 		)
 		(stroke
@@
 	(wire
 		(pts
-			(xy 50.8 142.24) (xy 50.8 143.51)
+			(xy 52.07 46.99) (xy 62.23 46.99)
 		)
 		(stroke
@@
 	(wire
 		(pts
-			(xy 54.61 170.18) (xy 59.69 170.18)
+			(xy 50.8 142.24) (xy 50.8 143.51)
 		)
 		(stroke
@@
 	(wire
 		(pts
-			(xy 54.61 170.18) (xy 49.53 170.18)
+			(xy 49.53 170.18) (xy 59.69 170.18)
 		)
 		(stroke
@@
 	(symbol
 		(lib_id "power:PWR_FLAG")
-		(at 59.69 170.18 270)
+		(at 71.12 170.18 270)
 		(unit 1)
 		(exclude_from_sim no)
@@
 		(dnp no)
 		(property "Reference" "#FLG02"
-			(at 61.595 170.18 0)
+			(at 73.025 170.18 0)
 			(effects
 				(font
@@
 		)
 		(property "Value" "PWR_FLAG"
-			(at 62.865 170.18 0)
+			(at 74.295 170.18 0)
 			(effects
 				(font
@@
 		)
 		(property "Footprint" ""
-			(at 59.69 170.18 0)
+			(at 71.12 170.18 0)
 			(effects
 				(font
@@
 		)
 		(property "Datasheet" "~"
-			(at 59.69 170.18 0)
+			(at 71.12 170.18 0)
 			(effects
 				(font
@@
 		)
 		(property "Description" "Special symbol for telling ERC where power comes from"
-			(at 59.69 170.18 0)
+			(at 71.12 170.18 0)
 			(effects
 				(font
@@
 	(symbol
 		(lib_id "Connector:TestPoint")
-		(at 54.61 170.18 0)
+		(at 67.31 170.18 0)
 		(unit 1)
 		(exclude_from_sim no)
@@
 		(dnp no)
 		(property "Reference" "3.3V1"
-			(at 56.134 161.036 90)
+			(at 68.834 161.036 90)
 			(effects
 				(font
@@
 		)
 		(property "Value" "TestPoint"
-			(at 53.594 161.036 90)
+			(at 66.294 161.036 90)
 			(effects
 				(font
@@
 		)
 		(property "Footprint" "TestPoint:TestPoint_Pad_1.0x1.0mm"
-			(at 59.69 170.18 0)
+			(at 72.39 170.18 0)
 			(effects
 				(font
@@
 		)
 		(property "Datasheet" "~"
-			(at 59.69 170.18 0)
+			(at 72.39 170.18 0)
 			(effects
 				(font
@@
 		)
 		(property "Description" "test point"
-			(at 54.61 170.18 0)
+			(at 67.31 170.18 0)
 			(effects
 				(font
@@
 		)
 		(property "Color" ""
-			(at 54.61 170.18 0)
+			(at 67.31 170.18 0)
 			(effects
 				(font
@@
 		)
 		(property "If" ""
-			(at 54.61 170.18 0)
+			(at 67.31 170.18 0)
 			(effects
 				(font
@@
 		)
 		(property "Mfg" ""
-			(at 54.61 170.18 0)
+			(at 67.31 170.18 0)
 			(effects
 				(font
@@
 		)
 		(property "Vf" ""
-			(at 54.61 170.18 0)
+			(at 67.31 170.18 0)
 			(effects
 				(font
@@
 	)
 	(symbol
+		(lib_id "Device:D_Schottky")
+		(at 63.5 170.18 180)
+		(unit 1)
+		(exclude_from_sim no)
+		(in_bom yes)
+		(on_board yes)
+		(dnp no)
+		(property "Reference" "D18"
+			(at 60.96 164.465 0)
+			(effects
+				(font
+					(size 1.27 1.27)
+				)
+			)
+		)
+		(property "Value" "D_Schottky"
+			(at 60.96 167.005 0)
+			(effects
+				(font
+					(size 1.27 1.27)
+				)
+			)
+		)
+		(property "Footprint" "Diode_SMD:D_SOD-123"
+			(at 63.5 170.18 0)
+			(effects
+				(font
+					(size 1.27 1.27)
+				)
+				(hide yes)
+			)
+		)
+		(property "Datasheet" "~"
+			(at 63.5 170.18 0)
+			(effects
+				(font
+					(size 1.27 1.27)
+				)
+				(hide yes)
+			)
+		)
+		(property "Description" "Schottky diode"
+			(at 63.5 170.18 0)
+			(effects
+				(font
+					(size 1.27 1.27)
+				)
+				(hide yes)
+			)
+		)
+		(property "P/N" "BAT760-7"
+			(at 63.5 170.18 0)
+			(effects
+				(font
+					(size 1.27 1.27)
+				)
+				(hide yes)
+			)
+		)
+		(property "Sim.Type" ""
+			(at 63.5 170.18 0)
+			(effects
+				(font
+					(size 1.27 1.27)
+				)
+				(hide yes)
+			)
+		)
+		(property "Inventory" ""
+			(at 63.5 170.18 0)
+			(effects
+				(font
+					(size 1.27 1.27)
+				)
+				(hide yes)
+			)
+		)
+		(property "Color" ""
+			(at 63.5 170.18 0)
+			(effects
+				(font
+					(size 1.27 1.27)
+				)
+			)
+		)
+		(property "If" ""
+			(at 63.5 170.18 0)
+			(effects
+				(font
+					(size 1.27 1.27)
+				)
+			)
+		)
+		(property "Mfg" ""
+			(at 63.5 170.18 0)
+			(effects
+				(font
+					(size 1.27 1.27)
+				)
+			)
+		)
+		(property "Vf" ""
+			(at 63.5 170.18 0)
+			(effects
+				(font
+					(size 1.27 1.27)
+				)
+			)
+		)
+		(property "Mouser Part Number" "1N5819HW-7-F"
+			(at 63.5 170.18 0)
+			(effects
+				(font
+					(size 1.27 1.27)
+				)
+				(hide yes)
+			)
+		)
+		(pin "2"
+		)
+		(pin "1"
+		)
+		(instances
+			(project "LeaderSOM"
+				(path "/192d0c36-944e-4927-949b-263b8c85a7ca/07cef2e6-f2f4-4f04-bcaf-7b98b53ab0fe"
+					(reference "D18")
+					(unit 1)
+				)
+			)
+		)
+	)
+	(symbol
 		(lib_id "power:+24V")
 		(at 52.07 45.72 0)
@@
 	(symbol
 		(lib_id "power:+3.3V")
-		(at 59.69 170.18 0)
+		(at 71.12 170.18 0)
 		(unit 1)
 		(exclude_from_sim no)
@@
 		(dnp no)
 		(property "Reference" "#PWR052"
-			(at 59.69 173.99 0)
+			(at 71.12 173.99 0)
 			(effects
 				(font
@@
 		)
 		(property "Value" "+3V3"
-			(at 60.071 165.7858 0)
+			(at 71.501 165.7858 0)
 			(effects
 				(font
@@
 		)
 		(property "Footprint" ""
-			(at 59.69 170.18 0)
+			(at 71.12 170.18 0)
 			(effects
 				(font
@@
 		)
 		(property "Datasheet" ""
-			(at 59.69 170.18 0)
+			(at 71.12 170.18 0)
 			(effects
 				(font
@@
 		)
 		(property "Description" "Power symbol creates a global label with name \"+3.3V\""
-			(at 59.69 170.18 0)
+			(at 71.12 170.18 0)
 			(effects
 				(font
@@
 					(size 1.27 1.27)
 				)
+				(hide yes)
 			)
 		)
@@
 					(size 1.27 1.27)
 				)
+				(hide yes)
 			)
 		)

Commit message: comp spares with fixed ldo diode
Parts:
- R19: value 120 -> 1k
- R21, R28, R34: value 768 -> 1k
Connections:
- net +3V3: now also C14.1, U4.3 (OUT); no longer D18.1 (K)
- net +5V: now also D18.2 (A); no longer U4.1 (IN)
- new net: D18.1 (K), U4.1 (IN)
Other:
- moved on the sheet: C14, D18, U4
