File: SDCard.kicad_sch (KiCad schematic)
At the start: 0 parts

Commit message: Updated UART
Parts:
- added J4: Micro_SD_Card_Det, UTSVT_Connectors:microSD_HC_Hirose_DM3AT-SF-PEJM5, symbol Connector:Micro_SD_Card_Det2
Connections:
- new net +3.3V: J4.4 (VDD)
- new net DET: J4.9 (DET_B)
- new net GND: J4.11 (SHIELD), J4.6 (VSS)
- new net SPI_CLK: J4.5 (CLK)
- new net SPI_CS: J4.2 (DAT3/CD)
- new net SPI_MISO: J4.7 (DAT0)
- new net SPI_MOSI: J4.3 (CMD)
- no-connect marks 0 -> 3
Other:
- note added: "From telemtry primary PCB"
Changed lines of the file:
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@@
 (kicad_sch (version 20230121) (generator eeschema)
   (paper "A4")
+  (junction (at 128.27 88.9) (diameter 0) (color 0 0 0 0)
+  )
+  (junction (at 152.4 110.49) (diameter 0) (color 0 0 0 0)
+  )
+  (junction (at 128.27 93.98) (diameter 0) (color 0 0 0 0)
+  )
+  (no_connect (at 130.81 101.6))
+  (no_connect (at 130.81 81.28))
+  (no_connect (at 130.81 99.06))
+  (wire (pts (xy 130.81 93.98) (xy 128.27 93.98))
+    (stroke (width 0) (type default))
+  )
+  (wire (pts (xy 130.81 88.9) (xy 128.27 88.9))
+    (stroke (width 0) (type default))
+  )
+  (wire (pts (xy 115.57 99.06) (xy 123.19 99.06))
+    (stroke (width 0) (type default))
+  )
+  (wire (pts (xy 176.53 104.14) (xy 173.99 104.14))
+    (stroke (width 0) (type default))
+  )
+  (wire (pts (xy 130.81 91.44) (xy 115.57 91.44))
+    (stroke (width 0) (type default))
+  )
+  (wire (pts (xy 128.27 74.93) (xy 128.27 88.9))
+    (stroke (width 0) (type default))
+  )
+  (wire (pts (xy 130.81 86.36) (xy 115.57 86.36))
+    (stroke (width 0) (type default))
+  )
+  (wire (pts (xy 176.53 110.49) (xy 176.53 104.14))
+    (stroke (width 0) (type default))
+  )
+  (wire (pts (xy 128.27 110.49) (xy 128.27 93.98))
+    (stroke (width 0) (type default))
+  )
+  (wire (pts (xy 152.4 110.49) (xy 128.27 110.49))
+    (stroke (width 0) (type default))
+  )
+  (wire (pts (xy 123.19 99.06) (xy 123.19 104.14))
+    (stroke (width 0) (type default))
+  )
+  (wire (pts (xy 123.19 104.14) (xy 130.81 104.14))
+    (stroke (width 0) (type default))
+  )
+  (wire (pts (xy 130.81 83.82) (xy 115.57 83.82))
+    (stroke (width 0) (type default))
+  )
+  (wire (pts (xy 128.27 93.98) (xy 115.57 93.98))
+    (stroke (width 0) (type default))
+  )
+  (wire (pts (xy 128.27 88.9) (xy 115.57 88.9))
+    (stroke (width 0) (type default))
+  )
+  (wire (pts (xy 115.57 96.52) (xy 130.81 96.52))
+    (stroke (width 0) (type default))
+  )
+  (wire (pts (xy 152.4 110.49) (xy 176.53 110.49))
+    (stroke (width 0) (type default))
+  )
+  (wire (pts (xy 152.4 113.03) (xy 152.4 110.49))
+    (stroke (width 0) (type default))
+  )
+  (text "From telemtry primary PCB" (at 130.175 53.975 0)
+    (effects (font (size 1.27 1.27)) (justify left bottom))
+  )
+  (label "VDD" (at 115.57 88.9 0) (fields_autoplaced)
+    (effects (font (size 1.27 1.27)) (justify left bottom))
+  )
+  (label "MOSI" (at 115.57 86.36 0) (fields_autoplaced)
+    (effects (font (size 1.27 1.27)) (justify left bottom))
+  )
+  (label "CS" (at 115.57 83.82 0) (fields_autoplaced)
+    (effects (font (size 1.27 1.27)) (justify left bottom))
+  )
+  (label "DET" (at 115.57 99.06 0) (fields_autoplaced)
+    (effects (font (size 1.27 1.27)) (justify left bottom))
+  )
+  (label "GND" (at 115.57 93.98 0) (fields_autoplaced)
+    (effects (font (size 1.27 1.27)) (justify left bottom))
+  )
+  (label "MISO" (at 115.57 96.52 0) (fields_autoplaced)
+    (effects (font (size 1.27 1.27)) (justify left bottom))
+  )
+  (label "CLOCK" (at 115.57 91.44 0) (fields_autoplaced)
+    (effects (font (size 1.27 1.27)) (justify left bottom))
+  )
+  (hierarchical_label "SPI_MOSI" (shape input) (at 115.57 86.36 180) (fields_autoplaced)
+    (effects (font (size 1.27 1.27)) (justify right))
+  )
+  (hierarchical_label "SPI_MISO" (shape output) (at 115.57 96.52 180) (fields_autoplaced)
+    (effects (font (size 1.27 1.27)) (justify right))
+  )
+  (hierarchical_label "SPI_CLK" (shape input) (at 115.57 91.44 180) (fields_autoplaced)
+    (effects (font (size 1.27 1.27)) (justify right))
+  )
+  (hierarchical_label "DET" (shape output) (at 115.57 99.06 180) (fields_autoplaced)
+    (effects (font (size 1.27 1.27)) (justify right))
+  )
+  (hierarchical_label "SPI_CS" (shape input) (at 115.57 83.82 180) (fields_autoplaced)
+    (effects (font (size 1.27 1.27)) (justify right))
+  )
+  (symbol (lib_id "power:GND") (at 152.4 113.03 0) (unit 1)
+    (in_bom yes) (on_board yes) (dnp no)
+    (property "Reference" "#PWR019" (at 152.4 119.38 0)
+      (effects (font (size 1.27 1.27)) hide)
+    )
+    (property "Value" "GND" (at 152.527 117.4242 0)
+      (effects (font (size 1.27 1.27)))
+    )
+    (property "Footprint" "" (at 152.4 113.03 0)
+      (effects (font (size 1.27 1.27)) hide)
+    )
+    (property "Datasheet" "" (at 152.4 113.03 0)
+      (effects (font (size 1.27 1.27)) hide)
+    )
+    (pin "1")
+    (instances
+      (project "LeaderSOM"
+        (path "/192d0c36-944e-4927-949b-263b8c85a7ca/54eecd34-7b2b-4895-a003-33708e7ad7e6"
+          (reference "#PWR019") (unit 1)
+        )
+      )
+      (project "Telemetry-Primary"
+        (path "/7f2a449b-14af-42b3-8d38-5f0f8a5ee7ce/00000000-0000-0000-0000-00005f71644d"
+          (reference "#PWR0147") (unit 1)
+        )
+        (path "/7f2a449b-14af-42b3-8d38-5f0f8a5ee7ce"
+          (reference "#PWR?") (unit 1)
+        )
+      )
+    )
+  )
+  (symbol (lib_id "power:+3.3V") (at 128.27 74.93 0) (unit 1)
+    (in_bom yes) (on_board yes) (dnp no)
+    (property "Reference" "#PWR018" (at 128.27 78.74 0)
+      (effects (font (size 1.27 1.27)) hide)
+    )
+    (property "Value" "+3.3V" (at 128.651 70.5358 0)
+      (effects (font (size 1.27 1.27)))
+    )
+    (property "Footprint" "" (at 128.27 74.93 0)
+      (effects (font (size 1.27 1.27)) hide)
+    )
+    (property "Datasheet" "" (at 128.27 74.93 0)
+      (effects (font (size 1.27 1.27)) hide)
+    )
+    (pin "1")
+    (instances
+      (project "LeaderSOM"
+        (path "/192d0c36-944e-4927-949b-263b8c85a7ca/54eecd34-7b2b-4895-a003-33708e7ad7e6"
+          (reference "#PWR018") (unit 1)
+        )
+      )
+      (project "Telemetry-Primary"
+        (path "/7f2a449b-14af-42b3-8d38-5f0f8a5ee7ce/00000000-0000-0000-0000-00005f71644d"
+          (reference "#PWR0148") (unit 1)
+        )
+      )
+    )
+  )
+  (symbol (lib_id "Connector:Micro_SD_Card_Det2") (at 153.67 91.44 0) (unit 1)
+    (in_bom yes) (on_board yes) (dnp no)
+    (property "Reference" "J4" (at 152.4 70.6882 0)
+      (effects (font (size 1.27 1.27)))
+    )
+    (property "Value" "Micro_SD_Card_Det" (at 152.4 72.9996 0)
+      (effects (font (size 1.27 1.27)))
+    )
+    (property "Footprint" "UTSVT_Connectors:microSD_HC_Hirose_DM3AT-SF-PEJM5" (at 205.74 73.66 0)
+      (effects (font (size 1.27 1.27)) hide)
+    )
+    (property "Datasheet" "https://www.mouser.com/datasheet/2/185/DM3AT_SF_PEJM5_CL0609_0031_0_00_2DDrawing_00009471-1614303.pdf" (at 153.67 88.9 0)
+      (effects (font (size 1.27 1.27)) hide)
+    )
+    (property "P/N" "DM3AT-SF-PEJM5" (at 153.67 91.44 0)
+      (effects (font (size 1.27 1.27)) hide)
+    )
+    (pin "1")
+    (pin "10")
+    (pin "11")
+    (pin "2")
+    (pin "3")
+    (pin "4")
+    (pin "5")
+    (pin "6")
+    (pin "7")
+    (pin "8")
+    (pin "9")
+    (instances
+      (project "LeaderSOM"
+        (path "/192d0c36-944e-4927-949b-263b8c85a7ca/54eecd34-7b2b-4895-a003-33708e7ad7e6"
+          (reference "J4") (unit 1)
+        )
+      )
+      (project "Telemetry-Primary"
+        (path "/7f2a449b-14af-42b3-8d38-5f0f8a5ee7ce/00000000-0000-0000-0000-00005f71644d"
+          (reference "J9") (unit 1)
+        )
+      )
+    )
+  )
 )

Commit message: Updated pin assignments
Other:
- note added: "From telemetry primary PCB"
- note removed: "From telemtry primary PCB"
Changed lines of the file:
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@@
     (stroke (width 0) (type default))
   )
-  (text "From telemtry primary PCB" (at 130.175 53.975 0)
+  (text "From telemetry primary PCB" (at 137.795 56.515 0)
     (effects (font (size 1.27 1.27)) (justify left bottom))
   )

Commit message: Updated pinouts and added protection circuitry for signals
Parts:
- added CR1: D5V0P4UR6SO-7, UTSVT_ICs:SOT26_DIO, symbol utsvt-chips:D5V0P4UR6SO-7
- added R12, R13: 50, Resistor_SMD:R_0805_2012Metric, symbol Device:R
Connections:
- net GND: now also CR1.2
- net SPI_CLK: now also CR1.4, R12.1; no longer J4.5 (CLK)
- net SPI_CS: now also CR1.1
- net SPI_MISO: now also CR1.3
- net SPI_MOSI: now also CR1.6, R13.1; no longer J4.3 (CMD)
- new net: J4.5 (CLK), R12.2
- new net: J4.3 (CMD), R13.2
- no-connect marks 3 -> 4
Other:
- moved on the sheet: J4

Commit message: Updated power dist and CAN circuitry
Parts:
- removed R12, R13: 50, Resistor_SMD:R_0805_2012Metric, symbol Device:R
- added R15: 49.9, Resistor_SMD:R_0805_2012Metric, symbol Device:R
Connections:
- net SPI_CLK: now also J4.5 (CLK)
- net SPI_MISO: now also R15.1; no longer J4.7 (DAT0)
- net SPI_MOSI: now also J4.3 (CMD)
- new net: J4.7 (DAT0), R15.2
Changed lines of the file:
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@@
     (stroke (width 0) (type default))
   )
-  (wire (pts (xy 178.435 98.425) (xy 173.355 98.425))
-    (stroke (width 0) (type default))
-  )
-  (wire (pts (xy 165.735 98.425) (xy 163.195 98.425))
+  (wire (pts (xy 163.195 98.425) (xy 178.435 98.425))
     (stroke (width 0) (type default))
   )
@@
   )
   (wire (pts (xy 175.895 81.915) (xy 175.895 95.885))
-    (stroke (width 0) (type default))
-  )
-  (wire (pts (xy 174.625 91.44) (xy 173.355 91.44))
     (stroke (width 0) (type default))
   )
@@
     (stroke (width 0) (type default))
   )
-  (wire (pts (xy 163.195 91.44) (xy 165.735 91.44))
+  (wire (pts (xy 163.195 91.44) (xy 174.625 91.44))
     (stroke (width 0) (type default))
   )
-  (wire (pts (xy 163.195 103.505) (xy 178.435 103.505))
+  (wire (pts (xy 173.99 103.505) (xy 178.435 103.505))
+    (stroke (width 0) (type default))
+  )
+  (wire (pts (xy 163.195 103.505) (xy 166.37 103.505))
     (stroke (width 0) (type default))
   )
@@
     (effects (font (size 1.27 1.27)) (justify right))
   )
-  (symbol (lib_id "Device:R") (at 169.545 98.425 90) (unit 1)
-    (in_bom yes) (on_board yes) (dnp no) (fields_autoplaced)
-    (property "Reference" "R12" (at 169.545 93.98 90)
-      (effects (font (size 1.27 1.27)))
+  (symbol (lib_id "Device:R") (at 170.18 103.505 90) (unit 1)
+    (in_bom yes) (on_board yes) (dnp no)
+    (property "Reference" "R15" (at 172.085 99.06 90)
+      (effects (font (size 1.27 1.27)) (justify left))
     )
-    (property "Value" "50" (at 169.545 96.52 90)
-      (effects (font (size 1.27 1.27)))
+    (property "Value" "49.9" (at 171.323 101.092 90)
+      (effects (font (size 1.27 1.27)) (justify left))
     )
-    (property "Footprint" "Resistor_SMD:R_0805_2012Metric" (at 169.545 100.203 90)
+    (property "Footprint" "Resistor_SMD:R_0805_2012Metric" (at 170.18 105.283 90)
       (effects (font (size 1.27 1.27)) hide)
     )
-    (property "Datasheet" "https://www.vishay.com/docs/20008/dcrcw.pdf" (at 169.545 98.425 0)
+    (property "Datasheet" "https://www.mouser.com/datasheet/2/427/dcrcwe3-1762152.pdf" (at 170.18 103.505 0)
       (effects (font (size 1.27 1.27)) hide)
     )
-    (property "Mouser Part Number" "71-CRCW0805-50" (at 169.545 98.425 0)
-      (effects (font (size 1.27 1.27)) hide)
-    )
-    (property "P/N" "CRCW080550R0FKTA" (at 169.545 98.425 0)
+    (property "P/N" "CRCW08054K70FKEA" (at 170.18 103.505 0)
       (effects (font (size 1.27 1.27)) hide)
     )
@@
     (instances
       (project "LeaderSOM"
+        (path "/192d0c36-944e-4927-949b-263b8c85a7ca"
+          (reference "R15") (unit 1)
+        )
         (path "/192d0c36-944e-4927-949b-263b8c85a7ca/54eecd34-7b2b-4895-a003-33708e7ad7e6"
           (reference "R12") (unit 1)
         )
       )
-      (project "BPS-PeripheralSOM"
-        (path "/d5ebd247-5a7c-47c2-8aee-beabaef72d6d"
-          (reference "R15") (unit 1)
+      (project "Telemetry-Primary"
+        (path "/7f2a449b-14af-42b3-8d38-5f0f8a5ee7ce/00000000-0000-0000-0000-00005f6cdfd6"
+          (reference "R?") (unit 1)
         )
-      )
-    )
-  )
-  (symbol (lib_id "Device:R") (at 169.545 91.44 90) (unit 1)
-    (in_bom yes) (on_board yes) (dnp no) (fields_autoplaced)
-    (property "Reference" "R13" (at 169.545 86.995 90)
-      (effects (font (size 1.27 1.27)))
-    )
-    (property "Value" "50" (at 169.545 89.535 90)
-      (effects (font (size 1.27 1.27)))
-    )
-    (property "Footprint" "Resistor_SMD:R_0805_2012Metric" (at 169.545 93.218 90)
-      (effects (font (size 1.27 1.27)) hide)
-    )
-    (property "Datasheet" "https://www.vishay.com/docs/20008/dcrcw.pdf" (at 169.545 91.44 0)
-      (effects (font (size 1.27 1.27)) hide)
-    )
-    (property "Mouser Part Number" "71-CRCW0805-50" (at 169.545 91.44 0)
-      (effects (font (size 1.27 1.27)) hide)
-    )
-    (property "P/N" "CRCW080550R0FKTA" (at 169.545 91.44 0)
-      (effects (font (size 1.27 1.27)) hide)
-    )
-    (pin "1")
-    (pin "2")
-    (instances
-      (project "LeaderSOM"
-        (path "/192d0c36-944e-4927-949b-263b8c85a7ca/54eecd34-7b2b-4895-a003-33708e7ad7e6"
-          (reference "R13") (unit 1)
-        )
-      )
-      (project "BPS-PeripheralSOM"
-        (path "/d5ebd247-5a7c-47c2-8aee-beabaef72d6d"
-          (reference "R15") (unit 1)
+        (path "/7f2a449b-14af-42b3-8d38-5f0f8a5ee7ce"
+          (reference "R2") (unit 1)
         )
       )
@@
           (reference "CR1") (unit 1)
         )
-        (path "/192d0c36-944e-4927-949b-263b8c85a7ca/fa2783bd-2a74-4366-90d0-efc036e3ce36"
-          (reference "CR1") (unit 1)
-        )

Commit message: a
Connections:
- net +3.3V: now also CR1.5
- no-connect marks 4 -> 3
Changed lines of the file:
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@@
   (no_connect (at 178.435 108.585))
   (no_connect (at 178.435 88.265))
-  (no_connect (at 131.445 96.52))
   (no_connect (at 178.435 106.045))
   (wire (pts (xy 163.195 111.125) (xy 178.435 111.125))
@@
     (stroke (width 0) (type default))
   )
+  (wire (pts (xy 143.51 87.63) (xy 143.51 96.52))
+    (stroke (width 0) (type default))
+  )
   (wire (pts (xy 163.195 98.425) (xy 178.435 98.425))
     (stroke (width 0) (type default))
@@
     (stroke (width 0) (type default))
   )
-  (wire (pts (xy 76.835 96.52) (xy 90.805 96.52))
-    (stroke (width 0) (type default))
-  )
   (wire (pts (xy 175.895 81.915) (xy 175.895 95.885))
     (stroke (width 0) (type default))
   )
+  (wire (pts (xy 77.47 96.52) (xy 90.805 96.52))
+    (stroke (width 0) (type default))
+  )
   (wire (pts (xy 224.155 117.475) (xy 224.155 111.125))
     (stroke (width 0) (type default))
@@
     (stroke (width 0) (type default))
   )
+  (wire (pts (xy 77.47 102.87) (xy 77.47 96.52))
+    (stroke (width 0) (type default))
+  )
   (wire (pts (xy 175.895 117.475) (xy 175.895 100.965))
     (stroke (width 0) (type default))
@@
   )
   (wire (pts (xy 173.99 103.505) (xy 178.435 103.505))
+    (stroke (width 0) (type default))
+  )
+  (wire (pts (xy 131.445 96.52) (xy 143.51 96.52))
     (stroke (width 0) (type default))
   )
@@
       (effects (font (size 1.27 1.27)) hide)
     )
-    (property "Datasheet" "https://www.mouser.com/datasheet/2/427/dcrcwe3-1762152.pdf" (at 170.18 103.505 0)
+    (property "Datasheet" "~" (at 170.18 103.505 0)
       (effects (font (size 1.27 1.27)) hide)
     )
@@
     )
   )
-  (symbol (lib_id "power:GND") (at 76.835 96.52 0) (unit 1)
-    (in_bom yes) (on_board yes) (dnp no)
-    (property "Reference" "#PWR016" (at 76.835 102.87 0)
-      (effects (font (size 1.27 1.27)) hide)
-    )
-    (property "Value" "GND" (at 76.962 100.9142 0)
-      (effects (font (size 1.27 1.27)))
-    )
-    (property "Footprint" "" (at 76.835 96.52 0)
-      (effects (font (size 1.27 1.27)) hide)
-    )
-    (property "Datasheet" "" (at 76.835 96.52 0)
+  (symbol (lib_id "power:GND") (at 77.47 102.87 0) (unit 1)
+    (in_bom yes) (on_board yes) (dnp no)
+    (property "Reference" "#PWR016" (at 77.47 109.22 0)
+      (effects (font (size 1.27 1.27)) hide)
+    )
+    (property "Value" "GND" (at 77.597 107.2642 0)
+      (effects (font (size 1.27 1.27)))
+    )
+    (property "Footprint" "" (at 77.47 102.87 0)
+      (effects (font (size 1.27 1.27)) hide)
+    )
+    (property "Datasheet" "" (at 77.47 102.87 0)
       (effects (font (size 1.27 1.27)) hide)
     )
@@
       (effects (font (size 1.27 1.27)) hide)
     )
-    (property "Datasheet" "https://www.mouser.com/datasheet/2/185/DM3AT_SF_PEJM5_CL0609_0031_0_00_2DDrawing_00009471-1614303.pdf" (at 201.295 95.885 0)
+    (property "Datasheet" "https://www.hirose.com/en/product/document?clcode=&productname=&series=DM3&documenttype=Catalog&lang=en&documentid=D49662_en" (at 201.295 95.885 0)
       (effects (font (size 1.27 1.27)) hide)
     )
@@
         )
       )
+    )
+  )
+  (symbol (lib_id "power:+3.3V") (at 143.51 87.63 0) (unit 1)
+    (in_bom yes) (on_board yes) (dnp no)
+    (property "Reference" "#PWR028" (at 143.51 91.44 0)
+      (effects (font (size 1.27 1.27)) hide)
+    )
+    (property "Value" "+3.3V" (at 143.891 83.2358 0)
+      (effects (font (size 1.27 1.27)))
+    )
+    (property "Footprint" "" (at 143.51 87.63 0)
+      (effects (font (size 1.27 1.27)) hide)
+    )
+    (property "Datasheet" "" (at 143.51 87.63 0)
+      (effects (font (size 1.27 1.27)) hide)
+    )
+    (pin "1")
+    (instances
+      (project "LeaderSOM"
+        (path "/192d0c36-944e-4927-949b-263b8c85a7ca/54eecd34-7b2b-4895-a003-33708e7ad7e6"
+          (reference "#PWR028") (unit 1)
+        )
+      )
+      (project "Telemetry-Primary"
+        (path "/7f2a449b-14af-42b3-8d38-5f0f8a5ee7ce/00000000-0000-0000-0000-00005f71644d"
+          (reference "#PWR0148") (unit 1)
+        )
+      )

Commit message: updated pin assignments
Changed lines of the file:
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@@
     (effects (font (size 1.27 1.27)) (justify right))
+  )
+  (symbol (lib_id "power:+3.3V") (at 143.51 87.63 0) (unit 1)
+    (in_bom yes) (on_board yes) (dnp no) (fields_autoplaced)
+    (property "Reference" "#PWR025" (at 143.51 91.44 0)
+      (effects (font (size 1.27 1.27)) hide)
+    )
+    (property "Value" "+3.3V" (at 143.51 83.82 0)
+      (effects (font (size 1.27 1.27)))
+    )
+    (property "Footprint" "" (at 143.51 87.63 0)
+      (effects (font (size 1.27 1.27)) hide)
+    )
+    (property "Datasheet" "" (at 143.51 87.63 0)
+      (effects (font (size 1.27 1.27)) hide)
+    )
+    (pin "1")
+    (instances
+      (project "LeaderSOM"
+        (path "/192d0c36-944e-4927-949b-263b8c85a7ca"
+          (reference "#PWR025") (unit 1)
+        )
+        (path "/192d0c36-944e-4927-949b-263b8c85a7ca/07cef2e6-f2f4-4f04-bcaf-7b98b53ab0fe"
+          (reference "#PWR025") (unit 1)
+        )
+        (path "/192d0c36-944e-4927-949b-263b8c85a7ca/54eecd34-7b2b-4895-a003-33708e7ad7e6"
+          (reference "#PWR028") (unit 1)
+        )
+      )
+      (project "BPS-PeripheralSOM"
+        (path "/d5ebd247-5a7c-47c2-8aee-beabaef72d6d"
+          (reference "#PWR02") (unit 1)
+        )
+      )
+    )
   )
   (symbol (lib_id "Device:R") (at 170.18 103.505 90) (unit 1)
@@
         (path "/7f2a449b-14af-42b3-8d38-5f0f8a5ee7ce"
           (reference "#PWR?") (unit 1)
+        )
+      )
+    )
+  )
+  (symbol (lib_id "power:+3.3V") (at 175.895 81.915 0) (unit 1)
+    (in_bom yes) (on_board yes) (dnp no) (fields_autoplaced)
+    (property "Reference" "#PWR025" (at 175.895 85.725 0)
+      (effects (font (size 1.27 1.27)) hide)
+    )
+    (property "Value" "+3.3V" (at 175.895 78.105 0)
+      (effects (font (size 1.27 1.27)))
+    )
+    (property "Footprint" "" (at 175.895 81.915 0)
+      (effects (font (size 1.27 1.27)) hide)
+    )
+    (property "Datasheet" "" (at 175.895 81.915 0)
+      (effects (font (size 1.27 1.27)) hide)
+    )
+    (pin "1")
+    (instances
+      (project "LeaderSOM"
+        (path "/192d0c36-944e-4927-949b-263b8c85a7ca"
+          (reference "#PWR025") (unit 1)
+        )
+        (path "/192d0c36-944e-4927-949b-263b8c85a7ca/07cef2e6-f2f4-4f04-bcaf-7b98b53ab0fe"
+          (reference "#PWR025") (unit 1)
+        )
+        (path "/192d0c36-944e-4927-949b-263b8c85a7ca/54eecd34-7b2b-4895-a003-33708e7ad7e6"
+          (reference "#PWR018") (unit 1)
+        )
+      )
+      (project "BPS-PeripheralSOM"
+        (path "/d5ebd247-5a7c-47c2-8aee-beabaef72d6d"
+          (reference "#PWR02") (unit 1)
         )
       )
@@
         (path "/d5ebd247-5a7c-47c2-8aee-beabaef72d6d"
           (reference "CR1") (unit 1)
-        )
-      )
-    )
-  )
-  (symbol (lib_id "power:+3.3V") (at 175.895 81.915 0) (unit 1)
-    (in_bom yes) (on_board yes) (dnp no)
-    (property "Reference" "#PWR018" (at 175.895 85.725 0)
-      (effects (font (size 1.27 1.27)) hide)
-    )
-    (property "Value" "+3.3V" (at 176.276 77.5208 0)
-      (effects (font (size 1.27 1.27)))
-    )
-    (property "Footprint" "" (at 175.895 81.915 0)
-      (effects (font (size 1.27 1.27)) hide)
-    )
-    (property "Datasheet" "" (at 175.895 81.915 0)
-      (effects (font (size 1.27 1.27)) hide)
-    )
-    (pin "1")
-    (instances
-      (project "LeaderSOM"
-        (path "/192d0c36-944e-4927-949b-263b8c85a7ca/54eecd34-7b2b-4895-a003-33708e7ad7e6"
-          (reference "#PWR018") (unit 1)
-        )
-      )
-      (project "Telemetry-Primary"
-        (path "/7f2a449b-14af-42b3-8d38-5f0f8a5ee7ce/00000000-0000-0000-0000-00005f71644d"
-          (reference "#PWR0148") (unit 1)
         )
       )
@@
         )
       )
-    )
-  )
-  (symbol (lib_id "power:+3.3V") (at 143.51 87.63 0) (unit 1)
-    (in_bom yes) (on_board yes) (dnp no)
-    (property "Reference" "#PWR028" (at 143.51 91.44 0)
-      (effects (font (size 1.27 1.27)) hide)
-    )
-    (property "Value" "+3.3V" (at 143.891 83.2358 0)
-      (effects (font (size 1.27 1.27)))
-    )
-    (property "Footprint" "" (at 143.51 87.63 0)
-      (effects (font (size 1.27 1.27)) hide)
-    )
-    (property "Datasheet" "" (at 143.51 87.63 0)
-      (effects (font (size 1.27 1.27)) hide)
-    )
-    (pin "1")
-    (instances
-      (project "LeaderSOM"
-        (path "/192d0c36-944e-4927-949b-263b8c85a7ca/54eecd34-7b2b-4895-a003-33708e7ad7e6"
-          (reference "#PWR028") (unit 1)
-        )
-      )
-      (project "Telemetry-Primary"
-        (path "/7f2a449b-14af-42b3-8d38-5f0f8a5ee7ce/00000000-0000-0000-0000-00005f71644d"
-          (reference "#PWR0148") (unit 1)
-        )
-      )
