File: SDCard.kicad_sch (KiCad schematic)
At the start: 3 parts, among them J4 Micro_SD_Card_Det

Commit message: u is for u n me
Connections:
- net SPI_CLK: now also CR1.1; no longer CR1.4
- net SPI_CS: now also CR1.4; no longer CR1.1
Changed lines of the file:
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@@
     (effects (font (size 1.27 1.27)) (justify right))
   )
-  (hierarchical_label "SPI_CS" (shape input) (at 90.805 93.98 180) (fields_autoplaced)
+  (hierarchical_label "SPI_CLK" (shape input) (at 90.805 93.98 180) (fields_autoplaced)
     (effects (font (size 1.27 1.27)) (justify right))
   )
@@
     (effects (font (size 1.27 1.27)) (justify left))
   )
-  (hierarchical_label "SPI_CLK" (shape input) (at 131.445 99.06 0) (fields_autoplaced)
+  (hierarchical_label "SPI_CS" (shape input) (at 131.445 99.06 0) (fields_autoplaced)
     (effects (font (size 1.27 1.27)) (justify left))
   )

Commit message: fix power dist, update to kicad 8
Parts:
- renumbered CR1 to CR2, R15 to R12

Commit message: Updated schem for redesign
Parts:
- added R5: 49.9, Resistor_SMD:R_0805_2012Metric, symbol Device:R
Connections:
- net +3.3V: now also J4.10 (DET_A)
- net DET: now also R5.1
- net GND: now also R5.2
- no-connect marks 3 -> 2
Other:
- note removed: "From telemetry primary PCB"
- moved on the sheet: R12

Commit message: fix lakshay things
Parts:
- R5: value 49.9 -> 10k
Changed lines of the file:
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@@
 			)
 		)
-		(property "Value" "49.9"
+		(property "Value" "10k"
 			(at 169.418 115.824 0)
 			(effects

Commit message: laid things out but still need to fix things :(
Connections:
- net SPI_CLK: now also CR2.4; no longer CR2.1
- net SPI_CS: now also CR2.1; no longer CR2.4
Changed lines of the file:
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@@
 	(hierarchical_label "SPI_CLK"
 		(shape input)
-		(at 90.805 93.98 180)
+		(at 131.445 99.06 0)
 		(fields_autoplaced yes)
 		(effects
@@
 				(size 1.27 1.27)
 			)
-			(justify right)
+			(justify left)
 		)
 	)
@@
 	(hierarchical_label "SPI_CS"
 		(shape input)
-		(at 131.445 99.06 0)
+		(at 90.805 93.98 180)
 		(fields_autoplaced yes)
 		(effects
@@
 				(size 1.27 1.27)
 			)
-			(justify left)
+			(justify right)
 		)
 	)

Commit message: hi again lakshay
Changed lines of the file:
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@@
 (kicad_sch
-	(version 20231120)
+	(version 20250114)
 	(generator "eeschema")
-	(generator_version "8.0")
+	(generator_version "9.0")
 	(paper "A4")
 	(junction
@@
 		(shape input)
 		(at 162.56 93.345 180)
-		(fields_autoplaced yes)
 		(effects
 			(font
@@
 		(shape output)
 		(at 162.56 103.505 180)
-		(fields_autoplaced yes)
 		(effects
 			(font
@@
 		(shape input)
 		(at 163.195 98.425 180)
-		(fields_autoplaced yes)
 		(effects
 			(font
@@
 		(shape input)
 		(at 131.445 99.06 0)
-		(fields_autoplaced yes)
 		(effects
 			(font
@@
 		(shape output)
 		(at 90.805 99.06 180)
-		(fields_autoplaced yes)
 		(effects
 			(font
@@
 		(shape input)
 		(at 131.445 93.98 0)
-		(fields_autoplaced yes)
 		(effects
 			(font
@@
 		(shape input)
 		(at 90.805 93.98 180)
-		(fields_autoplaced yes)
 		(effects
 			(font
@@
 		(shape output)
 		(at 162.56 111.125 180)
-		(fields_autoplaced yes)
 		(effects
 			(font
@@
 		(shape input)
 		(at 162.56 90.805 180)
-		(fields_autoplaced yes)
 		(effects
 			(font
@@
 			)
 			(project "Telemetry-Primary"
+				(path "/7f2a449b-14af-42b3-8d38-5f0f8a5ee7ce"
+					(reference "R2")
+					(unit 1)
+				)
 				(path "/7f2a449b-14af-42b3-8d38-5f0f8a5ee7ce/00000000-0000-0000-0000-00005f6cdfd6"
 					(reference "R?")
-					(unit 1)
-				)
-				(path "/7f2a449b-14af-42b3-8d38-5f0f8a5ee7ce"
-					(reference "R2")
 					(unit 1)
 				)
@@
 			)
 			(project "Telemetry-Primary"
+				(path "/7f2a449b-14af-42b3-8d38-5f0f8a5ee7ce"
+					(reference "#PWR?")
+					(unit 1)
+				)
 				(path "/7f2a449b-14af-42b3-8d38-5f0f8a5ee7ce/00000000-0000-0000-0000-00005f71644d"
 					(reference "#PWR0147")
-					(unit 1)
-				)
-				(path "/7f2a449b-14af-42b3-8d38-5f0f8a5ee7ce"
-					(reference "#PWR?")
 					(unit 1)
 				)
@@
 			)
 			(project "Telemetry-Primary"
+				(path "/7f2a449b-14af-42b3-8d38-5f0f8a5ee7ce"
+					(reference "#PWR?")
+					(unit 1)
+				)
 				(path "/7f2a449b-14af-42b3-8d38-5f0f8a5ee7ce/00000000-0000-0000-0000-00005f71644d"
 					(reference "#PWR0147")
 					(unit 1)
 				)
-				(path "/7f2a449b-14af-42b3-8d38-5f0f8a5ee7ce"
-					(reference "#PWR?")
-					(unit 1)
-				)
