File: SDCard.kicad_sch (KiCad schematic)
At the start: 4 parts, among them J4 Micro_SD_Card_Det

Commit message: net class fixes and ERC
Connections:
- net +3.3V renamed +3V3
Changed lines of the file:
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@@
 	(symbol
 		(lib_id "power:+3.3V")
-		(at 143.51 87.63 0)
-		(unit 1)
-		(exclude_from_sim no)
-		(in_bom yes)
-		(on_board yes)
-		(dnp no)
-		(fields_autoplaced yes)
-		(property "Reference" "#PWR028"
-			(at 143.51 91.44 0)
-			(effects
-				(font
-					(size 1.27 1.27)
-				)
-				(hide yes)
-			)
-		)
-		(property "Value" "+3.3V"
-			(at 143.51 83.82 0)
+		(at 174.625 85.725 0)
+		(unit 1)
+		(exclude_from_sim no)
+		(in_bom yes)
+		(on_board yes)
+		(dnp no)
+		(property "Reference" "#PWR0129"
+			(at 174.625 89.535 0)
+			(effects
+				(font
+					(size 1.27 1.27)
+				)
+				(hide yes)
+			)
+		)
+		(property "Value" "+3V3"
+			(at 175.006 81.3308 0)
 			(effects
 				(font
@@
 		)
 		(property "Footprint" ""
-			(at 143.51 87.63 0)
+			(at 174.625 85.725 0)
 			(effects
 				(font
@@
 		)
 		(property "Datasheet" ""
-			(at 143.51 87.63 0)
+			(at 174.625 85.725 0)
 			(effects
 				(font
@@
 		)
 		(property "Description" "Power symbol creates a global label with name \"+3.3V\""
-			(at 143.51 87.63 0)
-			(effects
-				(font
-					(size 1.27 1.27)
-				)
-				(hide yes)
-			)
-		)
-		(pin "1"
-		)
-		(instances
-			(project "LeaderSOM"
-				(path "/192d0c36-944e-4927-949b-263b8c85a7ca/54eecd34-7b2b-4895-a003-33708e7ad7e6"
-					(reference "#PWR028")
-					(unit 1)
-				)
-			)
-			(project "BPS-PeripheralSOM"
-				(path "/d5ebd247-5a7c-47c2-8aee-beabaef72d6d"
-					(reference "#PWR02")
+			(at 174.625 85.725 0)
+			(effects
+				(font
+					(size 1.27 1.27)
+				)
+				(hide yes)
+			)
+		)
+		(pin "1"
+		)
+		(instances
+			(project "LeaderSOM"
+				(path "/192d0c36-944e-4927-949b-263b8c85a7ca/54eecd34-7b2b-4895-a003-33708e7ad7e6"
+					(reference "#PWR0129")
 					(unit 1)
 				)
@@
 	)
 	(symbol
-		(lib_id "power:+3.3V")
-		(at 174.625 85.725 0)
-		(unit 1)
-		(exclude_from_sim no)
-		(in_bom yes)
-		(on_board yes)
-		(dnp no)
-		(fields_autoplaced yes)
-		(property "Reference" "#PWR018"
-			(at 174.625 89.535 0)
-			(effects
-				(font
-					(size 1.27 1.27)
-				)
-				(hide yes)
-			)
-		)
-		(property "Value" "+3.3V"
-			(at 174.625 81.915 0)
-			(effects
-				(font
-					(size 1.27 1.27)
-				)
-			)
-		)
-		(property "Footprint" ""
-			(at 174.625 85.725 0)
-			(effects
-				(font
-					(size 1.27 1.27)
-				)
-				(hide yes)
-			)
-		)
-		(property "Datasheet" ""
-			(at 174.625 85.725 0)
-			(effects
-				(font
-					(size 1.27 1.27)
-				)
-				(hide yes)
-			)
-		)
-		(property "Description" "Power symbol creates a global label with name \"+3.3V\""
-			(at 174.625 85.725 0)
-			(effects
-				(font
-					(size 1.27 1.27)
-				)
-				(hide yes)
-			)
-		)
-		(pin "1"
-		)
-		(instances
-			(project "LeaderSOM"
-				(path "/192d0c36-944e-4927-949b-263b8c85a7ca/54eecd34-7b2b-4895-a003-33708e7ad7e6"
-					(reference "#PWR018")
-					(unit 1)
-				)
-			)
-			(project "BPS-PeripheralSOM"
-				(path "/d5ebd247-5a7c-47c2-8aee-beabaef72d6d"
-					(reference "#PWR02")
-					(unit 1)
-				)
-			)
-		)
-	)
-	(symbol
 		(lib_id "utsvt-chips:D5V0P4UR6SO-7")
 		(at 90.805 93.98 0)
@@
 					(unit 1)
 				)
+			)
+		)
+	)
+	(symbol
+		(lib_id "power:+3.3V")
+		(at 143.51 87.63 0)
+		(unit 1)
+		(exclude_from_sim no)
+		(in_bom yes)
+		(on_board yes)
+		(dnp no)
+		(property "Reference" "#PWR0128"
+			(at 143.51 91.44 0)
+			(effects
+				(font
+					(size 1.27 1.27)
+				)
+				(hide yes)
+			)
+		)
+		(property "Value" "+3V3"
+			(at 143.891 83.2358 0)
+			(effects
+				(font
+					(size 1.27 1.27)
+				)
+			)
+		)
+		(property "Footprint" ""
+			(at 143.51 87.63 0)
+			(effects
+				(font
+					(size 1.27 1.27)
+				)
+				(hide yes)
+			)
+		)
+		(property "Datasheet" ""
+			(at 143.51 87.63 0)
+			(effects
+				(font
+					(size 1.27 1.27)
+				)
+				(hide yes)
+			)
+		)
+		(property "Description" "Power symbol creates a global label with name \"+3.3V\""
+			(at 143.51 87.63 0)
+			(effects
+				(font
+					(size 1.27 1.27)
+				)
+				(hide yes)
+			)
+		)
+		(pin "1"
+		)
+		(instances
+			(project "LeaderSOM"
+				(path "/192d0c36-944e-4927-949b-263b8c85a7ca/54eecd34-7b2b-4895-a003-33708e7ad7e6"
+					(reference "#PWR0128")
+					(unit 1)
+				)

Commit message: workday for review
Parts:
- CR2: footprint UTSVT_ICs:SOT26_DIO -> UTSVT_ICs:D5V0P4UR6SO-7; symbol utsvt-chips:D5V0P4UR6SO-7 -> UTSVT-ICs:D5V0P4UR6SO-7; Mouser Part Number (none) -> 621-D5V0P4UR6SO-7; P/N (none) -> D5V0P4UR6SO-7
- J4: footprint UTSVT_Connectors:microSD_HC_Hirose_DM3AT-SF-PEJM5 -> SD_CARD:microSD_HC_Hirose_DM3AT-SF-PEJM5
Changed lines of the file:
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@@
 	)
 	(symbol
-		(lib_id "utsvt-chips:D5V0P4UR6SO-7")
+		(lib_id "UTSVT-ICs:D5V0P4UR6SO-7")
 		(at 90.805 93.98 0)
 		(unit 1)
@@
 			)
 		)
-		(property "Footprint" "UTSVT_ICs:SOT26_DIO"
+		(property "Footprint" "UTSVT_ICs:D5V0P4UR6SO-7"
 			(at 111.125 90.17 0)
 			(effects
@@
 		)
 		(property "Description" ""
+			(at 90.805 93.98 0)
+			(effects
+				(font
+					(size 1.27 1.27)
+				)
+				(hide yes)
+			)
+		)
+		(property "Mouser Part Number" "621-D5V0P4UR6SO-7"
+			(at 90.805 93.98 0)
+			(effects
+				(font
+					(size 1.27 1.27)
+				)
+				(hide yes)
+			)
+		)
+		(property "P/N" "D5V0P4UR6SO-7"
+			(at 90.805 93.98 0)
+			(effects
+				(font
+					(size 1.27 1.27)
+				)
+				(hide yes)
+			)
+		)
+		(property "PN" ""
+			(at 90.805 93.98 0)
+			(effects
+				(font
+					(size 1.27 1.27)
+				)
+				(hide yes)
+			)
+		)
+		(property "p/n" ""
 			(at 90.805 93.98 0)
 			(effects
@@
 			)
 		)
-		(property "Footprint" "UTSVT_Connectors:microSD_HC_Hirose_DM3AT-SF-PEJM5"
+		(property "Footprint" "SD_CARD:microSD_HC_Hirose_DM3AT-SF-PEJM5"
 			(at 253.365 80.645 0)
 			(effects

Commit message: crazy? i used to be crazy
Parts:
- R12: renamed from R5; footprint Resistor_SMD:R_0805_2012Metric -> Resistor_SMD:R_0603_1608Metric
- R13: renamed from R12; footprint Resistor_SMD:R_0805_2012Metric -> Resistor_SMD:R_0603_1608Metric
- renumbered CR2 to CR1
Changed lines of the file:
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@@
 		(on_board yes)
 		(dnp no)
-		(property "Reference" "#PWR014"
+		(property "Reference" "#PWR038"
 			(at 167.64 125.095 0)
 			(effects
@@
 			(project "LeaderSOM"
 				(path "/192d0c36-944e-4927-949b-263b8c85a7ca/54eecd34-7b2b-4895-a003-33708e7ad7e6"
-					(reference "#PWR014")
+					(reference "#PWR038")
 					(unit 1)
 				)
@@
 		(on_board yes)
 		(dnp no)
-		(property "Reference" "#PWR0129"
+		(property "Reference" "#PWR039"
 			(at 174.625 89.535 0)
 			(effects
@@
 			(project "LeaderSOM"
 				(path "/192d0c36-944e-4927-949b-263b8c85a7ca/54eecd34-7b2b-4895-a003-33708e7ad7e6"
-					(reference "#PWR0129")
+					(reference "#PWR039")
 					(unit 1)
 				)
@@
 		(on_board yes)
 		(dnp no)
-		(property "Reference" "R12"
+		(property "Reference" "R13"
 			(at 170.815 99.06 90)
 			(effects
@@
 			)
 		)
-		(property "Footprint" "Resistor_SMD:R_0805_2012Metric"
+		(property "Footprint" "Resistor_SMD:R_0603_1608Metric"
 			(at 168.91 105.283 90)
 			(effects
@@
 			(project "LeaderSOM"
 				(path "/192d0c36-944e-4927-949b-263b8c85a7ca/54eecd34-7b2b-4895-a003-33708e7ad7e6"
-					(reference "R12")
+					(reference "R13")
 					(unit 1)
 				)
@@
 		(on_board yes)
 		(dnp no)
-		(property "Reference" "#PWR019"
+		(property "Reference" "#PWR040"
 			(at 200.025 126.365 0)
 			(effects
@@
 			(project "LeaderSOM"
 				(path "/192d0c36-944e-4927-949b-263b8c85a7ca/54eecd34-7b2b-4895-a003-33708e7ad7e6"
-					(reference "#PWR019")
+					(reference "#PWR040")
 					(unit 1)
 				)
@@
 		(on_board yes)
 		(dnp no)
-		(property "Reference" "#PWR016"
+		(property "Reference" "#PWR036"
 			(at 77.47 109.22 0)
 			(effects
@@
 			(project "LeaderSOM"
 				(path "/192d0c36-944e-4927-949b-263b8c85a7ca/54eecd34-7b2b-4895-a003-33708e7ad7e6"
-					(reference "#PWR016")
+					(reference "#PWR036")
 					(unit 1)
 				)
@@
 		(dnp no)
 		(fields_autoplaced yes)
-		(property "Reference" "CR2"
+		(property "Reference" "CR1"
 			(at 111.125 83.82 0)
 			(effects
@@
 			(project "LeaderSOM"
 				(path "/192d0c36-944e-4927-949b-263b8c85a7ca/54eecd34-7b2b-4895-a003-33708e7ad7e6"
-					(reference "CR2")
+					(reference "CR1")
 					(unit 1)
 				)
@@
 		(on_board yes)
 		(dnp no)
-		(property "Reference" "#PWR0128"
+		(property "Reference" "#PWR037"
 			(at 143.51 91.44 0)
 			(effects
@@
 			(project "LeaderSOM"
 				(path "/192d0c36-944e-4927-949b-263b8c85a7ca/54eecd34-7b2b-4895-a003-33708e7ad7e6"
-					(reference "#PWR0128")
+					(reference "#PWR037")
 					(unit 1)
 				)
@@
 		(on_board yes)
 		(dnp no)
-		(property "Reference" "R5"
+		(property "Reference" "R12"
 			(at 170.18 113.792 0)
 			(effects
@@
 			)
 		)
-		(property "Footprint" "Resistor_SMD:R_0805_2012Metric"
+		(property "Footprint" "Resistor_SMD:R_0603_1608Metric"
 			(at 165.862 114.935 90)
 			(effects
@@
 			(project "LeaderSOM"
 				(path "/192d0c36-944e-4927-949b-263b8c85a7ca/54eecd34-7b2b-4895-a003-33708e7ad7e6"
-					(reference "R5")
-					(unit 1)
-				)
+					(reference "R12")
+					(unit 1)
+				)

Commit message: workday
Parts:
- R12, R13: footprint Resistor_SMD:R_0603_1608Metric -> Resistor_SMD:R_0603_1608Metric_Pad0.98x0.95mm_HandSolder
Changed lines of the file:
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@@
 			)
 		)
-		(property "Footprint" "Resistor_SMD:R_0603_1608Metric"
+		(property "Footprint" "Resistor_SMD:R_0603_1608Metric_Pad0.98x0.95mm_HandSolder"
 			(at 168.91 105.283 90)
 			(effects
@@
 			)
 		)
-		(property "Footprint" "Resistor_SMD:R_0603_1608Metric"
+		(property "Footprint" "Resistor_SMD:R_0603_1608Metric_Pad0.98x0.95mm_HandSolder"
 			(at 165.862 114.935 90)
 			(effects

Commit message: tweaking
Parts:
- J4: footprint SD_CARD:microSD_HC_Hirose_DM3AT-SF-PEJM5 -> Connector_Card:microSD_HC_Hirose_DM3AT-SF-PEJM5
Changed lines of the file:
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@@
 			)
 		)
-		(property "Footprint" "SD_CARD:microSD_HC_Hirose_DM3AT-SF-PEJM5"
+		(property "Footprint" "Connector_Card:microSD_HC_Hirose_DM3AT-SF-PEJM5"
 			(at 253.365 80.645 0)
 			(effects

Commit message: bom
Parts:
- J4: Mouser Part Number (none) -> DM3AT-SF-PEJM5
- R12: Mouser Part Number (none) -> CRCW060310K0FKEI
- R13: Mouser Part Number (none) -> RT0603BRE0750RL
Changed lines of the file:
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@@
+			)
+		)
+		(property "Mouser Part Number" "RT0603BRE0750RL"
+			(at 168.91 103.505 0)
+			(effects
+				(font
+					(size 1.27 1.27)
+				)
 			)
 		)
@@
 			)
 		)
+		(property "Mouser Part Number" "DM3AT-SF-PEJM5"
+			(at 201.295 98.425 0)
+			(effects
+				(font
+					(size 1.27 1.27)
+				)
+			)
+		)
 		(pin "1"
 		)
@@
 			(at 167.64 114.935 0)
 			(effects
+				(font
+					(size 1.27 1.27)
+				)
+			)
+		)
+		(property "Mouser Part Number" "CRCW060310K0FKEI "
+			(at 167.64 114.935 0)
+			(effects

Commit message: updated pins
Parts:
- renumbered R13 to R10, R12 to R9
Changed lines of the file:
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@@
 		(on_board yes)
 		(dnp no)
-		(property "Reference" "#PWR038"
+		(property "Reference" "#PWR030"
 			(at 167.64 125.095 0)
 			(effects
@@
 			(project "LeaderSOM"
 				(path "/192d0c36-944e-4927-949b-263b8c85a7ca/54eecd34-7b2b-4895-a003-33708e7ad7e6"
-					(reference "#PWR038")
+					(reference "#PWR030")
 					(unit 1)
 				)
@@
 		(on_board yes)
 		(dnp no)
-		(property "Reference" "#PWR039"
+		(property "Reference" "#PWR031"
 			(at 174.625 89.535 0)
 			(effects
@@
 			(project "LeaderSOM"
 				(path "/192d0c36-944e-4927-949b-263b8c85a7ca/54eecd34-7b2b-4895-a003-33708e7ad7e6"
-					(reference "#PWR039")
+					(reference "#PWR031")
 					(unit 1)
 				)
@@
 		(on_board yes)
 		(dnp no)
-		(property "Reference" "R13"
+		(property "Reference" "R10"
 			(at 170.815 99.06 90)
 			(effects
@@
 			(project "LeaderSOM"
 				(path "/192d0c36-944e-4927-949b-263b8c85a7ca/54eecd34-7b2b-4895-a003-33708e7ad7e6"
-					(reference "R13")
+					(reference "R10")
 					(unit 1)
 				)
@@
 		(on_board yes)
 		(dnp no)
-		(property "Reference" "#PWR040"
+		(property "Reference" "#PWR032"
 			(at 200.025 126.365 0)
 			(effects
@@
 			(project "LeaderSOM"
 				(path "/192d0c36-944e-4927-949b-263b8c85a7ca/54eecd34-7b2b-4895-a003-33708e7ad7e6"
-					(reference "#PWR040")
+					(reference "#PWR032")
 					(unit 1)
 				)
@@
 		(on_board yes)
 		(dnp no)
-		(property "Reference" "#PWR036"
+		(property "Reference" "#PWR028"
 			(at 77.47 109.22 0)
 			(effects
@@
 			(project "LeaderSOM"
 				(path "/192d0c36-944e-4927-949b-263b8c85a7ca/54eecd34-7b2b-4895-a003-33708e7ad7e6"
-					(reference "#PWR036")
+					(reference "#PWR028")
 					(unit 1)
 				)
@@
 		(on_board yes)
 		(dnp no)
-		(property "Reference" "#PWR037"
+		(property "Reference" "#PWR029"
 			(at 143.51 91.44 0)
 			(effects
@@
 			(project "LeaderSOM"
 				(path "/192d0c36-944e-4927-949b-263b8c85a7ca/54eecd34-7b2b-4895-a003-33708e7ad7e6"
-					(reference "#PWR037")
+					(reference "#PWR029")
 					(unit 1)
 				)
@@
 		(on_board yes)
 		(dnp no)
-		(property "Reference" "R12"
+		(property "Reference" "R9"
 			(at 170.18 113.792 0)
 			(effects
@@
 			(project "LeaderSOM"
 				(path "/192d0c36-944e-4927-949b-263b8c85a7ca/54eecd34-7b2b-4895-a003-33708e7ad7e6"
-					(reference "R12")
-					(unit 1)
-				)
+					(reference "R9")
+					(unit 1)
+				)
