File: Display.kicad_sch (KiCad schematic)
At the start: 16 parts

Commit message: changed 12V/5V DC/DC output setting resistors to a generic 1K and 0 Ohm pair, updated LED display to proper model
Parts:
- LED1, LED2: value 157112B12800 -> 157121S12800; P/N 157112B12800 -> 157121S12800
Changed lines of the file:
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@@
       (effects (font (size 1.524 1.524)))
     )
-    (property "Value" "157112B12800" (at 206.6965 78.74 0)
+    (property "Value" "157121S12800" (at 206.6965 78.74 0)
       (effects (font (size 1.524 1.524)))
     )
@@
       (effects (font (size 1.27 1.27) italic) hide)
     )
-    (property "Datasheet" "157121S12800" (at 182.245 81.915 0)
-      (effects (font (size 1.27 1.27) italic) hide)
-    )
-    (property "P/N" "157112B12800" (at 182.245 81.915 0)
+    (property "Datasheet" "https://www.we-online.com/components/products/datasheet/157121S12800.pdf" (at 182.245 81.915 0)
+      (effects (font (size 1.27 1.27) italic) hide)
+    )
+    (property "P/N" "157121S12800" (at 182.245 81.915 0)
       (effects (font (size 1.27 1.27)) hide)
     )
@@
       (effects (font (size 1.524 1.524)))
     )
-    (property "Value" "157112B12800" (at 131.1315 79.375 0)
+    (property "Value" "157121S12800" (at 131.1315 79.375 0)
       (effects (font (size 1.524 1.524)))
     )
@@
       (effects (font (size 1.27 1.27) italic) hide)
     )
-    (property "Datasheet" "157121S12800" (at 106.68 82.55 0)
-      (effects (font (size 1.27 1.27) italic) hide)
-    )
-    (property "P/N" "157112B12800" (at 106.68 82.55 0)
-      (effects (font (size 1.27 1.27)) hide)
-    )
+    (property "Datasheet" "https://www.we-online.com/components/products/datasheet/157121S12800.pdf" (at 106.68 82.55 0)
+      (effects (font (size 1.27 1.27) italic) hide)
+    )
+    (property "P/N" "157121S12800" (at 106.68 82.55 0)
+      (effects (font (size 1.27 1.27)) hide)
+    )

Commit message: starting redesign
Parts:
- added C?: 0.1u, symbol Device:C
- added C?: C_Small, symbol Device:C_Small
- added R9, R?: 10k, symbol Device:R_Small
- added U?: SN74HCS595DYYR, SOT_95DYYR_TEX, symbol SN74HCS595DYYR:SN74HCS595DYYR
Connections:
- net LED3 is gone; now on net LEDC: R21.1
- net LED4 is gone; now on net LEDD: R23.1
- net LED5 is gone; now on net LEDE: R24.1
- net LED6 is gone; now on net LEDF: R25.1
- net LED7 is gone; now on net LEDG: R26.1
- net LED8 is gone; now on net LEDA: R27.1
- net LED9 is gone; now on net LEDB: R28.1
- net +3.3V: now also C?.1, R?.1, U?.16; no longer LED1.3, LED1.8, LED2.3, LED2.8
- net LED1 renamed LEDA
- net LEDA: now also U?.15
- net LED10 renamed LEDC
- net LEDC: now also U?.2
- net LED11 renamed LEDD
- net LEDD: now also U?.3
- net LED12 renamed LEDE
- net LEDE: now also U?.4
- net LED13 renamed LEDF
- net LEDF: now also U?.5
- net LED14 renamed LEDG
- net LEDG: now also U?.6
- net LED2 renamed LEDB
- net LEDB: now also U?.1
- new net: C?.1, R?.2, U?.10
- new net: R9.2, U?.13
- new net Cathode1: LED1.3, LED1.8, U?.7
- new net Cathode2: LED2.3, LED2.8, U?.9
- new net GND: C?.2, C?.2, R9.1, U?.8
- new net Output Clock: U?.12
- new net SR Clock: U?.11
- new net Serial Input: U?.14
Other:
- moved on the sheet: LED1, LED2, R14, R16, R21, R23, R24, R25, R26, R27, R28, R29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

Commit message: MCU pins, PSON power distribution, KiCad-Sharepoint, and 7 seg
Parts:
- gave numbers to parts that had none: 4
Changed lines of the file:
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@@
 		(dnp no)
 		(fields_autoplaced yes)
-		(property "Reference" "C?"
+		(property "Reference" "C1"
 			(at 30.48 99.6949 0)
 			(effects
@@
 			(project ""
 				(path "/192d0c36-944e-4927-949b-263b8c85a7ca/8c1921d3-7d8b-4937-baba-7ed9d4d1349f"
-					(reference "C?")
+					(reference "C1")
 					(unit 1)
 				)
@@
 		(dnp no)
 		(fields_autoplaced yes)
-		(property "Reference" "C?"
+		(property "Reference" "C2"
 			(at 113.03 108.5912 0)
 			(effects
@@
 			(project ""
 				(path "/192d0c36-944e-4927-949b-263b8c85a7ca/8c1921d3-7d8b-4937-baba-7ed9d4d1349f"
-					(reference "C?")
+					(reference "C2")
 					(unit 1)
 				)
@@
 		(dnp no)
 		(fields_autoplaced yes)
-		(property "Reference" "U?"
+		(property "Reference" "U8"
 			(at 76.2 80.645 0)
 			(effects
@@
 			(project ""
 				(path "/192d0c36-944e-4927-949b-263b8c85a7ca/8c1921d3-7d8b-4937-baba-7ed9d4d1349f"
-					(reference "U?")
+					(reference "U8")
 					(unit 1)
 				)
@@
 		(dnp no)
 		(fields_autoplaced yes)
-		(property "Reference" "R?"
+		(property "Reference" "R1"
 			(at 113.665 100.33 90)
 			(effects
@@
 			(project ""
 				(path "/192d0c36-944e-4927-949b-263b8c85a7ca/8c1921d3-7d8b-4937-baba-7ed9d4d1349f"
-					(reference "R?")
-					(unit 1)
-				)
+					(reference "R1")
+					(unit 1)
+				)

Commit message: net class fixes and ERC
Parts:
- C1, C2: footprint (none) -> Capacitor_SMD:C_0603_1608Metric
- R1, R9: footprint (none) -> Resistor_SMD:R_0603_1608Metric
- U8: footprint SOT_95DYYR_TEX -> SN74HC595:SOT_95DYYR_TEX
Connections:
- net +3.3V renamed +3V3
