File: Display.kicad_sch (KiCad schematic)
At the start: 21 parts, among them U8 SN74HCS595DYYR

Commit message: workday for review
Parts:
- added R44, R55: 160, Resistor_SMD:R_0805_2012Metric, symbol Device:R_Small
- LED1, LED2: footprint UTSVT_Special:SMT_1S12800_WRE -> 7-segment:SMT_1S12800_WRE; symbol utsvt-misc:157112B12800 -> Seven-Segment:157121512800
Connections:
- net +3V3: no longer LED1.5 (DP), LED2.5 (DP)
- net Cathode1 renamed Anode1
- net Anode1: no longer U8.7
- net Cathode2 renamed Anode2
- net Anode2: no longer U8.9
- new net: LED2.5 (DP), R55.2
- new net: LED1.5 (DP), R44.2
- new net LEDH: R44.1, R55.1, U8.7
- no-connect marks 0 -> 1

Commit message: macbook hater
Parts:
- U8: footprint SN74HC595:SOT_95DYYR_TEX -> SOT_95DYYR_TEX
Changed lines of the file:
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@@
 			)
 		)
-		(property "Footprint" "SN74HC595:SOT_95DYYR_TEX"
+		(property "Footprint" "SOT_95DYYR_TEX"
 			(at 55.88 90.17 0)
 			(effects
