File: LeaderSOM.kicad_sch (KiCad schematic)
At the start: 27 parts, among them IC2 TPS1120DR, J1 SWD, J10 SOMConnector, J9 SOMConnector, SW1 Reset, SW2 BTN1, U6 STM32F413RHTx, Y2 8M

Commit message: 👹
Parts:
- IC2: footprint SOIC127P600X175-8N -> UTSVT_ICs:SOIC127P600X175-8N
Connections:
- net VDDA is gone; now on net +3.3VA: C28.1, C30.1, U6.13 (VDDA)
Changed lines of the file:
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@@
   (junction (at 123.19 124.46) (diameter 0) (color 0 0 0 0)
   )
-  (junction (at 138.43 27.305) (diameter 0) (color 0 0 0 0)
-  )
-  (junction (at 130.81 24.765) (diameter 0) (color 0 0 0 0)
-  )
   (junction (at 247.65 80.645) (diameter 0) (color 0 0 0 0)
   )
@@
   )
   (junction (at 90.17 118.745) (diameter 0) (color 0 0 0 0)
-  )
-  (junction (at 141.605 128.27) (diameter 0) (color 0 0 0 0)
   )
   (junction (at 215.9 152.4) (diameter 0) (color 0 0 0 0)
@@
     (stroke (width 0) (type default))
   )
-  (wire (pts (xy 141.605 128.27) (xy 141.605 129.54))
+  (wire (pts (xy 141.605 124.46) (xy 141.605 129.54))
     (stroke (width 0) (type default))
   )
@@
     (stroke (width 0) (type default))
   )
-  (wire (pts (xy 138.43 26.035) (xy 138.43 27.305))
+  (wire (pts (xy 138.43 26.035) (xy 138.43 28.575))
     (stroke (width 0) (type default))
   )
@@
     (stroke (width 0) (type default))
   )
-  (wire (pts (xy 138.43 27.305) (xy 138.43 28.575))
-    (stroke (width 0) (type default))
-  )
   (wire (pts (xy 220.98 31.115) (xy 222.885 31.115))
     (stroke (width 0) (type default))
@@
     (stroke (width 0) (type default))
   )
-  (wire (pts (xy 130.81 27.305) (xy 130.81 24.765))
-    (stroke (width 0) (type default))
-  )
   (wire (pts (xy 148.59 76.835) (xy 171.45 76.835))
     (stroke (width 0) (type default))
@@
     (stroke (width 0) (type default))
   )
-  (wire (pts (xy 141.605 124.46) (xy 141.605 128.27))
-    (stroke (width 0) (type default))
-  )
-  (wire (pts (xy 130.81 24.765) (xy 130.81 22.86))
+  (wire (pts (xy 130.81 22.86) (xy 130.81 27.305))
     (stroke (width 0) (type default))
   )
@@
         (path "/d5ebd247-5a7c-47c2-8aee-beabaef72d6d"
           (reference "#PWR045") (unit 1)
-        )
-      )
-    )
-  )
-  (symbol (lib_id "power:PWR_FLAG") (at 141.605 128.27 270) (unit 1)
-    (in_bom yes) (on_board yes) (dnp no) (fields_autoplaced)
-    (property "Reference" "#FLG04" (at 143.51 128.27 0)
-      (effects (font (size 1.27 1.27)) hide)
-    )
-    (property "Value" "PWR_FLAG" (at 144.78 128.905 90)
-      (effects (font (size 1.27 1.27)) (justify left))
-    )
-    (property "Footprint" "" (at 141.605 128.27 0)
-      (effects (font (size 1.27 1.27)) hide)
-    )
-    (property "Datasheet" "~" (at 141.605 128.27 0)
-      (effects (font (size 1.27 1.27)) hide)
-    )
-    (pin "1")
-    (instances
-      (project "LeaderSOM"
-        (path "/192d0c36-944e-4927-949b-263b8c85a7ca"
-          (reference "#FLG04") (unit 1)
         )
       )
@@
     )
   )
-  (symbol (lib_id "power:PWR_FLAG") (at 130.81 24.765 90) (unit 1)
+  (symbol (lib_id "power:+3.3VA") (at 246.38 109.22 0) (unit 1)
     (in_bom yes) (on_board yes) (dnp no) (fields_autoplaced)
-    (property "Reference" "#FLG05" (at 128.905 24.765 0)
-      (effects (font (size 1.27 1.27)) hide)
-    )
-    (property "Value" "PWR_FLAG" (at 127.635 25.4 90)
-      (effects (font (size 1.27 1.27)) (justify left))
-    )
-    (property "Footprint" "" (at 130.81 24.765 0)
-      (effects (font (size 1.27 1.27)) hide)
-    )
-    (property "Datasheet" "~" (at 130.81 24.765 0)
-      (effects (font (size 1.27 1.27)) hide)
-    )
-    (pin "1")
-    (instances
-      (project "LeaderSOM"
-        (path "/192d0c36-944e-4927-949b-263b8c85a7ca"
-          (reference "#FLG05") (unit 1)
+    (property "Reference" "#PWR052" (at 246.38 113.03 0)
+      (effects (font (size 1.27 1.27)) hide)
+    )
+    (property "Value" "+3.3VA" (at 246.38 104.775 0)
+      (effects (font (size 1.27 1.27)))
+    )
+    (property "Footprint" "" (at 246.38 109.22 0)
+      (effects (font (size 1.27 1.27)) hide)
+    )
+    (property "Datasheet" "" (at 246.38 109.22 0)
+      (effects (font (size 1.27 1.27)) hide)
+    )
+    (pin "1")
+    (instances
+      (project "LeaderSOM"
+        (path "/192d0c36-944e-4927-949b-263b8c85a7ca/07cef2e6-f2f4-4f04-bcaf-7b98b53ab0fe"
+          (reference "#PWR052") (unit 1)
+        )
+        (path "/192d0c36-944e-4927-949b-263b8c85a7ca"
+          (reference "#PWR053") (unit 1)
         )
       )
@@
     )
   )
-  (symbol (lib_id "power:VDDA") (at 138.43 26.035 0) (unit 1)
-    (in_bom yes) (on_board yes) (dnp no) (fields_autoplaced)
-    (property "Reference" "#PWR050" (at 138.43 29.845 0)
-      (effects (font (size 1.27 1.27)) hide)
-    )
-    (property "Value" "VDDA" (at 138.43 22.86 0)
-      (effects (font (size 1.27 1.27)))
-    )
-    (property "Footprint" "" (at 138.43 26.035 0)
-      (effects (font (size 1.27 1.27)) hide)
-    )
-    (property "Datasheet" "" (at 138.43 26.035 0)
-      (effects (font (size 1.27 1.27)) hide)
-    )
-    (pin "1")
-    (instances
-      (project "LeaderSOM"
-        (path "/192d0c36-944e-4927-949b-263b8c85a7ca"
-          (reference "#PWR050") (unit 1)
-        )
-      )
-      (project "BPS-PeripheralSOM"
-        (path "/d5ebd247-5a7c-47c2-8aee-beabaef72d6d"
-          (reference "#PWR01") (unit 1)
-        )
-      )
-    )
-  )
-  (symbol (lib_id "power:VDDA") (at 246.38 109.22 0) (unit 1)
-    (in_bom yes) (on_board yes) (dnp no)
-    (property "Reference" "#PWR053" (at 246.38 113.03 0)
-      (effects (font (size 1.27 1.27)) hide)
-    )
-    (property "Value" "VDDA" (at 246.38 105.41 0)
-      (effects (font (size 1.27 1.27)))
-    )
-    (property "Footprint" "" (at 246.38 109.22 0)
-      (effects (font (size 1.27 1.27)) hide)
-    )
-    (property "Datasheet" "" (at 246.38 109.22 0)
-      (effects (font (size 1.27 1.27)) hide)
-    )
-    (pin "1")
-    (instances
-      (project "LeaderSOM"
-        (path "/192d0c36-944e-4927-949b-263b8c85a7ca"
-          (reference "#PWR053") (unit 1)
-        )
-      )
-      (project "BPS-PeripheralSOM"
-        (path "/d5ebd247-5a7c-47c2-8aee-beabaef72d6d"
-          (reference "#PWR012") (unit 1)
-        )
-      )
-    )
-  )
   (symbol (lib_id "Device:C") (at 219.71 115.57 0) (unit 1)
     (in_bom yes) (on_board yes) (dnp no) (fields_autoplaced)
@@
       (effects (font (size 1.27 1.27)))
     )
-    (property "Footprint" "SOIC127P600X175-8N" (at 95.25 261.925 0)
+    (property "Footprint" "UTSVT_ICs:SOIC127P600X175-8N" (at 95.25 261.925 0)
       (effects (font (size 1.27 1.27)) (justify left top) hide)
     )
@@
     )
   )
-  (symbol (lib_id "power:PWR_FLAG") (at 138.43 27.305 270) (unit 1)
-    (in_bom yes) (on_board yes) (dnp no) (fields_autoplaced)
-    (property "Reference" "#FLG03" (at 140.335 27.305 0)
-      (effects (font (size 1.27 1.27)) hide)
-    )
-    (property "Value" "PWR_FLAG" (at 141.605 27.94 90)
-      (effects (font (size 1.27 1.27)) (justify left))
-    )
-    (property "Footprint" "" (at 138.43 27.305 0)
-      (effects (font (size 1.27 1.27)) hide)
-    )
-    (property "Datasheet" "~" (at 138.43 27.305 0)
-      (effects (font (size 1.27 1.27)) hide)
-    )
-    (pin "1")
-    (instances
-      (project "LeaderSOM"
-        (path "/192d0c36-944e-4927-949b-263b8c85a7ca"
-          (reference "#FLG03") (unit 1)
-        )
-      )
-    )
-  )
   (symbol (lib_id "power:GNDA") (at 246.38 120.65 0) (unit 1)
     (in_bom yes) (on_board yes) (dnp no)
@@
         )
       )
+    )
+  )
+  (symbol (lib_id "power:+3.3VA") (at 138.43 26.035 0) (unit 1)
+    (in_bom yes) (on_board yes) (dnp no) (fields_autoplaced)
+    (property "Reference" "#PWR052" (at 138.43 29.845 0)
+      (effects (font (size 1.27 1.27)) hide)
+    )
+    (property "Value" "+3.3VA" (at 138.43 21.59 0)
+      (effects (font (size 1.27 1.27)))
+    )
+    (property "Footprint" "" (at 138.43 26.035 0)
+      (effects (font (size 1.27 1.27)) hide)
+    )
+    (property "Datasheet" "" (at 138.43 26.035 0)
+      (effects (font (size 1.27 1.27)) hide)
+    )
+    (pin "1")
+    (instances
+      (project "LeaderSOM"
+        (path "/192d0c36-944e-4927-949b-263b8c85a7ca/07cef2e6-f2f4-4f04-bcaf-7b98b53ab0fe"
+          (reference "#PWR052") (unit 1)
+        )
+        (path "/192d0c36-944e-4927-949b-263b8c85a7ca"
+          (reference "#PWR050") (unit 1)
+        )
+      )

Commit message: f is for friends that do stuff together
Parts:
- added H1, H2: M.3, MountingHole:MountingHole_3mm, symbol Mechanical:MountingHole
Changed lines of the file:
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@@
+    )
+  )
+  (symbol (lib_id "Mechanical:MountingHole") (at 271.145 146.05 0) (unit 1)
+    (in_bom yes) (on_board yes) (dnp no) (fields_autoplaced)
+    (property "Reference" "H2" (at 274.32 144.78 0)
+      (effects (font (size 1.27 1.27)) (justify left))
+    )
+    (property "Value" "M.3" (at 274.32 147.32 0)
+      (effects (font (size 1.27 1.27)) (justify left))
+    )
+    (property "Footprint" "MountingHole:MountingHole_3mm" (at 271.145 146.05 0)
+      (effects (font (size 1.27 1.27)) hide)
+    )
+    (property "Datasheet" "~" (at 271.145 146.05 0)
+      (effects (font (size 1.27 1.27)) hide)
+    )
+    (instances
+      (project "LeaderSOM"
+        (path "/192d0c36-944e-4927-949b-263b8c85a7ca"
+          (reference "H2") (unit 1)
+        )
+      )
     )
   )
@@
         )
       )
+    )
+  )
+  (symbol (lib_id "Mechanical:MountingHole") (at 271.145 139.7 0) (unit 1)
+    (in_bom yes) (on_board yes) (dnp no) (fields_autoplaced)
+    (property "Reference" "H1" (at 274.32 138.43 0)
+      (effects (font (size 1.27 1.27)) (justify left))
+    )
+    (property "Value" "M.3" (at 274.32 140.97 0)
+      (effects (font (size 1.27 1.27)) (justify left))
+    )
+    (property "Footprint" "MountingHole:MountingHole_3mm" (at 271.145 139.7 0)
+      (effects (font (size 1.27 1.27)) hide)
+    )
+    (property "Datasheet" "~" (at 271.145 139.7 0)
+      (effects (font (size 1.27 1.27)) hide)
+    )
+    (instances
+      (project "LeaderSOM"
+        (path "/192d0c36-944e-4927-949b-263b8c85a7ca"
+          (reference "H1") (unit 1)
+        )
+      )

Commit message: u is for u n me
Changed lines of the file:
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@@
-    (effects (font (size 1.27 1.27)) (justify right bottom))
-  )
-  (label "SPI1_MOSI" (at 63.5 97.155 180) (fields_autoplaced)
     (effects (font (size 1.27 1.27)) (justify right bottom))
   )
   (label "SPI2_CS{slash}TIM1_CH4{slash}GPIO" (at 272.415 43.815 180) (fields_autoplaced)
-    (effects (font (size 1.27 1.27)) (justify right bottom))
-  )
-  (label "SPI1_MISO" (at 63.5 103.505 180) (fields_autoplaced)
     (effects (font (size 1.27 1.27)) (justify right bottom))
   )
@@
     (effects (font (size 1.27 1.27)) (justify left bottom))
   )
+  (label "SPI1_MISO" (at 63.5 97.155 180) (fields_autoplaced)
+    (effects (font (size 1.27 1.27)) (justify right bottom))
+  )
   (label "SPI2_CS{slash}TIM1_CH4{slash}GPIO" (at 176.53 61.595 180) (fields_autoplaced)
     (effects (font (size 1.27 1.27)) (justify right bottom))
@@
     (effects (font (size 1.27 1.27)) (justify right bottom))
   )
+  (label "SPI1_MOSI" (at 63.5 103.505 180) (fields_autoplaced)
+    (effects (font (size 1.27 1.27)) (justify right bottom))
+  )

Commit message: n is for anywhere and anytime at all
Connections:
- net DISP1: now also U6.29 (PB10); no longer U6.24 (PC4)
- net DISP2: now also U6.27 (PB1); no longer U6.25 (PC5)
- net DISP3: now also U6.35 (PB14); no longer U6.26 (PB0)
- net DISP4: now also U6.28 (PB2); no longer U6.27 (PB1)
- net DISP5: now also U6.26 (PB0); no longer U6.28 (PB2)
- net DISP6: now also U6.25 (PC5); no longer U6.29 (PB10)
- net DISP7: now also U6.24 (PC4); no longer U6.35 (PB14)
Changed lines of the file:
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@@
     (effects (font (size 1.27 1.27)) (justify right bottom))
   )
-  (label "DISP4" (at 171.45 79.375 180) (fields_autoplaced)
+  (label "DISP2" (at 171.45 79.375 180) (fields_autoplaced)
     (effects (font (size 1.27 1.27)) (justify right bottom))
   )
@@
     (effects (font (size 1.27 1.27)) (justify left bottom))
   )
-  (label "DISP6" (at 171.45 102.235 180) (fields_autoplaced)
+  (label "DISP1" (at 171.45 102.235 180) (fields_autoplaced)
     (effects (font (size 1.27 1.27)) (justify right bottom))
   )
@@
     (effects (font (size 1.27 1.27)) (justify right bottom))
   )
-  (label "DISP2" (at 95.885 69.215 0) (fields_autoplaced)
+  (label "DISP6" (at 95.885 69.215 0) (fields_autoplaced)
     (effects (font (size 1.27 1.27)) (justify left bottom))
   )
-  (label "DISP7" (at 171.45 109.855 180) (fields_autoplaced)
+  (label "DISP3" (at 171.45 109.855 180) (fields_autoplaced)
     (effects (font (size 1.27 1.27)) (justify right bottom))
   )
@@
     (effects (font (size 1.27 1.27)) (justify right bottom))
   )
-  (label "DISP1" (at 95.885 66.675 0) (fields_autoplaced)
+  (label "DISP7" (at 95.885 66.675 0) (fields_autoplaced)
     (effects (font (size 1.27 1.27)) (justify left bottom))
   )
@@
     (effects (font (size 1.27 1.27)) (justify right bottom))
   )
-  (label "DISP5" (at 171.45 81.915 180) (fields_autoplaced)
+  (label "DISP4" (at 171.45 81.915 180) (fields_autoplaced)
     (effects (font (size 1.27 1.27)) (justify right bottom))
   )
@@
     (effects (font (size 1.27 1.27)) (justify right bottom))
   )
-  (label "DISP3" (at 171.45 76.835 180) (fields_autoplaced)
+  (label "DISP5" (at 171.45 76.835 180) (fields_autoplaced)
     (effects (font (size 1.27 1.27)) (justify right bottom))
   )
