File: LeaderSOM.kicad_sch (KiCad schematic)
At the start: 33 parts, among them IC2 TPS1120DR, J1 SWD, J3 52465-2470, J5 52465-2470, SW1 Reset, SW2 BTN1, U6 STM32F413RHTx, Y1 8M

Commit message: Updated symbols
Parts:
- IC2: footprint UTSVT_ICs:SOIC127P600X175-8N -> SOIC127P600X175-8N
Changed lines of the file:
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@@
 			)
 		)
-		(property "Description" ""
+		(property "Description" "Power symbol creates a global label with name \"GNDA\" , analog ground"
 			(at 221.615 82.55 0)
 			(effects
@@
 			)
 		)
-		(property "Description" ""
+		(property "Description" "Power symbol creates a global label with name \"GND\" , ground"
 			(at 74.93 70.485 0)
 			(effects
@@
 			)
 		)
-		(property "Description" ""
+		(property "Description" "Power symbol creates a global label with name \"GND\" , ground"
 			(at 222.25 92.71 0)
 			(effects
@@
 			)
 		)
-		(property "Description" ""
+		(property "Description" "Resistor"
 			(at 44.45 169.545 0)
 			(effects
@@
 			)
 		)
-		(property "Description" ""
+		(property "Description" "Unpolarized capacitor"
 			(at 232.41 117.475 0)
 			(effects
@@
 			)
 		)
-		(property "Description" ""
+		(property "Description" "Resistor"
 			(at 154.305 51.435 0)
 			(effects
@@
 			)
 		)
-		(property "Description" ""
+		(property "Description" "Unpolarized capacitor"
 			(at 80.01 65.405 0)
 			(effects
@@
 			)
 		)
-		(property "Description" ""
+		(property "Description" "Power symbol creates a global label with name \"GND\" , ground"
 			(at 248.92 92.71 0)
 			(effects
@@
 			)
 		)
-		(property "Description" ""
+		(property "Description" "Resistor"
 			(at 154.305 46.355 0)
 			(effects
@@
 			)
 		)
-		(property "Description" ""
+		(property "Description" "Resistor"
 			(at 100.33 167.64 0)
 			(effects
@@
 			)
 		)
-		(property "Description" ""
+		(property "Description" "Graph footprint placeholder"
 			(at 187.325 173.99 0)
 			(effects
@@
 			)
 		)
-		(property "Description" ""
+		(property "Description" "Power symbol creates a global label with name \"+3.3V\""
 			(at 147.955 165.1 0)
 			(effects
@@
 			)
 		)
-		(property "Description" ""
+		(property "Description" "Resistor"
 			(at 100.33 175.26 0)
 			(effects
@@
 			)
 		)
-		(property "Description" ""
+		(property "Description" "Power symbol creates a global label with name \"+3.3V\""
 			(at 196.85 111.125 0)
 			(effects
@@
 			)
 		)
-		(property "Description" ""
+		(property "Description" "Power symbol creates a global label with name \"+3.3V\""
 			(at 222.25 67.31 0)
 			(effects
@@
 			)
 		)
-		(property "Description" ""
+		(property "Description" "STMicroelectronics Arm Cortex-M4 MCU, 1536KB flash, 320KB RAM, 100 MHz, 1.7-3.6V, 50 GPIO, LQFP64"
 			(at 130.81 74.295 0)
 			(effects
@@
 			)
 		)
-		(property "Description" ""
+		(property "Description" "Power symbol creates a global label with name \"+3.3V\""
 			(at 248.92 67.31 0)
 			(effects
@@
 			)
 		)
-		(property "Datasheet" "https://www.mouser.com/datasheet/2/3/abm3-1774854.pdf"
+		(property "Datasheet" "~"
 			(at 74.93 56.515 0)
 			(effects
@@
 			)
 		)
-		(property "Description" ""
+		(property "Description" "Two pin crystal"
 			(at 74.93 56.515 0)
 			(effects
@@
 			)
 		)
-		(property "Description" ""
+		(property "Description" "Graph footprint placeholder"
 			(at 218.44 173.99 0)
 			(effects
@@
 			)
 		)
-		(property "Description" ""
+		(property "Description" "Unpolarized capacitor"
 			(at 208.28 117.475 0)
 			(effects
@@
 			)
 		)
-		(property "Description" ""
+		(property "Description" "Unpolarized capacitor"
 			(at 69.85 65.405 0)
 			(effects
@@
 			)
 		)
-		(property "Description" ""
+		(property "Description" "Power symbol creates a global label with name \"+3.3VA\""
 			(at 246.38 111.125 0)
 			(effects
@@
 			)
 		)
-		(property "Description" ""
+		(property "Description" "Power symbol creates a global label with name \"+3.3V\""
 			(at 222.25 51.435 0)
 			(effects
@@
 			)
 		)
-		(property "Description" ""
+		(property "Description" "Mounting Hole without connection"
 			(at 271.145 146.685 0)
 			(effects
@@
 			)
 		)
-		(property "Description" ""
+		(property "Description" "Resistor"
 			(at 144.145 171.45 0)
 			(effects
@@
 			)
 		)
-		(property "Description" ""
+		(property "Description" "Unpolarized capacitor"
 			(at 196.85 117.475 0)
 			(effects
@@
 			)
 		)
-		(property "Description" ""
+		(property "Description" "Power symbol creates a global label with name \"GND\" , ground"
 			(at 248.92 82.55 0)
 			(effects
@@
 			)
 		)
-		(property "Description" ""
+		(property "Description" "Power symbol creates a global label with name \"+3.3V\""
 			(at 54.61 163.195 0)
 			(effects
@@
 			)
 		)
-		(property "Description" ""
+		(property "Description" "Unpolarized capacitor"
 			(at 261.62 117.475 0)
 			(effects
@@
 			)
 		)
-		(property "Description" ""
+		(property "Description" "Mounting Hole without connection"
 			(at 271.145 158.115 0)
 			(effects
@@
 			)
 		)
-		(property "Description" ""
+		(property "Description" "Unpolarized capacitor"
 			(at 219.71 117.475 0)
 			(effects
@@
 			)
 		)
-		(property "Description" ""
+		(property "Description" "Unpolarized capacitor"
 			(at 187.96 146.685 0)
 			(effects
@@
 			)
 		)
-		(property "Description" ""
+		(property "Description" "Generic connector, single row, 01x04, script generated (kicad-library-utils/schlib/autogen/connector/)"
 			(at 252.73 145.415 0)
 			(effects
@@
 			)
 		)
-		(property "Description" ""
+		(property "Description" "Power symbol creates a global label with name \"GND\" , ground"
 			(at 243.84 153.67 0)
 			(effects
@@
 			)
 		)
-		(property "Description" ""
+		(property "Description" "Power symbol creates a global label with name \"GND\" , ground"
 			(at 196.85 122.555 0)
 			(effects
@@
 			)
 		)
-		(property "Footprint" "UTSVT_ICs:SOIC127P600X175-8N"
+		(property "Footprint" "SOIC127P600X175-8N"
 			(at 90.805 262.56 0)
 			(effects
@@
 			)
 		)
-		(property "Description" ""
+		(property "Description" "Dual P-channel Enhancemenent-Mode MOSFET"
 			(at 56.515 167.64 0)
 			(effects
@@
 			)
 		)
-		(property "Description" ""
+		(property "Description" "Power symbol creates a global label with name \"GNDA\" , analog ground"
 			(at 141.605 129.54 0)
 			(effects
@@
 			)
 		)
-		(property "Description" ""
+		(property "Description" "Mounting Hole without connection"
 			(at 271.145 152.4 0)
 			(effects
@@
 			)
 		)
-		(property "Description" ""
+		(property "Description" "Power symbol creates a global label with name \"GND\" , ground"
 			(at 101.6 38.735 0)
 			(effects
@@
 			)
 		)
-		(property "Description" ""
+		(property "Description" "Mounting Hole without connection"
 			(at 271.145 140.97 0)
 			(effects
@@
 			)
 		)
-		(property "Description" ""
+		(property "Description" "Unpolarized capacitor"
 			(at 215.9 146.05 0)
 			(effects
@@
 			)
 		)
-		(property "Description" ""
+		(property "Description" "Power symbol creates a global label with name \"GND\" , ground"
 			(at 222.25 41.275 0)
 			(effects
@@
 			)
 		)
-		(property "Description" ""
+		(property "Description" "Resistor"
 			(at 49.53 175.26 0)
 			(effects
@@
 			)
 		)
-		(property "Description" ""
+		(property "Description" "Resistor"
 			(at 151.765 171.45 0)
 			(effects
@@
 			)
 		)
-		(property "Description" ""
+		(property "Description" "Push button switch, generic, two pins"
 			(at 227.33 146.05 0)
 			(effects
@@
 			)
 		)
-		(property "Description" ""
+		(property "Description" "Unpolarized capacitor, small symbol"
 			(at 107.315 113.665 0)
 			(effects
@@
 			)
 		)
-		(property "Description" ""
+		(property "Description" "Push button switch, generic, two pins"
 			(at 199.39 146.685 0)
 			(effects
@@
 			)
 		)
-		(property "Description" ""
+		(property "Description" "Unpolarized capacitor"
 			(at 246.38 117.475 0)
 			(effects
@@
 			)
 		)
-		(property "Description" ""
+		(property "Description" "Power symbol creates a global label with name \"+3.3V\""
 			(at 248.92 51.435 0)
 			(effects
@@
 			)
 		)
-		(property "Description" ""
+		(property "Description" "Power symbol creates a global label with name \"GNDA\" , analog ground"
 			(at 246.38 122.555 0)
 			(effects
@@
 			)
 		)
-		(property "Description" ""
+		(property "Description" "Power symbol creates a global label with name \"+3.3VA\""
 			(at 138.43 26.035 0)
 			(effects
@@
 			)
 		)
-		(property "Description" ""
+		(property "Description" "Power symbol creates a global label with name \"GND\" , ground"
 			(at 248.92 41.275 0)
 			(effects
@@
 			)
 		)
-		(property "Description" ""
+		(property "Description" "Power symbol creates a global label with name \"GND\" , ground"
 			(at 187.96 154.305 0)
 			(effects
@@
 			)
 		)
-		(property "Description" ""
+		(property "Description" "Power symbol creates a global label with name \"+3.3V\""
 			(at 243.84 142.875 0)
 			(effects
@@
 			)
 		)
-		(property "Description" ""
+		(property "Description" "Power symbol creates a global label with name \"GND\" , ground"
 			(at 123.19 129.54 0)
 			(effects
@@
 			)
 		)
-		(property "Description" ""
+		(property "Description" "Power symbol creates a global label with name \"+3.3VA\""
 			(at 221.615 77.47 0)
 			(effects
@@
 			)
 		)
-		(property "Description" ""
+		(property "Description" "Power symbol creates a global label with name \"GND\" , ground"
 			(at 215.9 153.67 0)
 			(effects
@@
 			)
 		)
-		(property "Description" ""
+		(property "Description" "Power symbol creates a global label with name \"+3.3V\""
 			(at 130.81 22.86 0)
 			(effects

Commit message: laid things out but still need to fix things :(
Parts:
- removed R11, R13: 49.9, Resistor_SMD:R_0805_2012Metric, symbol Device:R
- added D7: LED, LED_SMD:LED_0805_2012Metric, symbol Device:LED
- added R6: 2.2k, Resistor_SMD:R_0805_2012Metric, symbol Device:R
Connections:
- net +V_CarCAN is gone; now on net UART5_RX/GPIO: J3.19
- net -V_CarCAN is gone; now on net GND: J3.13
- net ADC1_IN10/GPIO: now also J5.7; no longer J5.19
- net ADC1_IN2/USART2_TX/GPIO: now also J5.18; no longer J5.20
- net ADC1_IN3/USART2_RX/GPIO: now also J5.20; no longer J5.18
- net CarCAN_H: now also J5.6; no longer J3.17
- net CarCAN_L: now also J5.8; no longer J3.15
- net GND: now also J1.3 (Pin_3), J3.15, J5.14, J5.16, J5.5, D7.1 (K); no longer J1.4 (Pin_4), J3.11, J3.9, J5.10, J5.12
- net GNDA: now also J5.10, J5.12
- net I2C1_SCL: now also J3.7; no longer J3.8
- net I2C1_SDA: now also J3.5; no longer J3.6
- net I2C3_SCL/TIM1_CH1/GPIO: now also J3.11; no longer J3.7
- net I2C3_SDA/GPIO: now also J3.9; no longer J3.5
- net IntCAN_H: now also J3.6; no longer J5.8
- net IntCAN_L: now also J3.8; no longer J5.6
- net SPI1_MOSI: now also U6.23 (PA7)
- net SPI1_SCK: now also U6.21 (PA5)
- net SWDIO: now also J1.4 (Pin_4); no longer J1.3 (Pin_3)
- net UART5_RX/GPIO: no longer J5.16
- net UART5_TX/GPIO: now also J3.17; no longer J5.14
- net ADC_IN12/GPIO renamed ADC1_IN12/GPIO
- net ADC1_IN12/GPIO: now also J5.19; no longer J5.7
- net ADC_IN13/GPIO renamed LED
- net LED: now also R6.1; no longer J5.5
- new net: D7.2 (A), R6.2
Other:
- sheet CarCAN ports: added none; removed +V_CarCAN, -V_CarCAN
- moved on the sheet: C23, C24, C26, C27, C28, C30, IC2, J1, R17, R18, R19, R20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

Commit message: changed cap on osc
Parts:
- C4, C5: value 12p -> 26p
Changed lines of the file:
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@@
 			)
 		)
-		(property "Value" "12p"
+		(property "Value" "26p"
 			(at 82.931 66.548 0)
 			(effects
@@
 			)
 		)
-		(property "Value" "12p"
+		(property "Value" "26p"
 			(at 72.771 66.548 0)
 			(effects

Commit message: fixed can stuff
Parts:
- renumbered SW2 to BTN1, SW1 to Reset1, J1 to SWD1
Changed lines of the file:
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@@
 		(dnp no)
 		(fields_autoplaced yes)
-		(property "Reference" "J1"
-			(at 260.35 146.05 0)
+		(property "Reference" "SWD1"
+			(at 260.35 145.4149 0)
 			(effects
 				(font
@@
 		)
 		(property "Value" "SWD"
-			(at 260.35 148.59 0)
+			(at 260.35 147.9549 0)
 			(effects
 				(font
@@
 			(project "LeaderSOM"
 				(path "/192d0c36-944e-4927-949b-263b8c85a7ca"
-					(reference "J1")
+					(reference "SWD1")
 					(unit 1)
 				)
@@
 		(on_board yes)
 		(dnp no)
-		(property "Reference" "SW1"
+		(property "Reference" "Reset1"
 			(at 231.0892 144.8816 90)
 			(effects
@@
 			(project "LeaderSOM"
 				(path "/192d0c36-944e-4927-949b-263b8c85a7ca"
-					(reference "SW1")
+					(reference "Reset1")
 					(unit 1)
 				)
@@
 		(on_board yes)
 		(dnp no)
-		(property "Reference" "SW2"
+		(property "Reference" "BTN1"
 			(at 203.1492 145.5166 90)
 			(effects
@@
 			(project "LeaderSOM"
 				(path "/192d0c36-944e-4927-949b-263b8c85a7ca"
-					(reference "SW2")
-					(unit 1)
-				)
+					(reference "BTN1")
+					(unit 1)
+				)

Commit message: hi again lakshay
Parts:
- added R38: 10k, Resistor_SMD:R_0805_2012Metric, symbol Device:R
- H1, H2, H3, H4: footprint MountingHole:MountingHole_3mm -> MountingHole:MountingHole_3.2mm_M3
Connections:
- net GND: now also R38.1; no longer U6.60 (BOOT0)
- new net: R38.2, U6.60 (BOOT0)
Other:
- sheet USB ports: added CHIP_RX, CHIP_TX; removed UART_RX, UART_TX
- moved on the sheet: BTN1, C15, C17, C23, C24, C26, C27, C28, C29, C30, C4, C5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

Commit message: starting redesign
Parts:
- removed U6: STM32F413RHTx, Package_QFP:LQFP-64_10x10mm_P0.5mm, symbol MCU_ST_STM32F4:STM32F413RHTx
- added U? (x2): STM32G473RET6, LQFP64-10x10mm, symbol STM32G473RET6:STM32G473RET6
- IC2: footprint SOIC127P600X175-8N -> UTSVT_ICs:SOIC127P600X175-8N
Connections:
- net BTN1: now also U?.60 (PB7)
- net I2C3_PU_En: now also U?.59 (PB6)
- net LED: now also U?.62 (PB9)
- net NRST: now also U?.55 (PD2)
- net OSC_IN: now also U?.3 (PC14-OSC32_IN)
- net OSC_OUT: now also U?.4 (PC15-OSC32_OUT)
- net SDC_DET: now also U?.26 (PB2)
- net SPI1_CS: now also U?.18 (PA4)
- net SPI1_MISO: now also U?.20 (PA6)
- net SPI1_MOSI: now also U?.21 (PA7)
- net SPI1_SCK: now also U?.19 (PA5)
- net SWCLK: now also U?.50 (PA14)
- net SWDIO: now also U?.49 (PA13)
- new net BOOT: U?.61 (PB8-BOOT0)
- new net USB_UART1_RX: U?.23 (PC5)
- new net USB_UART1_TX: U?.22 (PC4)
Other:
- sheet Display ports: added Output Clock, Output Enable, SR Clock, Serial Input; removed LED[1..14]
- moved on the sheet: C4, C5, R38, Y1

Commit message: MCU pins, PSON power distribution, KiCad-Sharepoint, and 7 seg
Parts:
- removed C17: 4.7u, Capacitor_SMD:C_0805_2012Metric, symbol Device:C_Small
- removed R38: 10k, Resistor_SMD:R_0805_2012Metric, symbol Device:R
- added C14: 100nF, Capacitor_SMD:C_0805_2012Metric, symbol Device:C
- added FB4: FerriteBead, Inductor_SMD:L_0805_2012Metric, symbol Device:FerriteBead
- added NT1: NetTie_2, NetTie:NetTie-2_SMD_Pad0.5mm, symbol Device:NetTie_2
- added SW1: SW_SPDT, symbol Switch:SW_SPDT
- IC2: footprint UTSVT_ICs:SOIC127P600X175-8N -> UTSVT_ICs:TPS1120DR; symbol utsvt-chips:TPS1120DR -> UTSVT-ICs:TPS1120DR
- J3, J5: symbol utsvt-connectors:52465-2470 -> UTSVT-Connectors:52465-2470
- gave numbers to parts that had none: 1
Connections:
- net ADC1_IN10/GPIO is gone; now on net ADC1_IN3/TIM2_CH3/GPIO: J5.7
- net ADC1_IN11/GPIO is gone; now on net ADC1_IN12/TIM1_CH3N/GPIO: J5.17
- net ADC1_IN12/GPIO is gone; now on net ADC1_IN15/TIM1_CH2N/GPIO: J5.19
- net SPI2_CS/TIM1_CH4/GPIO is gone; now on net SPI3_NSS/FDCAN3_TX/GPIO: J3.16
- net SPI2_MISO/GPIO is gone; now on net SPI3_MISO/TIM3_CH1/GPIO: J3.14
- net SPI2_MOSI/TIM1_CH3/GPIO is gone; now on net SPI3_MOSI/TIM3_CH2/GPIO: J3.18
- net SPI2_SCK/TIM1_CH2/GPIO is gone; now on net SPI3_SCK/TIM2_CH2/GPIO: J3.20
- net UART5_TX/GPIO is gone; now on net UART5_TX/TIM5_CH2/GPIO: J3.17
- net +3.3V: now also U1.1 (VBAT), U1.16 (VDD), U1.32 (VDD), U1.48 (VDD), U1.64 (VDD), FB4.1, SW1.1 (A)
- net +3.3VA: now also U1.28 (VREF+), U1.29 (VDDA), C14.1, FB4.2
- net ADC1_IN2/USART2_TX/GPIO: now also U1.36 (PB14)
- net ADC1_IN3/USART2_RX/GPIO: now also U1.26 (PB2)
- net BOOT: now also SW1.2 (B)
- net CarCAN_H: now also J5.8; no longer J5.6
- net CarCAN_L: now also J5.6; no longer J5.8
- net DISP1: now also U1.8 (PC0)
- net DISP2: now also U1.9 (PC1)
- net DISP3: now also U1.10 (PC2)
- net GND: now also U1.15 (VSS), U1.31 (VSS), U1.47 (VSS), U1.63 (VSS), NT1.1, SW1.3 (C); no longer J3.10, J3.12, J3.13, J3.15, J5.14, J5.16, J5.5
- net GNDA: now also J5.14, J5.16, U1.27 (VSSA), C14.2, NT1.2; no longer J5.10, J5.11, J5.12, J5.9
- net I2C3_SCL/TIM1_CH1/GPIO: no longer J3.11
- net I2C3_SDA/GPIO: no longer J3.9
- net IntCAN_H: now also J3.8; no longer J3.6
- net IntCAN_L: now also J3.6; no longer J3.8
- net LED: no longer R6.1
- net NRST: now also U1.7 (PG10-NRST); no longer U1.55 (PD2)
- net SDC_DET: now also U1.37 (PB15); no longer U1.26 (PB2)
- net UART5_RX/GPIO: now also U1.55 (PD2)
- net IMON: now reaches U1.11 (PC3)
- net ADC1_IN1/TIM2_CH1/GPIO: now reaches U1.12 (PA0)
- net ADC1_IN1/TIM2_CH1/GPIO: now also J5.11
- net ADC1_IN2/TIM2_CH2/GPIO: now reaches U1.13 (PA1)
- net ADC1_IN2/TIM2_CH2/GPIO: now also J5.9
- net ADC1_IN3/TIM2_CH3/GPIO: now reaches U1.14 (PA2)
- net OP5_VINM/ADC1_IN4/TIM2_CH4: now reaches U1.17 (PA3)
- net OP5_VINM/ADC1_IN4/TIM2_CH4: now also J5.5
- net ADC1_IN15/TIM1_CH2N/GPIO: now reaches U1.24 (PB0)
- net ADC1_IN12/TIM1_CH3N/GPIO: now reaches U1.25 (PB1)
- net USART3_TX/TIM1_BKIN/GPIO: now reaches U1.30 (PB10)
- net USART3_TX/TIM1_BKIN/GPIO: now also J5.12
- net USART3_RX/ADC1_IN14/GPIO: now reaches U1.33 (PB11)
- net USART3_RX/ADC1_IN14/GPIO: now also J5.10
- net FDCAN2_RX: now reaches U1.34 (PB12)
- net FDCAN2_TX: now reaches U1.35 (PB13)
- net I2C4_SCL/TIM3_CH1/GPIO: now reaches U1.38 (PC6)
- net I2C4_SDA/TIM3_CH2/GPIO: now reaches U1.39 (PC7)
- net I2C3_SCL/TIM3_CH3/GPIO: now reaches U1.40 (PC8)
- net I2C3_SCL/TIM3_CH3/GPIO: now also J3.11
- net I2C3_SDA/TIM3_CH4/GPIO: now reaches U1.41 (PC9)
- net I2C3_SDA/TIM3_CH4/GPIO: now also J3.9
- net OP5_VOUT/CAN3_RX/TIM1_CH1: now reaches U1.42 (PA8)
- net OP5_VOUT/CAN3_RX/TIM1_CH1: now also J3.12
- net ADC5_IN2/TIM1_CH2/GPIO: now reaches U1.43 (PA9)
- net ADC5_IN2/TIM1_CH2/GPIO: now also J3.10
- net LED1: now reaches U1.44 (PA10)
- net LED1: now also R6.1
- net FDCAN3_RX: now reaches U1.45 (PA11)
- net FDCAN3_TX: now reaches U1.46 (PA12)
- net SPI3_NSS/FDCAN3_TX/GPIO: now reaches U1.51 (PA15)
- net UART4_TX/TIM8_CH1N/GPIO: now reaches U1.52 (PC10)
- net UART4_TX/TIM8_CH1N/GPIO: now also J3.13
- net UART4_RX/TIM8_CH2N/GPIO: now reaches U1.53 (PC11)
- net UART4_RX/TIM8_CH2N/GPIO: now also J3.15
- net UART5_TX/TIM5_CH2/GPIO: now reaches U1.54 (PC12)
- net SPI3_SCK/TIM2_CH2/GPIO: now reaches U1.56 (PB3)
- net SPI3_MISO/TIM3_CH1/GPIO: now reaches U1.57 (PB4)
- net SPI3_MOSI/TIM3_CH2/GPIO: now reaches U1.58 (PB5)
- net 12V_Ext renamed +24V
- net I2C1_SCL renamed I2C4_SCL
- net I2C1_SDA renamed I2C4_SDA
- no-connect marks 4 -> 3
Other:
- sheet Display ports: added none; removed Output Enable
- sheet Power_Distribution ports: added IMON_OUT; removed 12V_In
- note added: "Buttons & Stuff"
- note added: "Bypass/Separation"
- note added: "Changelog: - Changed MCU to STM32G473RET6 - Changed most SOM connector pins slightly - Replaced redunant GND/GNDA pins with more data pins - Added extra functionality to some pins - Change pp values to be 24V - Swap out power stuff to match PSOM - 24v - 5v buck - 5v power mux - overvoltage/current values - 5v - 3v LDO - Connect IMON to MCU - Changed a couple circuits to look better - Workinmg on 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"
- note added: "VDDA Separation"
- moved on the sheet: C4, C5, D7, H1, H2, H3, H4, R6, SWD1, U1A, U1B, Y1

Commit message: net class fixes and ERC
Parts:
- removed IC2: TPS1120DR, UTSVT_ICs:TPS1120DR, symbol UTSVT-ICs:TPS1120DR
- removed R17: 100k, Resistor_SMD:R_0805_2012Metric, symbol Device:R
- removed R18: 1k, Resistor_SMD:R_0805_2012Metric, symbol Device:R
- removed R19, R20: 10K, Resistor_SMD:R_0805_2012Metric, symbol Device:R
- removed R4: 10k, Resistor_SMD:R_0805_2012Metric, symbol Device:R
- added D15: LED, LED_SMD:LED_0805_2012Metric, symbol Device:LED
- R7: value 10k -> 2.2k; Mouser Part Number (none) -> Inventory; P/N CRCW08054K70FKEA -> SDR10EZPF2200
- SW1: footprint (none) -> UTSVT_Special:SW_SPST_B3SL-1002P
- U1: footprint LQFP64-10x10mm -> STM32G473RET6:LQFP64-10x10mm
Connections:
- net I2C4_SCL is gone; now on net I2C4_SCL/TIM3_CH1/GPIO: J3.7
- net GND: now also D15.1 (K)
- net I2C4_SDA/TIM3_CH2/GPIO: now also J3.5
- net +24V renamed 24V_Ext
- net +3.3V renamed +3V3
- net +3V3: no longer R7.1
- net I2C3_PU_En: no longer names the net of U1.59 (PB6)
- net I2C4_SDA: no longer names the net of R7.2
- net I2C4_SDA: now also D15.2 (A); no longer J3.5
- net LED renamed LEDHB
- net LEDHB: now also R7.1
- no-connect marks 3 -> 4
Other:
- sheet Power_Distribution ports: added 24V_In; removed none
- note removed: "I2C Pullups"
- moved on the sheet: D7, R6
