File: LeaderSOM.kicad_sch (KiCad schematic)
At the start: 10 parts, among them J3 52465-2470, J5 52465-2470

Commit message: crazy? i used to be crazy
Parts:
- removed J? (x2): ~, symbol UTSVT-Connectors:LSOM_DaughterConn
- renumbered J3 to J1, J5 to J2
Other:
- removed sheet Display
- sheet LEDS & Buttons ports: added none; removed BOOT, BOOT_GPIO, NRST, SWCLK, SWDIO
- sheet MCU ports: added AddressableLED, IMON, {ADC}, {CAN}, {I2C}, {SPI}, {UART}, {USB}; removed none

Commit message: impending doom is approaching
Parts:
- H1, H2, H3, H4: footprint MountingHole:MountingHole_3.2mm_M3 -> MountingHole:MountingHole_3.2mm_M3_Pad_TopBottom
Changed lines of the file:
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@@
 			)
 		)
-		(property "Footprint" "MountingHole:MountingHole_3.2mm_M3"
+		(property "Footprint" "MountingHole:MountingHole_3.2mm_M3_Pad_TopBottom"
 			(at 235.585 175.895 0)
 			(effects
@@
 			)
 		)
-		(property "Footprint" "MountingHole:MountingHole_3.2mm_M3"
+		(property "Footprint" "MountingHole:MountingHole_3.2mm_M3_Pad_TopBottom"
 			(at 247.015 175.895 0)
 			(effects
@@
 			)
 		)
-		(property "Footprint" "MountingHole:MountingHole_3.2mm_M3"
+		(property "Footprint" "MountingHole:MountingHole_3.2mm_M3_Pad_TopBottom"
 			(at 247.015 170.18 0)
 			(effects
@@
 			)
 		)
-		(property "Footprint" "MountingHole:MountingHole_3.2mm_M3"
+		(property "Footprint" "MountingHole:MountingHole_3.2mm_M3_Pad_TopBottom"
 			(at 235.585 170.18 0)
 			(effects

Commit message: redid the traces
Changed lines of the file:
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@@
 		)
 	)
-	(label "FDCAN2_RX"
+	(label "FDCAN1_RX"
 		(at 70.485 40.64 0)
 		(effects
@@
 		)
 	)
-	(label "FDCAN2_TX"
+	(label "FDCAN1_TX"
 		(at 70.485 43.815 0)
 		(effects
@@
 		)
 	)
-	(label "FDCAN2_RX"
+	(label "FDCAN1_RX"
 		(at 61.976 47.371 180)
 		(effects
@@
 		)
 	)
-	(label "FDCAN2_TX"
+	(label "FDCAN1_TX"
 		(at 61.976 44.196 180)
 		(effects

Commit message: ripping my hair out
Connections:
- net CarCAN_H: now also J1.8; no longer J2.8
- net CarCAN_L: now also J1.6; no longer J2.6
- net IntCAN_H: now also J2.8; no longer J1.8
- net IntCAN_L: now also J2.6; no longer J1.6
- net SPI2_MISO/ADC1_IN5/TIM1_CH2N: now also J1.14; no longer J2.20
- net SPI2_MOSI/ADC2_IN15/TIM1_CH3N: now also J1.18; no longer J2.18
- net SPI2_NSS/TIM4_CH4/COMP2_OUT: now also J1.16; no longer J2.24
- net SPI2_SCK/OPAMP3_VINP/FDCAN2_TX: now also J1.20; no longer J2.22
- net SPI3_MISO/TIM3_CH1/USART2_RX: now also J2.18; no longer J1.14
- net SPI3_MOSI/TIM3_CH2/TIM17_CH1: now also J2.22; no longer J1.18
- net SPI3_NSS/TIM1_CH3/COMP6_OUT: now also J2.20; no longer J1.16
- net SPI3_SCK/TIM2_CH2/USART2_TX: now also J2.24; no longer J1.20
- net UART5_RX: no longer J1.19
- net UART5_TX/TIM5_CH2: no longer J1.17
- new net UART1_RX: J1.19
- new net UART1_TX: J1.17
Other:
- moved on the sheet: J1, J2

Commit message: nuke
Changed lines of the file:
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@@
 		)
 		(pin "CHIP_TX" output
-			(at 48.895 72.39 0)
+			(at 48.26 72.39 0)
 			(effects
 				(font
@@
 		)
 		(pin "CHIP_RX" input
-			(at 48.895 68.58 0)
+			(at 48.26 68.58 0)
 			(effects
 				(font

Commit message: 6:21:27 split
Connections:
- net ADC1_IN11/COMP7_INM/FDCAN2_RX: now also J1.12; no longer J2.16
- net ADC1_IN12/TIM1_CH3N/COMP1_INP: now also J2.7; no longer J2.21
- net ADC1_IN15/TIM1_CH2N/COMP4_INP: now also J2.9; no longer J2.19
- net ADC1_IN1/TIM2_CH1/COMP1_OUT: now also J2.19; no longer J2.15
- net ADC1_IN2/TIM2_CH2/COMP1_INP: now also J2.17; no longer J2.11
- net ADC1_IN3/TIM2_CH3/COMP2_INM: now also J2.15; no longer J2.9
- net ADC1_IN6/TIM1_CH1/COMP3_INM: now also J2.23; no longer J1.12
- net ADC1_IN7/TIM1_CH2/COMP3_INP: now also J2.16; no longer J1.10
- net ADC1_IN8/TIM1_CH3/COMP3_OUT: now also J2.21; no longer J2.17
- net ADC2_IN12/TIM5_CH1/COMP4_INM: now also J1.10; no longer J2.23
- net OPAMP5_VINM/ADC1_IN4/TIM2_CH4: now also J2.11; no longer J2.7
- net UART4_RX/TIM8_CH2N: now also J2.12; no longer J1.15
- net UART4_TX/TIM8_CH1N: now also J2.10; no longer J1.13
- net USART3_RX/ADC1_IN14/TIM2_CH4: now also J1.15; no longer J2.10
- net USART3_TX/OPAMP3_VINM/TIM2_CH3: now also J1.13; no longer J2.12
Changed lines of the file:
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@@
 	(wire
 		(pts
-			(xy 185.42 111.76) (xy 218.44 111.76)
-		)
-		(stroke
-			(width 0)
-			(type default)
-		)
-	)
-	(wire
-		(pts
-			(xy 185.42 99.06) (xy 218.44 99.06)
-		)
-		(stroke
-			(width 0)
-			(type default)
-		)
-	)
-	(wire
-		(pts
-			(xy 185.42 109.22) (xy 218.44 109.22)
+			(xy 182.88 111.76) (xy 218.44 111.76)
+		)
+		(stroke
+			(width 0)
+			(type default)
+		)
+	)
+	(wire
+		(pts
+			(xy 182.88 99.06) (xy 218.44 99.06)
+		)
+		(stroke
+			(width 0)
+			(type default)
+		)
+	)
+	(wire
+		(pts
+			(xy 182.88 109.22) (xy 218.44 109.22)
 		)
 		(stroke
@@
 	(wire
 		(pts
-			(xy 185.42 96.52) (xy 218.44 96.52)
+			(xy 182.88 96.52) (xy 218.44 96.52)
 		)
 		(stroke
@@
 	(wire
 		(pts
-			(xy 185.42 93.98) (xy 218.44 93.98)
+			(xy 182.88 93.98) (xy 218.44 93.98)
 		)
 		(stroke
@@
 	(wire
 		(pts
-			(xy 185.42 104.14) (xy 218.44 104.14)
+			(xy 182.88 104.14) (xy 218.44 104.14)
 		)
 		(stroke
@@
 	(wire
 		(pts
-			(xy 185.42 106.68) (xy 218.44 106.68)
+			(xy 182.88 106.68) (xy 218.44 106.68)
 		)
 		(stroke
@@
 	(wire
 		(pts
-			(xy 185.42 101.6) (xy 218.44 101.6)
+			(xy 182.88 101.6) (xy 218.44 101.6)
 		)
 		(stroke
@@
 		)
 	)
-	(label "ADC1_IN3{slash}TIM2_CH3{slash}COMP2_INM"
-		(at 184.15 147.32 0)
-		(effects
-			(font
-				(size 1.27 1.27)
-			)
-			(justify left bottom)
+	(label "ADC1_IN7{slash}TIM1_CH2{slash}COMP3_INP"
+		(at 275.59 139.7 180)
+		(effects
+			(font
+				(size 1.27 1.27)
+			)
+			(justify right bottom)
 		)
 	)
@@
 		)
 	)
+	(label "UART1_TX"
+		(at 182.88 96.52 0)
+		(effects
+			(font
+				(size 1.27 1.27)
+			)
+			(justify left bottom)
+		)
+	)
 	(label "I2C4_SDA{slash}TIM3_CH2"
-		(at 185.42 111.76 0)
+		(at 182.88 111.76 0)
+		(effects
+			(font
+				(size 1.27 1.27)
+			)
+			(justify left bottom)
+		)
+	)
+	(label "ADC1_IN8{slash}TIM1_CH3{slash}COMP3_OUT"
+		(at 184.15 132.08 0)
 		(effects
 			(font
@@
 	)
 	(label "I2C3_SCL{slash}TIM3_CH3"
-		(at 185.42 104.14 0)
-		(effects
-			(font
-				(size 1.27 1.27)
-			)
-			(justify left bottom)
+		(at 182.88 104.14 0)
+		(effects
+			(font
+				(size 1.27 1.27)
+			)
+			(justify left bottom)
+		)
+	)
+	(label "UART4_TX{slash}TIM8_CH1N"
+		(at 275.59 147.32 180)
+		(effects
+			(font
+				(size 1.27 1.27)
+			)
+			(justify right bottom)
 		)
 	)
@@
 		)
 	)
+	(label "UART1_RX"
+		(at 182.88 93.98 0)
+		(effects
+			(font
+				(size 1.27 1.27)
+			)
+			(justify left bottom)
+		)
+	)
 	(label "ADC1_IN7{slash}TIM1_CH2{slash}COMP3_INP"
 		(at 162.052 58.166 180)
@@
 		)
 	)
+	(label "ADC1_IN6{slash}TIM1_CH1{slash}COMP3_INM"
+		(at 184.15 129.54 0)
+		(effects
+			(font
+				(size 1.27 1.27)
+			)
+			(justify left bottom)
+		)
+	)
 	(label "SPI2_NSS{slash}TIM4_CH4{slash}COMP2_OUT"
 		(at 163.83 105.664 180)
@@
 		)
 	)
+	(label "USART3_TX{slash}OPAMP3_VINM{slash}TIM2_CH3"
+		(at 182.88 101.6 0)
+		(effects
+			(font
+				(size 1.27 1.27)
+			)
+			(justify left bottom)
+		)
+	)
 	(label "SPI3_SCK{slash}TIM2_CH2{slash}USART2_TX"
 		(at 275.59 129.54 180)
@@
 		)
 	)
-	(label "ADC1_IN2{slash}TIM2_CH2{slash}COMP1_INP"
-		(at 184.15 144.78 0)
-		(effects
-			(font
-				(size 1.27 1.27)
-			)
-			(justify left bottom)
-		)
-	)
 	(label "CarCAN_L"
 		(at 61.976 56.261 180)
@@
 		)
 	)
-	(label "ADC2_IN12{slash}TIM5_CH1{slash}COMP4_INM"
-		(at 184.15 129.54 0)
-		(effects
-			(font
-				(size 1.27 1.27)
-			)
-			(justify left bottom)
-		)
-	)
 	(label "UART1_TX"
 		(at 163.83 119.38 180)
@@
 		)
 	)
-	(label "ADC1_IN15{slash}TIM1_CH2N{slash}COMP4_INP"
-		(at 184.15 134.62 0)
-		(effects
-			(font
-				(size 1.27 1.27)
-			)
-			(justify left bottom)
-		)
-	)
 	(label "IMON"
 		(at 74.93 110.49 0)
@@
 		)
 	)
-	(label "ADC1_IN6{slash}TIM1_CH1{slash}COMP3_INM"
-		(at 275.59 104.14 180)
+	(label "ADC2_IN12{slash}TIM5_CH1{slash}COMP4_INM"
+		(at 275.59 106.68 180)
 		(effects
 			(font
@@
 		)
 	)
+	(label "ADC1_IN3{slash}TIM2_CH3{slash}COMP2_INM"
+		(at 184.15 139.7 0)
+		(effects
+			(font
+				(size 1.27 1.27)
+			)
+			(justify left bottom)
+		)
+	)
 	(label "FDCAN3_RX"
 		(at 71.12 48.26 0)
@@
 		)
 	)
-	(label "USART3_RX{slash}ADC1_IN14{slash}TIM2_CH4"
-		(at 275.59 147.32 180)
-		(effects
-			(font
-				(size 1.27 1.27)
-			)
-			(justify right bottom)
+	(label "ADC1_IN15{slash}TIM1_CH2N{slash}COMP4_INP"
+		(at 184.15 147.32 0)
+		(effects
+			(font
+				(size 1.27 1.27)
+			)
+			(justify left bottom)
 		)
 	)
@@
 		)
 	)
+	(label "OPAMP5_VINM{slash}ADC1_IN4{slash}TIM2_CH4"
+		(at 184.15 144.78 0)
+		(effects
+			(font
+				(size 1.27 1.27)
+			)
+			(justify left bottom)
+		)
+	)
 	(label "SPI1_NSS"
 		(at 62.357 85.471 180)
@@
 		)
 	)
+	(label "ADC1_IN2{slash}TIM2_CH2{slash}COMP1_INP"
+		(at 184.15 137.16 0)
+		(effects
+			(font
+				(size 1.27 1.27)
+			)
+			(justify left bottom)
+		)
+	)
 	(label "IMON"
 		(at 62.357 127.254 180)
@@
 		)
 	)
-	(label "ADC1_IN11{slash}COMP7_INM{slash}FDCAN2_RX"
-		(at 275.59 139.7 180)
+	(label "UART4_RX{slash}TIM8_CH2N"
+		(at 275.59 144.78 180)
 		(effects
 			(font
@@
 		)
 	)
-	(label "ADC1_IN12{slash}TIM1_CH3N{slash}COMP1_INP"
-		(at 184.15 132.08 0)
-		(effects
-			(font
-				(size 1.27 1.27)
-			)
-			(justify left bottom)
-		)
-	)
 	(label "24V_Ext"
 		(at 248.92 88.9 180)
@@
 		)
 	)
-	(label "ADC1_IN8{slash}TIM1_CH3{slash}COMP3_OUT"
-		(at 184.15 137.16 0)
-		(effects
-			(font
-				(size 1.27 1.27)
-			)
-			(justify left bottom)
-		)
-	)
 	(label "ADC2_IN12{slash}TIM5_CH1{slash}COMP4_INM"
 		(at 162.56 73.152 180)
@@
 		)
 	)
-	(label "OPAMP5_VINM{slash}ADC1_IN4{slash}TIM2_CH4"
-		(at 184.15 149.86 0)
-		(effects
-			(font
-				(size 1.27 1.27)
-			)
-			(justify left bottom)
-		)
-	)
 	(label "ADC1_IN11{slash}COMP7_INM{slash}FDCAN2_RX"
 		(at 162.814 81.28 180)
@@
 		)
 	)
-	(label "ADC1_IN7{slash}TIM1_CH2{slash}COMP3_INP"
-		(at 275.59 106.68 180)
-		(effects
-			(font
-				(size 1.27 1.27)
-			)
-			(justify right bottom)
-		)
-	)
 	(label "SPI2_MISO{slash}ADC1_IN5{slash}TIM1_CH2N"
 		(at 275.59 101.6 180)
@@
 		)
 	)
-	(label "UART4_RX{slash}TIM8_CH2N"
-		(at 185.42 99.06 0)
+	(label "USART3_RX{slash}ADC1_IN14{slash}TIM2_CH4"
+		(at 182.88 99.06 0)
 		(effects
 			(font
@@
 	)
 	(label "I2C4_SCL{slash}TIM3_CH1"
-		(at 185.42 109.22 0)
-		(effects
-			(font
-				(size 1.27 1.27)
-			)
-			(justify left bottom)
-		)
-	)
-	(label "UART1_RX"
-		(at 185.42 93.98 0)
+		(at 182.88 109.22 0)
 		(effects
 			(font
@@
 	)
 	(label "I2C3_SDA{slash}TIM3_CH4"
-		(at 185.42 106.68 0)
+		(at 182.88 106.68 0)
 		(effects
 			(font
@@
 		)
 	)
-	(label "ADC1_IN1{slash}TIM2_CH1{slash}COMP1_OUT"
-		(at 184.15 139.7 0)
+	(label "ADC1_IN12{slash}TIM1_CH3N{slash}COMP1_INP"
+		(at 184.15 149.86 0)
 		(effects
 			(font
@@
 		)
 	)
-	(label "USART3_TX{slash}OPAMP3_VINM{slash}TIM2_CH3"
-		(at 275.59 144.78 180)
-		(effects
-			(font
-				(size 1.27 1.27)
-			)
-			(justify right bottom)
-		)
-	)
 	(label "USART3_RX{slash}ADC1_IN14{slash}TIM2_CH4"
 		(at 165.1 121.92 180)
@@
 		)
 	)
+	(label "ADC1_IN1{slash}TIM2_CH1{slash}COMP1_OUT"
+		(at 184.15 134.62 0)
+		(effects
+			(font
+				(size 1.27 1.27)
+			)
+			(justify left bottom)
+		)
+	)
 	(label "SPI2_MOSI{slash}ADC2_IN15{slash}TIM1_CH3N"
 		(at 163.576 98.044 180)
@@
 		)
 	)
-	(label "UART4_TX{slash}TIM8_CH1N"
-		(at 185.42 101.6 0)
-		(effects
-			(font
-				(size 1.27 1.27)
-			)
-			(justify left bottom)
-		)
-	)
 	(label "FDCAN3_TX"
 		(at 71.12 52.07 0)
@@
 		)
 	)
-	(label "UART1_TX"
-		(at 185.42 96.52 0)
-		(effects
-			(font
-				(size 1.27 1.27)
-			)
-			(justify left bottom)
-		)
-	)
 	(label "I2C3_SDA{slash}TIM3_CH4"
 		(at 147.066 47.498 180)
@@
 		(effects
 			(font
+				(size 1.27 1.27)
+			)
+			(justify right bottom)
+		)
+	)
+	(label "ADC1_IN11{slash}COMP7_INM{slash}FDCAN2_RX"
+		(at 275.59 104.14 180)
+		(effects
+			(font

Commit message: lock in
Connections:
- net UART5_RX: now also J1.15
- net UART5_TX/TIM5_CH2: now also J1.13
- net USART3_RX/ADC1_IN14/TIM2_CH4: no longer J1.15
- net USART3_TX/OPAMP3_VINM/TIM2_CH3: no longer J1.13
Changed lines of the file:
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@@
 	(paper "A4")
 	(bus_alias "USB"
-		(members "UART5_TX/TIM5_CH2" "UART5_RX")
+		(members "USART3_RX/ADC1_IN14/TIM2_CH4" "USART3_TX/OPAMP3_VINM/TIM2_CH3")
 	)
 	(rectangle
@@
 	)
 	(bus_entry
+		(at 114.3 114.935)
+		(size 2.54 2.54)
+		(stroke
+			(width 0)
+			(type default)
+		)
+	)
+	(bus_entry
 		(at 125.222 100.584)
 		(size 2.54 2.54)
@@
 	)
 	(bus_entry
-		(at 85.09 64.77)
-		(size -2.54 2.54)
-		(stroke
-			(width 0)
-			(type default)
-		)
-	)
-	(bus_entry
-		(at 85.09 62.23)
-		(size -2.54 2.54)
-		(stroke
-			(width 0)
-			(type default)
-		)
-	)
-	(bus_entry
 		(at 125.222 73.152)
 		(size 2.54 2.54)
@@
 	)
 	(bus_entry
-		(at 125.222 92.964)
+		(at 109.22 114.935)
 		(size 2.54 2.54)
 		(stroke
@@
 	)
 	(bus_entry
-		(at 125.222 90.424)
+		(at 125.222 92.964)
 		(size 2.54 2.54)
 		(stroke
@@
 	)
 	(bus_entry
-		(at 125.222 40.386)
+		(at 125.222 90.424)
 		(size 2.54 2.54)
 		(stroke
@@
 	)
 	(bus_entry
-		(at 125.222 58.166)
+		(at 125.222 40.386)
 		(size 2.54 2.54)
 		(stroke
@@
 	)
 	(bus_entry
-		(at 85.09 62.23)
-		(size -2.54 2.54)
+		(at 125.222 58.166)
+		(size 2.54 2.54)
 		(stroke
 			(width 0)
@@
 		)
 	)
+	(bus
+		(pts
+			(xy 106.68 113.03) (xy 108.585 114.935)
+		)
+		(stroke
+			(width 0)
+			(type default)
+		)
+	)
 	(wire
 		(pts
@@
 		)
 	)
+	(wire
+		(pts
+			(xy 48.26 71.755) (xy 48.26 72.39)
+		)
+		(stroke
+			(width 0)
+			(type default)
+		)
+	)
 	(bus
 		(pts
@@
 	(wire
 		(pts
-			(xy 182.88 96.52) (xy 218.44 96.52)
+			(xy 116.84 117.475) (xy 116.84 153.035)
 		)
 		(stroke
@@
 		)
 	)
-	(bus
+	(wire
 		(pts
-			(xy 86.36 59.69) (xy 85.09 62.23)
+			(xy 182.88 96.52) (xy 218.44 96.52)
 		)
 		(stroke
@@
 		)
 	)
+	(bus
+		(pts
+			(xy 114.3 114.935) (xy 116.84 114.935)
+		)
+		(stroke
+			(width 0)
+			(type default)
+		)
+	)
 	(wire
 		(pts
@@
 		)
 	)
+	(bus
+		(pts
+			(xy 108.585 114.935) (xy 109.22 114.935)
+		)
+		(stroke
+			(width 0)
+			(type default)
+		)
+	)
 	(wire
 		(pts
@@
 		)
 	)
-	(bus
-		(pts
-			(xy 85.09 62.23) (xy 85.09 64.77)
-		)
-		(stroke
-			(width 0)
-			(type default)
-		)
-	)
 	(wire
 		(pts
@@
 	(wire
 		(pts
-			(xy 72.39 67.31) (xy 82.55 67.31)
-		)
-		(stroke
-			(width 0)
-			(type default)
-		)
-	)
-	(wire
-		(pts
-			(xy 48.26 68.58) (xy 68.58 68.58)
+			(xy 48.26 68.58) (xy 48.895 68.58)
 		)
 		(stroke
@@
 	(wire
 		(pts
-			(xy 128.27 124.46) (xy 165.1 124.46)
+			(xy 128.27 124.46) (xy 163.83 124.46)
 		)
 		(stroke
@@
 		)
 	)
+	(wire
+		(pts
+			(xy 111.76 117.475) (xy 111.76 153.035)
+		)
+		(stroke
+			(width 0)
+			(type default)
+		)
+	)
 	(bus
 		(pts
@@
 	(wire
 		(pts
-			(xy 128.27 121.92) (xy 165.1 121.92)
+			(xy 128.27 121.92) (xy 163.83 121.92)
 		)
 		(stroke
@@
 	(wire
 		(pts
-			(xy 48.26 72.39) (xy 64.77 72.39)
+			(xy 48.26 71.755) (xy 48.895 71.755)
 		)
 		(stroke
@@
 	(bus
 		(pts
+			(xy 109.22 114.935) (xy 114.3 114.935)
+		)
+		(stroke
+			(width 0)
+			(type default)
+		)
+	)
+	(bus
+		(pts
 			(xy 123.19 50.546) (xy 125.222 52.832)
 		)
@@
 		)
 	)
-	(wire
-		(pts
-			(xy 62.23 64.77) (xy 82.55 64.77)
-		)
-		(stroke
-			(width 0)
-			(type default)
-		)
-	)
 	(bus
 		(pts
@@
 		)
 	)
-	(label "UART5_RX"
-		(at 64.77 72.39 180)
-		(effects
-			(font
-				(size 1.27 1.27)
-			)
-			(justify right bottom)
-		)
-	)
 	(label "ADC1_IN7{slash}TIM1_CH2{slash}COMP3_INP"
 		(at 275.59 139.7 180)
@@
 		)
 	)
-	(label "USART3_TX{slash}OPAMP3_VINM{slash}TIM2_CH3"
-		(at 165.1 124.46 180)
-		(effects
-			(font
-				(size 1.27 1.27)
-			)
-			(justify right bottom)
-		)
-	)
 	(label "SDC_DET"
 		(at 62.357 98.806 180)
@@
 		)
 	)
+	(label "UART5_RX"
+		(at 163.83 124.46 180)
+		(effects
+			(font
+				(size 1.27 1.27)
+			)
+			(justify right bottom)
+		)
+	)
 	(label "ADC1_IN7{slash}TIM1_CH2{slash}COMP3_INP"
 		(at 162.052 58.166 180)
@@
 		)
 	)
-	(label "USART3_TX{slash}OPAMP3_VINM{slash}TIM2_CH3"
-		(at 182.88 101.6 0)
+	(label "SPI3_SCK{slash}TIM2_CH2{slash}USART2_TX"
+		(at 275.59 129.54 180)
 		(effects
 			(font
 				(size 1.27 1.27)
 			)
-			(justify left bottom)
+			(justify right bottom)
 		)
 	)
-	(label "SPI3_SCK{slash}TIM2_CH2{slash}USART2_TX"
-		(at 275.59 129.54 180)
+	(label "USART3_RX{slash}ADC1_IN14{slash}TIM2_CH4"
+		(at 48.895 68.58 0)
 		(effects
 			(font
 				(size 1.27 1.27)
 			)
-			(justify right bottom)
+			(justify left bottom)
 		)
 	)
@@
 		)
 	)
-	(label "UART5_TX{slash}TIM5_CH2"
-		(at 68.58 68.58 180)
-		(effects
-			(font
-				(size 1.27 1.27)
-			)
-			(justify right bottom)
-		)
-	)
 	(label "24V_Ext"
 		(at 248.92 88.9 180)
@@
 		)
 	)
-	(label "UART5_RX"
-		(at 72.39 67.31 0)
-		(effects
-			(font
-				(size 1.27 1.27)
-			)
-			(justify left bottom)
-		)
-	)
 	(label "SPI3_NSS{slash}TIM1_CH3{slash}COMP6_OUT"
 		(at 163.322 87.884 180)
@@
 		)
 	)
-	(label "USART3_RX{slash}ADC1_IN14{slash}TIM2_CH4"
-		(at 182.88 99.06 0)
-		(effects
-			(font
-				(size 1.27 1.27)
-			)
-			(justify left bottom)
-		)
-	)
 	(label "UART1_RX"
 		(at 163.83 116.84 180)
@@
 		)
 	)
+	(label "UART5_TX{slash}TIM5_CH2"
+		(at 182.88 101.6 0)
+		(effects
+			(font
+				(size 1.27 1.27)
+			)
+			(justify left bottom)
+		)
+	)
+	(label "UART5_TX{slash}TIM5_CH2"
+		(at 163.83 121.92 180)
+		(effects
+			(font
+				(size 1.27 1.27)
+			)
+			(justify right bottom)
+		)
+	)
+	(label "USART3_TX{slash}OPAMP3_VINM{slash}TIM2_CH3"
+		(at 48.895 71.755 0)
+		(effects
+			(font
+				(size 1.27 1.27)
+			)
+			(justify left bottom)
+		)
+	)
 	(label "SPI1_MISO"
 		(at 62.357 88.646 180)
@@
 		)
 	)
-	(label "SPI3_MOSI{slash}TIM3_CH2{slash}TIM17_CH1"
-		(at 275.59 132.08 180)
+	(label "USART3_TX{slash}OPAMP3_VINM{slash}TIM2_CH3"
+		(at 116.84 153.035 90)
 		(effects
 			(font
 				(size 1.27 1.27)
 			)
-			(justify right bottom)
+			(justify left bottom)
 		)
 	)
-	(label "AddressableLED"
-		(at 64.897 112.141 180)
+	(label "SPI3_MOSI{slash}TIM3_CH2{slash}TIM17_CH1"
+		(at 275.59 132.08 180)
 		(effects
 			(font
@@
 		)
 	)
-	(label "ADC1_IN15{slash}TIM1_CH2N{slash}COMP4_INP"
-		(at 162.56 78.486 180)
+	(label "AddressableLED"
+		(at 64.897 112.141 180)
 		(effects
 			(font
@@
 		)
 	)
-	(label "USART3_RX{slash}ADC1_IN14{slash}TIM2_CH4"
-		(at 165.1 121.92 180)
+	(label "ADC1_IN15{slash}TIM1_CH2N{slash}COMP4_INP"
+		(at 162.56 78.486 180)
 		(effects
 			(font
@@
 		)
 	)
+	(label "UART5_RX"
+		(at 182.88 99.06 0)
+		(effects
+			(font
+				(size 1.27 1.27)
+			)
+			(justify left bottom)
+		)
+	)
 	(label "ADC1_IN2{slash}TIM2_CH2{slash}COMP1_INP"
 		(at 162.306 68.072 180)
@@
 		)
 	)
-	(label "UART5_TX{slash}TIM5_CH2"
-		(at 62.23 64.77 0)
+	(label "USART3_RX{slash}ADC1_IN14{slash}TIM2_CH4"
+		(at 111.76 153.035 90)
 		(effects
 			(font
@@
 		)
 		(pin "{USB}" bidirectional
-			(at 86.36 59.69 180)
+			(at 106.68 113.03 270)
 			(effects
 				(font
