File: LeaderSOM.kicad_pcb (KiCad board)
At the start: 2 copper layers, 85 parts, among them IC1 LP5912-3.3DRVR, IC2 TPS1120DR, J1 SWD, J10 SOMConnector, J11 CAN_Int, J2 USB_B_Micro, J4 Micro_SD_Card_Det, J5 CAN_In2, J6 CAN_Out2, J7 CarPowerConnector, J9 SOMConnector, Q1 PBSS4330X,135, Q2 SI7149ADP-T1-GE3, SW2 Reset, U3 CP2102N-A02-GQFN24, U4 ISO1044BD, U5 CDSOT23-T24CAN, U6 STM32F413RHTx, U8 ISO1044BD, U9 CDSOT23-T24CAN, Y2 8M

Commit message: 👹
Parts:
- removed C25: 100nF, Capacitor_SMD:C_0805_2012Metric
- removed CR1: D5V0P4UR6SO-7, UTSVT_ICs:SOT26_DIO
- added C14: 100nF, Capacitor_SMD:C_0805_2012Metric, F.Cu at (141.6, 100.7)
- added C15: 100nF, Capacitor_SMD:C_0805_2012Metric, F.Cu at (141.6, 54.3)
- added D4: 3V3, LED_SMD:LED_0805_2012Metric, F.Cu at (159.4, 109.6)
- added D6: V_CAN2, LED_SMD:LED_0805_2012Metric, F.Cu at (199.4, 63.3)
- added F1: 1.8A, Fuse:Fuse_1206_3216Metric, F.Cu at (181.3, 108.3)
- added Q3: SI7149ADP-T1-GE3, UTSVT_ICs:POWERPAKSO-8, F.Cu at (148.4, 103.7)
- added R13: 49.9, Resistor_SMD:R_0805_2012Metric, F.Cu at (137.2, 63.1)
- added R14: 160, Resistor_SMD:R_0805_2012Metric, F.Cu at (185.1, 117.8)
- added R21: 160, Resistor_SMD:R_0805_2012Metric, F.Cu at (185.1, 123.7)
- added R23: 160, Resistor_SMD:R_0805_2012Metric, F.Cu at (185.1, 126.7)
- added R24: 160, Resistor_SMD:R_0805_2012Metric, F.Cu at (185.1, 129.6)
- added R25: 160, Resistor_SMD:R_0805_2012Metric, F.Cu at (189.6, 117.8)
- added R26: 160, Resistor_SMD:R_0805_2012Metric, F.Cu at (189.6, 120.8)
- added R27: 160, Resistor_SMD:R_0805_2012Metric, F.Cu at (189.6, 123.7)
- added R28: 160, Resistor_SMD:R_0805_2012Metric, F.Cu at (189.6, 126.7)
- added R29: 160, Resistor_SMD:R_0805_2012Metric, F.Cu at (189.6, 129.6)
- added R30: 160, Resistor_SMD:R_0805_2012Metric, F.Cu at (194.0, 117.8)
- added R31: 160, Resistor_SMD:R_0805_2012Metric, F.Cu at (194.0, 120.8)
- added R32: 160, Resistor_SMD:R_0805_2012Metric, F.Cu at (194.0, 123.7)
- added R33: 160, Resistor_SMD:R_0805_2012Metric, F.Cu at (194.0, 126.7)
- added R34: 5.1k, Resistor_SMD:R_0805_2012Metric, F.Cu at (186.5, 112.9)
- added R37: 5.1k, Resistor_SMD:R_0805_2012Metric, F.Cu at (198.8, 57.2)
- added R4: 10k, Resistor_SMD:R_0805_2012Metric, F.Cu at (137.2, 54.2)
- added SW1: Reset, Button_Switch_SMD:SW_SPST_B3SL-1002P, F.Cu at (166.0, 56.9)
- added U1: MAX16914AUB/V+T, UTSVT_ICs:21-0061L_MXM, F.Cu at (147.5, 109.1)
- D2: value PowerLED -> 12V
- D5: value PowerLED -> V_CAN1
- R1: value 5.1k -> 20k
- R11: value 10k -> 49.9
- R15: value 49.9 -> 138k
- R16: value 49.9 -> 160
- R2: value 1k -> 12k
- R9: value 1k -> 2.2k
- SW2: value Reset -> BTN1
- moved R16 88.5 mm to (185.1, 120.8)
- moved PS2 88.1 mm to (157.1, 99.4)
- moved C10 67.2 mm to (186.5, 103.9)
- moved C12 67.2 mm to (186.5, 106.9)
- moved C9 67.2 mm to (186.5, 100.9)
- moved Q2 57.3 mm to (148.4, 97.5)
- moved C18 53.4 mm to (211.1, 125.0)
- moved C19 53.4 mm to (211.1, 128.0)
- moved D1 53.4 mm to (200.3, 127.4)
- moved J2 53.4 mm to (207.5, 119.3)
- moved R5 53.4 mm to (200.4, 117.8)
- moved R6 53.4 mm to (200.4, 120.8)
- moved R8 53.4 mm to (200.4, 123.7)
- moved U3 53.4 mm to (205.7, 126.6)
- moved R10 49.5 mm to (186.5, 109.9)
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Connections:
- net /CAN1_Rx renamed /CAN3_RX
- net /CAN1_Tx renamed /CAN3_TX
- C13 pad 1: +3V3 -> +3.3V
- C28 pad 1: VDDA -> +3.3VA
- C28 pad 2: GNDA -> GND
- C29 pad 1: /NRST -> /BTN1
- C30 pad 1: VDDA -> +3.3VA
- C30 pad 2: GNDA -> GND
- C7 pad 1: +3V3 -> +3.3V
- CR2 pad 1: /SPI_CS -> /SPI1_CS
- CR2 pad 4: /SPI1_CLK -> /SPI1_SCK
- D5 pad 1: GND -> /InternalCAN/-V_CAN1
- FB2 pad 2: VDDA -> +3.3VA
- J10 pad 1: +12V -> GND
- J10 pad 10: VDDA -> GND
- J10 pad 11: GNDA -> GND
- J10 pad 12: GNDA -> GND
- J10 pad 13: /USART1_Tx -> /ADC1_IN11/GPIO
- J10 pad 14: /I2CL_SDA -> /UART5_TX/GPIO
- J10 pad 15: /USART1_Rx -> /ADC1_IN10/GPIO
- J10 pad 16: /I2C1_SCL -> /UART5_RX/GPIO
- J10 pad 17: GND -> +3.3V
- J10 pad 18: GND -> +3.3V
- J10 pad 2: +12V -> GND
- J10 pad 5: /USART2_Rx -> /ADC_IN13/GPIO
- J10 pad 6: /I2C2_SCL -> /ADC1_IN3/USART2_RX/GPIO
- J10 pad 7: /USART2_Tx -> /ADC_IN12/GPIO
- J10 pad 8: /USART3_Tx -> /ADC1_IN2/USART2_TX/GPIO
- J10 pad 9: VDDA -> +3.3VA
- J4 pad 2: /SPI_CS -> /SPI1_CS
- J4 pad 5: /SPI1_CLK -> /SPI1_SCK
- J4 pad 9: /PC8 -> /SDC_DET
- J9 pad 1: +3.3V -> +12V
- J9 pad 10: /PA12 -> /SPI2_CS/TIM1_CH4/GPIO
- J9 pad 11: /PA4 -> +3.3V
- J9 pad 12: /PA11 -> /SPI2_MOSI/TIM1_CH3/GPIO
- J9 pad 13: /PA3 -> /I2C1_SDA
- J9 pad 14: /PA10 -> /SPI2_SCK/TIM1_CH2/GPIO
- J9 pad 15: /PA2 -> /I2C1_SCL
- J9 pad 16: /PA9 -> GND
- J9 pad 2: +3.3V -> +12V
- J9 pad 5: /PA7 -> /I2C3_SDA/GPIO
- J9 pad 6: /PC8 -> GND
- J9 pad 7: /PA6 -> /I2C3_SCL/TIM1_CH1/GPIO
- J9 pad 8: /I2C2_SDA -> /SPI2_MISO/GPIO
- J9 pad 9: /PA5 -> +3.3V
- LED1 pad 1: /DISP5 -> Net-(LED1-E)
- LED1 pad 10: /DISP7 -> Net-(LED1-G)
- LED1 pad 2: /DISP4 -> Net-(LED1-D)
- LED1 pad 3: +3V3 -> +3.3V
- LED1 pad 4: /DISP3 -> Net-(LED1-C)
- LED1 pad 5: +3V3 -> +3.3V
- LED1 pad 6: /DISP2 -> Net-(LED1-B)
- LED1 pad 7: /DISP1 -> Net-(LED1-A)
- LED1 pad 8: +3V3 -> +3.3V
- LED1 pad 9: /DISP6 -> Net-(LED1-F)
- LED2 pad 1: /DISP12 -> Net-(LED2-E)
- LED2 pad 10: /DISP14 -> Net-(LED2-G)
- LED2 pad 2: /DISP11 -> Net-(LED2-D)
- LED2 pad 3: +3V3 -> +3.3V
- LED2 pad 4: /DISP10 -> Net-(LED2-C)
- LED2 pad 5: +3V3 -> +3.3V
- LED2 pad 6: /DISP9 -> Net-(LED2-B)
- LED2 pad 7: /DISP8 -> Net-(LED2-A)
- LED2 pad 8: +3V3 -> +3.3V
- LED2 pad 9: /DISP13 -> Net-(LED2-F)
- PS3 pad 6: /InternalCAN/+V_CAN1 -> Net-(PS3-+VOUT)
- Q2 pad 1: +12V -> Net-(Q2-S_1)
- Q2 pad 2: +12V -> Net-(Q2-S_1)
- Q2 pad 3: +12V -> Net-(Q2-S_1)
- R11 pad 1: +3.3V -> Net-(U6-PA5)
- R11 pad 2: /I2CL_SDA -> /SPI1_SCK
- R15 pad 1: /SPI1_CLK -> Net-(U1-SET)
- R15 pad 2: Net-(U6-PC10) -> GND
- R16 pad 1: /SPI1_MOSI -> /DISP2
- R16 pad 2: Net-(U6-PC12) -> Net-(LED1-B)
- R17 pad 2: /I2C2_PU_En -> /I2C3_PU_En
- R18 pad 1: /I2C2_PU_En -> /I2C3_PU_En
- R19 pad 2: /I2C2_SCL -> /I2C3_SCL/TIM1_CH1/GPIO
- R2 pad 1: Net-(Q2-G) -> Net-(U1-TERM)
- R2 pad 2: GND -> Net-(U1-SET)
- R20 pad 1: /I2C2_SDA -> /I2C3_SDA/GPIO
- R7 pad 2: /I2C1_SCL -> /I2C1_SDA
- R9 pad 2: Net-(D5-A) -> Net-(D4-A)
- SW2 pad 1: /NRST -> /BTN1
- U3 pad 20: /USART3_Tx -> /USB_UART4_TX
- U3 pad 21: /I2C2_SCL -> /USB_UART4_RX
- U6 pad 10: /DISP3 -> /ADC_IN12/GPIO
- U6 pad 11: /DISP4 -> /ADC_IN13/GPIO
- U6 pad 12: GNDA -> GND
- U6 pad 13: VDDA -> +3.3VA
- U6 pad 14: /USART1_Tx -> /USB_UART4_TX
- U6 pad 15: /USART1_Rx -> /USB_UART4_RX
- U6 pad 16: /PA2 -> /ADC1_IN2/USART2_TX/GPIO
- U6 pad 17: /PA3 -> /ADC1_IN3/USART2_RX/GPIO
- U6 pad 20: /PA4 -> /SPI1_CS
- U6 pad 21: /PA5 -> Net-(U6-PA5)
- U6 pad 22: /PA6 -> /SPI1_MISO
- U6 pad 23: /PA7 -> Net-(U6-PA7)
- U6 pad 24: /DISP5 -> /DISP1
- U6 pad 25: /DISP6 -> /DISP2
- U6 pad 26: /DISP7 -> /DISP3
- U6 pad 27: /DISP8 -> /DISP4
- U6 pad 28: /DISP9 -> /DISP5
- U6 pad 29: /DISP10 -> /DISP6
- U6 pad 33: /USART2_Rx -> /UART5_RX/GPIO
- U6 pad 34: /USART2_Tx -> /UART5_TX/GPIO
- U6 pad 35: /DISP11 -> /DISP7
- U6 pad 36: /DISP12 -> /DISP8
- U6 pad 37: /DISP13 -> /DISP9
- U6 pad 38: /DISP14 -> /DISP10
- U6 pad 39: /PC8 -> /BTN1
- U6 pad 40: /I2C2_SDA -> /I2C3_SDA/GPIO
- U6 pad 41: /I2C2_SCL -> /I2C3_SCL/TIM1_CH1/GPIO
- U6 pad 42: /PA9 -> /SPI2_SCK/TIM1_CH2/GPIO
- U6 pad 43: /PA10 -> /SPI2_MOSI/TIM1_CH3/GPIO
- U6 pad 44: /PA11 -> /SPI2_CS/TIM1_CH4/GPIO
- U6 pad 45: /PA12 -> /SPI2_MISO/GPIO
- U6 pad 50: /USART3_Tx -> /DISP11
- U6 pad 51: Net-(U6-PC10) -> /DISP12
- U6 pad 52: /SPI1_MISO -> /DISP13
- U6 pad 53: Net-(U6-PC12) -> /DISP14
- U6 pad 54: /SPI_CS -> /SDC_DET
- U6 pad 57: /CAN2_Rx -> /I2C3_PU_En
- U6 pad 58: /CAN2_Tx -> /I2C1_SCL
- U6 pad 59: /I2C2_PU_En -> /I2C1_SDA
- U6 pad 61: /I2C1_SCL -> /CAN1_RX
- U6 pad 62: /I2CL_SDA -> /CAN1_TX
- U6 pad 8: /DISP1 -> /ADC1_IN10/GPIO
- U6 pad 9: /DISP2 -> /ADC1_IN11/GPIO
- U8 pad 2: /CAN2_Tx -> /CAN1_TX
- U8 pad 3: /CAN2_Rx -> /CAN1_RX

Commit message: ahahaha ahehehe ahohohoho
Parts:
- removed TP3: +5V_TP, TestPoint:TestPoint_Keystone_5005-5009_Compact
- removed TP4: GND_TP, TestPoint:TestPoint_Keystone_5005-5009_Compact
- added C16: 100nF, Capacitor_SMD:C_0805_2012Metric, B.Cu at (113.0, 105.0)
- C1, C13, C14, C2, C5, C6, C7, D2, D4, FB2, R14, R15, R16, R2, R21, R23, R24, R25, R26, R27, R28, R29, R30, R31, R32, R33, R35, R36: moved to B.Cu
- moved PS3 233.5 mm to (44.0, -105.0)
- moved C12 230.2 mm to (69.0, -91.0)
- moved C10 224.3 mm to (54.0, -77.0)
- moved U4 216.2 mm to (51.0, -71.0)
- moved L1 216.1 mm to (37.0, -53.0)
- moved C9 211.0 mm to (50.0, -60.0)
- moved R34 206.7 mm to (58.0, -49.0)
- moved D5 205.9 mm to (53.0, -50.0)
- moved J11 204.9 mm to (62.0, -71.0)
- moved R10 204.1 mm to (69.0, -57.0)
- moved F1 203.8 mm to (58.0, -54.0)
- moved U5 201.7 mm to (69.0, -62.0)
- moved PS1 151.5 mm to (203.0, -75.0)
- moved R26 145.9 mm to (48.0, 156.0), turned to -90 degrees
- moved R25 144.7 mm to (50.0, 156.0), turned to -90 degrees
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Connections:
- Q1 pad 2: Net-(Q1-B) -> +5V
- Q1 pad 3: +5V -> Net-(Q1-B)

Commit message: f is for friends that do stuff together
Parts:
- removed FB1: 5VFB, Inductor_SMD:L_0805_2012Metric
- added H1: M.3, MountingHole:MountingHole_3mm, F.Cu at (120.0, 93.5)
- added H2: M.3, MountingHole:MountingHole_3mm, F.Cu at (120.0, 53.0)
- C10, C11, C12, C15, C17, C18, C19, C21, C22, C23, C24, C26, C27, C28, C29, C3, C30, C8, C9, D1, D3, IC1, J10, J4, J9, L1, Q2, Q3, R1, R10, R17, R18, R19, R20, R22, R3, R34, R37, R4, R5, R6, R7, R8, R9, U1, U4, U5, U8, U9: moved to B.Cu
- D2, D4: moved to F.Cu
- moved PS3 196.5 mm to (107.0, 81.2), turned to 90 degrees
- moved PS1 192.0 mm to (107.5, 91.5), turned to 180 degrees
- moved R37 184.4 mm to (98.5, 84.1), turned to -90 degrees
- moved J5 178.3 mm to (93.5, 81.5)
- moved D6 178.2 mm to (101.5, 82.5), turned to 90 degrees
- moved C12 175.2 mm to (112.0, 78.8), turned to 180 degrees
- moved JP2 166.2 mm to (98.2, 70.2), turned to 90 degrees
- moved JP3 164.6 mm to (98.2, 66.2), turned to 90 degrees
- moved U9 162.0 mm to (101.5, 74.5)
- moved C11 158.1 mm to (98.5, 79.0), turned to 90 degrees
- moved C8 157.5 mm to (103.0, 86.0), turned to 180 degrees
- moved C3 155.2 mm to (112.0, 86.0), turned to 180 degrees
- moved U8 150.6 mm to (102.5, 80.5), turned to 90 degrees
- moved U4 150.2 mm to (111.5, 66.5), turned to 90 degrees
- moved L1 149.9 mm to (112.0, 76.8), turned to 180 degrees
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Connections:
- C3 pad 1: Net-(JP2-B) -> /CarCAN/5V_ISO
- JP2 pad 2: Net-(JP2-B) -> /CarCAN/5V_ISO
Other:
- board outline added: 61 x 50 mm
- copper layers 2 -> 4

Commit message: hi lakshay
Parts:
- removed C3: 10uF, Capacitor_SMD:C_0805_2012Metric
- removed JP2: CAN_PWR Jumper, Connector_PinHeader_2.54mm:PinHeader_1x02_P2.54mm_Vertical
- removed PS1: 1769405141, UTSVT_Power:1769405141
- added TP1: +12V_TP, UTSVT_Special:TestPoint_HEX_3mmID, F.Cu at (166.0, 83.0)
- added TP2: +3V3_TP, UTSVT_Special:TestPoint_HEX_3mmID, F.Cu at (161.0, 79.0)
- added TP3: +5V_TP, UTSVT_Special:TestPoint_HEX_3mmID, F.Cu at (161.0, 83.0)
- added TP4: GND_TP, UTSVT_Special:TestPoint_HEX_3mmID, F.Cu at (166.0, 79.0)
- added TP6: GND_TP, UTSVT_Special:TestPoint_HEX_3mmID, B.Cu at (163.0, 81.0)
- J4: moved to F.Cu
- moved R22 53.4 mm to (65.0, 98.0)
- moved D5 50.1 mm to (151.7, 49.0), turned to 90 degrees
- moved R34 48.5 mm to (151.2, 50.0), turned to 180 degrees
- moved C18 48.1 mm to (173.0, 96.0)
- moved C19 48.1 mm to (175.0, 96.0)
- moved R5 48.1 mm to (177.0, 91.0)
- moved R6 48.1 mm to (175.0, 91.0)
- moved R8 48.1 mm to (177.0, 96.0)
- moved U3 48.1 mm to (175.2, 94.1)
- moved C10 44.5 mm to (151.2, 53.5), turned to 180 degrees
- moved R10 42.3 mm to (151.2, 55.5), turned to 180 degrees
- moved F1 40.7 mm to (151.7, 57.5), turned to 90 degrees
- moved J2 39.6 mm to (142.0, 51.7), turned to 180 degrees
- moved U5 39.2 mm to (151.2, 58.5), turned to -90 degrees
- moved J4 37.9 mm to (107.0, 88.0)
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
Commit message: u is for u n me
Parts:
- C16, D3, Q2, Q3, R15, R2, U1, U4, U8: moved to F.Cu
- J4, R11, R12, R13: moved to B.Cu
- moved C11 61.6 mm to (114.0, 58.5), turned to 0 degrees
- moved C8 60.5 mm to (114.0, 62.5), turned to 0 degrees
- moved U8 58.3 mm to (114.0, 60.5)
- moved CR2 57.5 mm to (113.5, 82.5)
- moved TP6 56.9 mm to (106.5, 74.5)
- moved R37 56.0 mm to (102.5, 60.5), turned to 0 degrees
- moved SW1 54.0 mm to (131.5, 90.0), turned to 0 degrees
- moved TP1 53.8 mm to (112.5, 77.0), turned to 180 degrees
- moved TP4 53.0 mm to (114.2, 68.0), turned to 180 degrees
- moved D6 52.1 mm to (102.5, 61.5), turned to 0 degrees
- moved SW2 51.0 mm to (144.5, 90.0), turned to 0 degrees
- moved D5 50.3 mm to (102.5, 59.5), turned to 180 degrees
- moved R17 49.9 mm to (127.5, 60.0), turned to 0 degrees
- moved R34 49.4 mm to (102.5, 58.5)
- moved C19 49.2 mm to (127.0, 85.0), turned to 90 degrees
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Connections:
- CR2 pad 1: /SPI1_CS -> /SPI1_SCK
- CR2 pad 3: /SPI1_MOSI -> /SPI1_MISO
- CR2 pad 4: /SPI1_SCK -> /SPI1_CS
- CR2 pad 6: /SPI1_MISO -> /SPI1_MOSI
- J4 pad 3: /SPI1_MISO -> /SPI1_MOSI
- R12 pad 1: /SPI1_MOSI -> /SPI1_MISO

Commit message: n is for anywhere and anytime at all
Parts:
- removed C13, C7: 1uF, Capacitor_SMD:C_0805_2012Metric
- moved C14 13.6 mm to (115.5, 66.5), turned to 90 degrees
- moved FB2 11.2 mm to (113.5, 66.5), turned to -90 degrees
- moved R27 5.39 mm to (139.5, 66.5)
- moved R23 2.50 mm to (139.5, 81.5), turned to 0 degrees
- moved R24 2.50 mm to (139.5, 83.5), turned to 0 degrees
- moved R25 2.50 mm to (134.4, 81.5), turned to 180 degrees
- moved R26 2.50 mm to (134.4, 83.5), turned to 180 degrees
- moved R14 2.00 mm to (134.4, 78.0), turned to 180 degrees
- moved R16 2.00 mm to (134.4, 76.0), turned to 180 degrees
- moved R21 2.00 mm to (139.5, 78.0), turned to 0 degrees
- moved R29 2.00 mm to (139.5, 68.5)
- moved R30 2.00 mm to (139.5, 70.5)
- moved R31 2.00 mm to (139.5, 72.5)
- moved R32 2.00 mm to (134.5, 70.5), turned to 180 degrees
- moved R33 2.00 mm to (134.5, 72.5), turned to 180 degrees
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Connections:
- U6 pad 24: /DISP1 -> /DISP7
- U6 pad 25: /DISP2 -> /DISP6
- U6 pad 26: /DISP3 -> /DISP5
- U6 pad 27: /DISP4 -> /DISP2
- U6 pad 28: /DISP5 -> /DISP4
- U6 pad 29: /DISP6 -> /DISP1
- U6 pad 35: /DISP7 -> /DISP3
Routing:
- net /CarCAN/CAN_H: track 0.00 -> 45.1 mm, vias 0 -> 1
- net /CarCAN/CAN_L: track 0.00 -> 45.0 mm, vias 0 -> 1
- net /SPI1_CS: track 0.00 -> 34.6 mm, vias 0 -> 2
- net /SPI1_MISO: track 0.00 -> 28.5 mm, vias 0 -> 2
- net GND: track 0.00 -> 24.7 mm, vias 0 -> 10
- net /SPI1_MOSI: track 0.00 -> 24.1 mm, vias 0 -> 2
- net +12V: track 0.00 -> 22.8 mm, vias 0 -> 4
- net /SPI1_SCK: track 0.00 -> 22.3 mm, vias 0 -> 2
- net Net-(U6-PA5): track 0.00 -> 21.3 mm, vias 0 -> 2
- net Net-(U6-PA7): track 0.00 -> 20.5 mm, vias 0 -> 2
- net /InternalCAN/CAN_H: track 0.00 -> 20.0 mm, vias 0 -> 1
- net /InternalCAN/CAN_L: track 0.00 -> 19.7 mm, vias 0 -> 1
- net /DISP5: track 0.00 -> 17.4 mm, vias 0 -> 1
- net /DISP4: track 0.00 -> 16.7 mm, vias 0 -> 1
- net /SDC_DET: track 0.00 -> 16.0 mm, vias 0 -> 2
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- added copper zone on F.Cu, net +12V
- added copper zone on B.Cu, net +3.3V
- added copper zone on F.Cu, net +3.3V
- added copper zone on In2.Cu, net +3.3V
- added copper zone on F.Cu, net +5V
- added copper zone on F.Cu, net /Power_Distribution/12V_In
- added copper zone on B.Cu, net GND
- added copper zone on F.Cu, net GND
- added copper zone on In1.Cu, net GND
- added copper zone on B.Cu, net Net-(IC1-EN)
- added copper zone on F.Cu, net Net-(Q2-S_1)

Commit message: fuck
Parts:
- R22: moved to F.Cu
- moved J10 12.0 mm to (145.9, 80.0)
- moved J9 12.0 mm to (145.9, 68.0)
- moved C10 7.16 mm to (114.0, 55.5)
- moved R17 4.04 mm to (124.5, 62.7), turned to 90 degrees
- moved R18 3.62 mm to (134.5, 62.6), turned to 90 degrees
- moved C11 1.50 mm to (114.0, 60.0)
Connections:
- U6 pad 36: /DISP8 -> /DISP10
- U6 pad 37: /DISP9 -> /DISP8
- U6 pad 38: /DISP10 -> /DISP9
Routing:
- net +3.3VA: track 3.32 -> 56.7 mm, vias 1 -> 3
- net /BTN1: track 0.00 -> 43.4 mm, vias 0 -> 2
- net /I2C1_SDA: track 2.36 -> 37.2 mm, vias 1 -> 3
- net /I2C1_SCL: track 2.39 -> 37.2 mm, vias 1 -> 3
- net GND: track 24.7 -> 56.0 mm, vias 10 -> 19
- net /SPI2_MISO/GPIO: track 0.00 -> 30.3 mm, vias 0 -> 2
- net /SPI2_CS/TIM1_CH4/GPIO: track 0.00 -> 29.5 mm, vias 0 -> 2
- net /SWDIO: track 0.00 -> 29.4 mm, vias 0 -> 1
- net /UART5_RX/GPIO: track 0.00 -> 29.4 mm, vias 0 -> 2
- net /SWCLK: track 0.00 -> 29.4 mm, vias 0 -> 1
- net /SPI2_MOSI/TIM1_CH3/GPIO: track 0.00 -> 28.9 mm, vias 0 -> 2
- net /UART5_TX/GPIO: track 0.00 -> 28.5 mm, vias 0 -> 2
- net /SPI2_SCK/TIM1_CH2/GPIO: track 0.00 -> 28.0 mm, vias 0 -> 2
- net /I2C3_PU_En: track 1.55 -> 27.6 mm
- net /ADC1_IN10/GPIO: track 0.00 -> 24.4 mm, vias 0 -> 2
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- added copper zone on In2.Cu, net +12V
- added copper zone on In2.Cu, net +5V
- added copper zone on B.Cu, net /CarCAN/+V_CAN2
- added copper zone on In1.Cu, net /CarCAN/+V_CAN2
- added copper zone on In2.Cu, net /CarCAN/+V_CAN2
- added copper zone on B.Cu, net /CarCAN/-V_CAN2
- added copper zone on F.Cu, net /CarCAN/-V_CAN2
- added copper zone on In1.Cu, net /CarCAN/-V_CAN2
- added copper zone on In2.Cu, net /CarCAN/-V_CAN2
- added copper zone on B.Cu, net /InternalCAN/+V_CAN1
- added copper zone on B.Cu, net /InternalCAN/-V_CAN1
- added copper zone on F.Cu, net /InternalCAN/-V_CAN1
- added copper zone on B.Cu, net Net-(PS3-+VOUT)

Commit message: All happy families are alike; each unhappy family is unhappy in its own way.
Parts:
- added G***: LOGO, LOGO, B.Cu at (145.5, 92.0)
Other:
- board text added: "+12V"
- board text added: "+V"
- board text added: "-V"
- board text added: "12V"
- board text added: "3V3"
- board text added: "5V"
- board text added: "<<< POWER CONNECTOR"
- board text added: "CAN TERM"
- board text added: "CAR CAN"
- board text added: "CLK"
- board text added: "GND"
- board text added: "HI"
- board text added: "INTERNAL CAN"
- board text added: "IO"
- board text added: "LO"
- board text added: "RESET"
