File: LeaderSOM.kicad_pcb (KiCad board)
At the start: 4 copper layers, 61 x 50 mm, 109 parts, among them IC1 LP5912-3.3DRVR, IC2 TPS1120DR, J1 SWD, J10 SOMConnector, J11 CAN_Int, J2 USB_B_Micro, J4 Micro_SD_Card_Det, J5 CAN_In2, J6 CAN_Out2, J7 CarPowerConnector, J9 SOMConnector, Q1 PBSS4330X,135, Q2 SI7149ADP-T1-GE3, Q3 SI7149ADP-T1-GE3, SW1 Reset, SW2 BTN1, U1 MAX16914AUB/V+T, U3 CP2102N-A02-GQFN24, U4 ISO1044BD, U5 CDSOT23-T24CAN, U6 STM32F413RHTx, U8 ISO1044BD, U9 CDSOT23-T24CAN, Y2 8M

Commit message: updated 12V/5V non-isolated coverter RVAR output-setting resistors to SMD options
Parts:
- R36: footprint Resistor_SMD:R_0805_2012Metric -> Resistor_SMD:R_0603_1608Metric
Changed lines of the file:
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@@
     (tags "resistor")
     (property "Field2" "")
-    (property "Mouser Part Number" "71-CRCW08051K00FKEAC")
-    (property "P/N" "CRCW08051K00FKEAC")
+    (property "Mouser Part Number" "660-RN73R2ATD1001B25")
+    (property "P/N" "RN73R2ATTD1001B25")
     (property "Sheetfile" "Power_Distribution.kicad_sch")
     (property "Sheetname" "Power_Distribution")
@@
     )
   )
-  (footprint "Resistor_SMD:R_0805_2012Metric" (layer "B.Cu")
+  (footprint "Resistor_SMD:R_0603_1608Metric" (layer "B.Cu")
     (at 102.500001 77.5 180)
-    (descr "Resistor SMD 0805 (2012 Metric), square (rectangular) end terminal, IPC_7351 nominal, (Body size source: IPC-SM-782 page 72, https://www.pcb-3d.com/wordpress/wp-content/uploads/ipc-sm-782a_amendment_1_and_2.pdf), generated with kicad-footprint-generator")
+    (descr "Resistor SMD 0603 (1608 Metric), square (rectangular) end terminal, IPC_7351 nominal, (Body size source: IPC-SM-782 page 72, https://www.pcb-3d.com/wordpress/wp-content/uploads/ipc-sm-782a_amendment_1_and_2.pdf), generated with kicad-footprint-generator")
     (tags "resistor")
     (property "Field2" "")
-    (property "Mouser Part Number" "71-CRCW08051K00FKEAC")
-    (property "P/N" "CRCW08051K00FKEAC")
+    (property "Mouser Part Number" "603-RT0603BRD0747RL")
+    (property "P/N" "RT0603BRD0747RL")
     (property "Sheetfile" "Power_Distribution.kicad_sch")
     (property "Sheetname" "Power_Distribution")
@@
     (property "ki_keywords" "R res resistor")
     (attr smd)
-    (fp_text reference "R36" (at 2.500001 -0.5 90) (layer "B.SilkS")
+    (fp_text reference "R36" (at 2.400001 -0.5 90) (layer "B.SilkS")
         (effects (font (size 1 1) (thickness 0.15)) (justify mirror))
     )
-    (fp_text value "47" (at 0 -1.65) (layer "B.Fab")
+    (fp_text value "47" (at 0 -1.43) (layer "B.Fab")
         (effects (font (size 1 1) (thickness 0.15)) (justify mirror))
     )
     (fp_text user "${REFERENCE}" (at 0 0) (layer "B.Fab")
-        (effects (font (size 0.5 0.5) (thickness 0.08)) (justify mirror))
+        (effects (font (size 0.4 0.4) (thickness 0.06)) (justify mirror))
     )
-    (fp_line (start -0.227064 -0.735) (end 0.227064 -0.735)
+    (fp_line (start -0.237258 -0.5225) (end 0.237258 -0.5225)
       (stroke (width 0.12) (type solid)) (layer "B.SilkS"))
-    (fp_line (start -0.227064 0.735) (end 0.227064 0.735)
+    (fp_line (start -0.237258 0.5225) (end 0.237258 0.5225)
       (stroke (width 0.12) (type solid)) (layer "B.SilkS"))
-    (fp_line (start -1.68 -0.95) (end -1.68 0.95)
+    (fp_line (start -1.48 -0.73) (end -1.48 0.73)
       (stroke (width 0.05) (type solid)) (layer "B.CrtYd"))
-    (fp_line (start -1.68 0.95) (end 1.68 0.95)
+    (fp_line (start -1.48 0.73) (end 1.48 0.73)
       (stroke (width 0.05) (type solid)) (layer "B.CrtYd"))
-    (fp_line (start 1.68 -0.95) (end -1.68 -0.95)
+    (fp_line (start 1.48 -0.73) (end -1.48 -0.73)
       (stroke (width 0.05) (type solid)) (layer "B.CrtYd"))
-    (fp_line (start 1.68 0.95) (end 1.68 -0.95)
+    (fp_line (start 1.48 0.73) (end 1.48 -0.73)
       (stroke (width 0.05) (type solid)) (layer "B.CrtYd"))
-    (fp_line (start -1 -0.625) (end -1 0.625)
+    (fp_line (start -0.8 -0.4125) (end -0.8 0.4125)
       (stroke (width 0.1) (type solid)) (layer "B.Fab"))
-    (fp_line (start -1 0.625) (end 1 0.625)
+    (fp_line (start -0.8 0.4125) (end 0.8 0.4125)
       (stroke (width 0.1) (type solid)) (layer "B.Fab"))
-    (fp_line (start 1 -0.625) (end -1 -0.625)
+    (fp_line (start 0.8 -0.4125) (end -0.8 -0.4125)
       (stroke (width 0.1) (type solid)) (layer "B.Fab"))
-    (fp_line (start 1 0.625) (end 1 -0.625)
+    (fp_line (start 0.8 0.4125) (end 0.8 -0.4125)
       (stroke (width 0.1) (type solid)) (layer "B.Fab"))
-    (pad "1" smd roundrect (at -0.9125 0 180) (size 1.025 1.4) (layers "B.Cu" "B.Paste" "B.Mask") (roundrect_rratio 0.243902)
+    (pad "1" smd roundrect (at -0.825 0 180) (size 0.8 0.95) (layers "B.Cu" "B.Paste" "B.Mask") (roundrect_rratio 0.25)
       (net 90 "Net-(R35-Pad2)") (pintype "passive"))
-    (pad "2" smd roundrect (at 0.9125 0 180) (size 1.025 1.4) (layers "B.Cu" "B.Paste" "B.Mask") (roundrect_rratio 0.243902)
+    (pad "2" smd roundrect (at 0.825 0 180) (size 0.8 0.95) (layers "B.Cu" "B.Paste" "B.Mask") (roundrect_rratio 0.25)
       (net 2 "GND") (pintype "passive"))
-    (model "${KICAD6_3DMODEL_DIR}/Resistor_SMD.3dshapes/R_0805_2012Metric.wrl"
+    (model "${KICAD6_3DMODEL_DIR}/Resistor_SMD.3dshapes/R_0603_1608Metric.wrl"
       (offset (xyz 0 0 0))
       (scale (xyz 1 1 1))
@@
     )
   )
+  (zone (net 0) (net_name "") (layer "B.Cu") (hatch edge 0.5)
+    (connect_pads (clearance 0))
+    (min_thickness 0.25) (filled_areas_thickness no)
+    (keepout (tracks not_allowed) (vias not_allowed) (pads not_allowed) (copperpour not_allowed) (footprints allowed))
+    (fill (thermal_gap 0.5) (thermal_bridge_width 0.5))
+    (polygon
+      (pts
+        (xy 101.7 76)
+        (xy 103.1 76)
+        (xy 103.2 77.3)
+        (xy 101.7 77.3)
+      )
+    )
+  )
   (zone (net 11) (net_name "/CarCAN/+V_CAN2") (layer "B.Cu") (hatch edge 0.5)
     (priority 12)
@@
       a6a1688e-45b4-4a2e-b2a2-ac6c711d11fd
       c36099ec-ac62-487a-8188-72d00687cd99
-      c751f372-0543-4589-878e-c32c99034cdc
       cd0c5f17-1640-47a8-af7e-a93810b6a5fd
       d5478be1-42d1-4ce1-864b-639d0b80dbb4

Commit message: added 3D files and placed properly for 3D view, and added my name on rear silkscreen
Parts:
- Y2: footprint Crystal:Crystal_SMD_TXC_7A-2Pin_5x3.2mm -> UTSVT_Special:ABM3
Other:
- board text added: "Jacob Pustilnik"

Commit message: changed 12V/5V DC/DC output setting resistors to a generic 1K and 0 Ohm pair, updated LED display to proper model
Parts:
- LED1, LED2: value 157112B12800 -> 157121S12800
- R36: value 47 -> 0; footprint Resistor_SMD:R_0603_1608Metric -> Resistor_SMD:R_0805_2012Metric
Connections:
- net Net-(IC1-EN) renamed /Power_Distribution/BJT_FILTD
- net Net-(PS2-VAR) renamed /Power_Distribution/VAR
- net Net-(Q1-B) renamed /Power_Distribution/base
- net Net-(R35-Pad2) renamed /Power_Distribution/RVARdiv
Routing:
- added copper zone on In2.Cu, net +3.3VA

Commit message: 🍜
Parts:
- added G***: LOGO, LOGO, B.Cu at (107.5, 90.0)
Routing:
- net GND: vias 19 -> 25

Commit message: gonna order this
Parts:
- removed the G*** at (107.5, 90.0)
- added LOGO1: hallock, UTSVT_Special:Hallock_Image_Tiny, B.Cu at (121.0, 91.0)
- added LOGO2: car, UTSVT_Special:UTSVT_Logo_Symbol, B.Cu at (140.0, 56.5)
Connections:
- net /Power_Distribution/BJT_FILTD renamed Net-(IC1-EN)
- net /Power_Distribution/RVARdiv renamed Net-(R35-Pad2)
- net /Power_Distribution/VAR renamed Net-(PS2-VAR)
- net /Power_Distribution/base renamed Net-(Q1-B)
Other:
- board text added: "Jacob Pustilnik Pratyush Patra Tianda Huang"
- board text removed: "Jacob Pustilnik"
