File: LeaderSOM.kicad_pcb (KiCad board)
At the start: 4 copper layers, 102.2 x 60.9 mm, 136 parts, among them IC1 TCAN337DCNR, IC2 TCAN337DCNR, IC3 LM76202QPWPRQ1, J1 52465-2470, J2 52465-2470, J3 USB_C_Receptacle_USB2.0_16P, J4 Micro_SD_Card_Det, SW1 SW_SPDT, U1 CDSOT23-T24CAN, U2 CP2102N-Axx-xQFN24, U3 CDSOT23-T24CAN, U4 LT1963AEST-3.3#TRPBF, U5 TPS2115ADRBR, U6 TPS5405DR, U7 STM32G473RETx, U8 74AHC1G32, Y1 8M

Commit message: workday
Parts:
- C1, C11, C2, C4, C5, C6, C7, C8, C9: footprint Capacitor_SMD:C_0603_1608Metric -> Capacitor_SMD:C_0603_1608Metric_Pad1.08x0.95mm_HandSolder
- C10, C16, C18, C19, C21, C22, C44, D3: moved to B.Cu
- C17: moved to F.Cu
- CC_FLT1, IC_FLT1: footprint LED_SMD:LED_0603_1608Metric -> LED_SMD:LED_0603_1608Metric_Pad1.05x0.95mm_HandSolder
- R1, R10, R11, R12, R13, R15, R18, R19, R2, R20, R22, R23, R24, R25, R26, R27, R29, R3, R30, R31, R4, R5, R6, R7, R8, R9: footprint Resistor_SMD:R_0603_1608Metric -> Resistor_SMD:R_0603_1608Metric_Pad0.98x0.95mm_HandSolder
- R14, R16, R21, R28, R32: footprint Resistor_SMD:R_0603_1608Metric -> Resistor_SMD:R_0603_1608Metric_Pad0.98x0.95mm_HandSolder; moved to F.Cu
- R17: footprint Resistor_SMD:R_0603_1608Metric -> Resistor_SMD:R_0603_1608Metric_Pad0.98x0.95mm_HandSolder; moved to B.Cu
- moved C46 134.8 mm to (210.0, 81.0), turned to 90 degrees
- moved C45 134.5 mm to (212.0, 81.0), turned to 90 degrees
- moved R20 120.2 mm to (181.6, 94.0), turned to -90 degrees
- moved R18 118.6 mm to (183.3, 94.0), turned to -90 degrees
- moved C22 106.5 mm to (172.7, 109.4)
- moved R15 104.9 mm to (171.4, 96.6), turned to 90 degrees
- moved D7 102.1 mm to (164.7, 93.2), turned to -90 degrees
- moved D3 101.8 mm to (177.0, 105.0), turned to 180 degrees
- moved R17 101.8 mm to (167.6, 98.5), turned to 90 degrees
- moved C21 101.4 mm to (172.7, 107.2)
- moved C16 101.1 mm to (172.2, 99.9), turned to -90 degrees
- moved C43 100.1 mm to (179.6, 84.2), turned to 90 degrees
- moved D17 98.4 mm to (183.8, 84.2), turned to 90 degrees
- moved C44 96.8 mm to (178.3, 92.9), turned to 90 degrees
- moved L1 96.6 mm to (175.3, 110.8), turned to 180 degrees
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Connections:
- C42 pad 1: /Power_Distribution/24V_IN -> /24V_Ext
- C43 pad 1: /Power_Distribution/24V_IN -> /24V_Ext
- D17 pad 1: /Power_Distribution/24V_IN -> /24V_Ext
- IC3 pad 1: /Power_Distribution/24V_IN -> /24V_Ext
- IC3 pad 2: /Power_Distribution/24V_IN -> /24V_Ext
- R24 pad 1: /Power_Distribution/24V_IN -> /24V_Ext
Routing:
- removed copper zone on F.Cu, net +3V3
- removed copper zone on In2.Cu, net +3V3
Other:
- board size 102.2 x 60.9 mm -> 58 x 43 mm

Commit message: power layout
Parts:
- C10, C11, C12, C13, C14, C15, C16, C18, C19, C20, C21, C22, C3, C4, C44, C6, C7, D1, D3, D5, R1, R17, R2, R24, R25, R26, R27, R29, R3, R30, R31, R4, R5: moved to F.Cu
- moved R2 91.3 mm to (156.6, 76.5)
- moved R19 87.8 mm to (156.2, 111.7), turned to -90 degrees
- moved R3 85.0 mm to (160.2, 76.5)
- moved R1 79.0 mm to (163.9, 76.4)
- moved CR1 77.3 mm to (154.8, 103.7), turned to -90 degrees
- moved D5 72.1 mm to (154.5, 111.7), turned to -90 degrees
- moved IC1 69.8 mm to (159.2, 89.7)
- moved U7 44.1 mm to (164.0, 99.5), turned to -135 degrees
- moved C46 30.5 mm to (181.5, 91.8), turned to -90 degrees
- moved C45 30.4 mm to (183.6, 91.8), turned to -90 degrees
- moved R29 28.7 mm to (185.6, 91.8)
- moved R15 18.1 mm to (186.1, 107.2)
- moved GND1 17.2 mm to (173.8, 101.2)
- moved R21 15.9 mm to (180.6, 98.5), turned to 180 degrees
- moved C13 15.4 mm to (189.1, 96.2), turned to 0 degrees
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Routing:
- net /USB/VBUS_IN: track 2.14 -> 5.70 mm, vias 1 -> 0
- net +3V3: track 0.00 -> 3.40 mm
- net VBUS: track 5.32 -> 6.18 mm, vias 1 -> 0
- net /USB/CC1: track 2.94 -> 2.51 mm, vias 1 -> 0
- net /USB/CC2: track 2.81 -> 2.83 mm, vias 1 -> 0

Commit message: late night premonitions of disaster
Parts:
- C23, C24, C25, C26, C27, C28, C29, C30, C8, CR2, R23, U2: moved to F.Cu
- J4: moved to B.Cu
- SW1: footprint UTSVT_Special:SW_SPST_B3SL-1002P -> UTSVT_Special:SW_CJS-1200TA
- moved CR3 98.5 mm to (161.9, 68.2)
- moved C24 95.9 mm to (138.9, 106.4), turned to 90 degrees
- moved C26 94.9 mm to (138.9, 99.5), turned to 90 degrees
- moved C27 93.0 mm to (143.7, 109.8), turned to 90 degrees
- moved C28 89.5 mm to (143.7, 106.4)
- moved C30 89.4 mm to (143.7, 99.5)
- moved C23 86.5 mm to (138.9, 109.9), turned to 90 degrees
- moved FB2 83.6 mm to (156.1, 87.7), turned to -90 degrees
- moved FB1 82.5 mm to (157.8, 87.7), turned to 90 degrees
- moved D16 81.9 mm to (168.8, 113.9), turned to -90 degrees
- moved R8 80.8 mm to (146.2, 88.8), turned to -90 degrees
- moved C25 79.6 mm to (138.9, 103.0), turned to 90 degrees
- moved R11 78.4 mm to (151.0, 98.6)
- moved Y1 77.0 mm to (166.4, 85.1), turned to 0 degrees
- moved CR2 76.2 mm to (168.0, 67.8), turned to 180 degrees
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Routing:
- net Net-(D11-DOUT): track 0.00 -> 15.9 mm, vias 0 -> 2
- net /USB/D+: track 10.1 -> 15.6 mm, vias 1 -> 2
- net /USB/D-: track 10.1 -> 14.8 mm, vias 1 -> 2
- net +3V3: track 3.40 -> 0.00 mm
- net Net-(D8-DOUT): track 0.00 -> 2.08 mm
- net Net-(D14-DOUT): track 0.00 -> 2.08 mm
- net Net-(D10-DOUT): track 0.00 -> 2.08 mm
- net Net-(D12-DOUT): track 0.00 -> 2.07 mm
- net Net-(D13-DOUT): track 0.00 -> 2.06 mm
- net Net-(D10-DIN): track 0.00 -> 2.03 mm
Other:
- board text added: "BOOT"
- board text added: "Tony Chen Pratyush Patra"
- board text removed: "Tony Chen Pratyush Patra Tianda Huang Jacob Pustilnik"

Commit message: impending doom is approaching
Parts:
- Reset1: footprint Button_Switch_SMD:SW_SPST_B3SL-1002P -> TL3365AF180QG:TL3365AF180QG
- SWD1: footprint Connector_PinHeader_2.54mm:PinHeader_1x04_P2.54mm_Vertical -> UTSVT_Connectors:Molex_Nano-Fit_105309-xx04_1x04_P2.50mm_Vertical
- moved SWD1 108.0 mm to (126.8, 110.4), turned to 90 degrees
- moved IC_FLT1 76.1 mm to (154.4, 105.0), turned to 180 degrees
- moved R10 75.2 mm to (155.3, 103.2), turned to 180 degrees
- moved CC_Term2 71.2 mm to (166.1, 112.9), turned to -90 degrees
- moved C2 68.3 mm to (155.3, 108.1), turned to 180 degrees
- moved C1 68.1 mm to (155.3, 106.6)
- moved JP1 66.2 mm to (144.6, 83.3), turned to 90 degrees
- moved 5V1 63.8 mm to (176.3, 115.3), turned to 180 degrees
- moved C40 63.1 mm to (154.4, 118.8), turned to -90 degrees
- moved GND1 60.7 mm to (178.1, 112.3), turned to 0 degrees
- moved U1 42.6 mm to (147.2, 107.5), turned to 180 degrees
- moved Reset1 40.5 mm to (158.9, 117.9)
- moved R2 33.2 mm to (155.3, 109.7), turned to 180 degrees
- moved R1 32.9 mm to (147.6, 105.0), turned to 0 degrees
- moved R3 29.9 mm to (151.0, 105.0), turned to 0 degrees
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Other:
- board text added: "3V3"
- board text added: "5V"
- board text added: "BUCK"
- board text added: "CarCAN"
- board text added: "IntCAN"
- board text added: "RESET"
- board text added: "RPP"

Commit message: routing nightmare
Parts:
- C5: moved to F.Cu
- IC1, IC2: moved to B.Cu
- moved C37 101.8 mm to (171.7, 98.9), turned to -90 degrees
- moved C35 89.2 mm to (155.4, 91.5), turned to 90 degrees
- moved C36 88.9 mm to (159.5, 101.7), turned to 180 degrees
- moved C5 86.5 mm to (154.0, 87.2), turned to 90 degrees
- moved C34 76.3 mm to (170.8, 87.9)
- moved R13 73.3 mm to (147.9, 108.8), turned to 90 degrees
- moved C38 69.2 mm to (158.5, 87.2), turned to -90 degrees
- moved C39 62.2 mm to (157.0, 87.2), turned to -90 degrees
- moved CR2 45.1 mm to (163.1, 112.5)
- moved CR3 43.5 mm to (158.0, 111.6)
- moved SWD1 36.6 mm to (163.0, 105.5)
- moved CC_Term2 12.8 mm to (153.3, 114.3)
- moved CC_Term1 12.8 mm to (147.0, 114.3)
- moved CR1 12.5 mm to (147.5, 101.5), turned to 0 degrees
- moved U1 8.50 mm to (155.8, 107.7)
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Routing:
- net +5V: track 0.00 -> 79.0 mm, vias 0 -> 16
- net +3V3: track 0.00 -> 41.8 mm, vias 0 -> 18
- net +24V: track 0.00 -> 30.3 mm, vias 0 -> 2
- net /MCU/BOOT: track 0.00 -> 29.6 mm, vias 0 -> 2
- net /MCU/BOOT_GPIO: track 0.00 -> 26.8 mm, vias 0 -> 2
- net VBUS: track 6.18 -> 32.0 mm, vias 0 -> 2
- net /Power_Distribution/Power Protection/RTN: track 0.00 -> 19.7 mm
- net /MCU/IntCAN_L: track 0.00 -> 18.8 mm, vias 0 -> 1
- net /MCU/OSC_OUT: track 0.00 -> 12.1 mm, vias 0 -> 2
- net /Power_Distribution/FAULT: track 0.00 -> 11.6 mm, vias 0 -> 2
- net /MCU/OSC_IN: track 0.00 -> 11.4 mm, vias 0 -> 2
- net /Power_Distribution/Power Protection/IMON: track 0.00 -> 8.68 mm, vias 0 -> 2
- net Net-(IC3-ILIM): track 0.00 -> 8.41 mm, vias 0 -> 2
- net /IMON: track 0.00 -> 8.23 mm
- net /USB/VBUS_IN: track 5.70 -> 13.7 mm
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- added copper zone on F.Cu, net +24V
- added copper zone on F.Cu, net +3V3
- added copper zone on In1.Cu, net +3V3
- added copper zone on F.Cu, net +5V
- added copper zone on In1.Cu, net +5V
- added copper zone on B.Cu, net +5V_BUCK
- added copper zone on F.Cu, net +5V_BUCK
- added copper zone on F.Cu, net /24V_Ext
- added copper zone on F.Cu, net Net-(D3-K)
- added copper zone on F.Cu, net VBUS
- removed copper zone on B.Cu, net GND
- removed copper zone on In1.Cu, net GND
Other:
- board text removed: "12V"
- board text removed: "FLT"
- board text removed: "LED"
