File: USB.kicad_sch (KiCad schematic)
At the start: 8 parts, among them J2 USB_B_Micro, U3 CP2102N-A02-GQFN24

Commit message: Updated schem for redesign
Parts:
- removed C18: 4.7uF, Capacitor_SMD:C_0805_2012Metric, symbol Device:C
- removed C19: 100nF, Capacitor_SMD:C_0805_2012Metric, symbol Device:C
- removed J2: USB_B_Micro, Connector_USB:USB_Micro-B_Molex-105017-0001, symbol utsvt-connectors:USB_B_Micro-Connector
- removed R5: 22.1k, Resistor_SMD:R_0805_2012Metric, symbol Device:R
- removed R6: 47.5k, Resistor_SMD:R_0805_2012Metric, symbol Device:R
- removed R8: 1k, Resistor_SMD:R_0805_2012Metric, symbol Device:R
- removed U3: CP2102N-A02-GQFN24, Package_DFN_QFN:QFN-24-1EP_4x4mm_P0.5mm_EP2.6x2.6mm, symbol utsvt-chips:CP2102N-A01-GQFN24
- added C1, C16, C20, C22: 100nF, Capacitor_SMD:C_0805_2012Metric, symbol Device:C
- added C21, C25: 47pF, Capacitor_SMD:C_0805_2012Metric, symbol Device:C
- added J6: USB_B_Micro, Connector_USB:USB_Micro-B_Molex-105017-0001, symbol Connector:USB_B_Micro
- added R15, R9: 27, Resistor_SMD:R_0805_2012Metric, symbol Device:R
- added R35: 4.7k, Resistor_SMD:R_0805_2012Metric, symbol Device:R
- added R44: 10k, Resistor_SMD:R_0805_2012Metric, symbol Device:R
- added U1: FT230XS-R, Package_SO:SSOP-16_3.9x4.9mm_P0.635mm, symbol utsvt-chips:FT230XS-R
Connections:
- net +3.3V: now also C1.1, C16.1, C20.1, C22.1, U1.10 (3V3OUT), U1.11 (RESET), U1.12 (VCC), U1.3 (VCCIO)
- net GND: now also C1.2, C16.2, C20.2, C21.2, C22.2, C25.2, J6.5 (GND), J6.6 (Shield), R44.2, U1.13 (AGND), U1.5 (GND)
- net UART_RX: now also U1.1 (TXD)
- net UART_TX: now also U1.4 (RXD)
- net vbus: now reaches D1.2 (K)
- net vbus: now also J6.1 (VBUS), R35.1
- net D+: now reaches D1.3 (K)
- net D+: now also C25.1, J6.3 (D+), R9.2
- net D-: now reaches D1.4 (K)
- net D-: now also C21.1, J6.2 (D-), R15.2
- new net: R15.1, U1.9 (USBDM)
- new net: R35.2, R44.1, U1.16 (CBUS3)
- new net: R9.1, U1.8 (USBDP)
- no-connect marks 13 -> 6
Other:
- note added: "Used for sensing presence of USB cable"
- note removed: "From BPS Peripheral SOM"
- moved on the sheet: D1
