File: USB.kicad_sch (KiCad schematic)
At the start: 13 parts, among them J6 USB_B_Micro, U1 FT230XS-R

Commit message: hi again lakshay
Parts:
- removed C1, C16, C20, C22: 100nF, Capacitor_SMD:C_0805_2012Metric, symbol Device:C
- removed C21: 47pF, Capacitor_SMD:C_0805_2012Metric, symbol Device:C
- removed D1: SP0503BAHT, Package_TO_SOT_SMD:SOT-143, symbol utsvt-chips:SP0503BAHT-Power_Protection
- removed J6: USB_B_Micro, Connector_USB:USB_Micro-B_Molex-105017-0001, symbol Connector:USB_B_Micro
- removed R15, R9: 27, Resistor_SMD:R_0805_2012Metric, symbol Device:R
- removed R44: 10k, Resistor_SMD:R_0805_2012Metric, symbol Device:R
- removed U1: FT230XS-R, Package_SO:SSOP-16_3.9x4.9mm_P0.635mm, symbol utsvt-chips:FT230XS-R
- added C41: 4.7uF, Capacitor_SMD:C_0805_2012Metric, symbol Device:C
- added C42: 0.1uF, Capacitor_SMD:C_0805_2012Metric, symbol Device:C
- added D11: D_Schottky, Diode_SMD:D_SOD-323_HandSoldering, symbol Device:D_Schottky
- added D8: SP0503BAHT, Package_TO_SOT_SMD:SOT-143, symbol utsvt-chips:SP0503BAHT-Power_Protection
- added J6: USB_C_Receptacle_USB2.0_16P, Connector_USB:USB_C_Receptacle_GCT_USB4105-xx-A_16P_TopMnt_Horizontal, symbol Connector:USB_C_Receptacle_USB2.0_16P
- added JP3: CC_TX_RX, Connector_PinHeader_2.54mm:PinHeader_1x02_P2.54mm_Vertical, symbol Jumper:Jumper_2_Open
- added R39: 5.1k, Resistor_SMD:R_0805_2012Metric, symbol Device:R
- added R45: 22.1k, Resistor_SMD:R_0805_2012Metric, symbol Device:R
- added R46: 47.5k, Resistor_SMD:R_0805_2012Metric, symbol Device:R
- added R47: 1k, Resistor_SMD:R_0805_2012Metric, symbol Device:R
- added U19: CP2102N-A02-GQFN24, Package_DFN_QFN:QFN-24-1EP_4x4mm_P0.5mm_EP2.6x2.6mm, symbol Interface_USB:CP2102N-A01-GQFN24
- C25: value 47pF -> 10uF; Mouser Part Number (none) -> 581-22201C106KAT2A; P/N (none) -> TMK212BBJ106MGHT
- R35: value 4.7k -> 5.1k
Connections:
- net vbus is gone; now on net GND: R35.1
- net D+: now also D8.2 (K), J6.A6 (D+), J6.B6 (D+), U19.3 (D+); no longer C25.1
- net D-: now also D8.3 (K), J6.A7 (D-), J6.B7 (D-), U19.4 (D-)
- net GND: now also C41.2, C42.2, D8.1 (A), J6.A1 (GND), J6.A12 (GND), J6.B1 (GND), J6.B12 (GND), J6.S1 (SHIELD), R39.1, R46.2, U19.2 (GND), U19.25 (GND)
- net CC1: now reaches R35.2
- net CC1: now also J6.A5 (CC1)
- new net: R45.1, R46.1, U19.8 (VBUS)
- new net: R47.2, U19.9 (~{RSTb})
- new net +3V3: C41.1, C42.1, R47.1, U19.5 (VIO), U19.6 (VDD), U19.7 (REGIN)
- new net CC2: J6.B5 (CC2), R39.2
- new net CHIP_RX: JP3.1 (A), U19.20 (RXD)
- new net CHIP_TX: JP3.2 (B), U19.21 (TXD)
- new net VBUS: C25.1, D11.1 (K), D8.4 (K), R45.2
- new net vbus_in: D11.2 (A), J6.A4 (VBUS), J6.A9 (VBUS), J6.B4 (VBUS), J6.B9 (VBUS)
- no-connect marks 6 -> 14
Other:
- note added: "Pulldowns for 5V USB-C PD"
- note removed: "The microcontroller should have Rx connected to UART_TX and Tx connected to UART_RX"
- note removed: "Used for sensing presence of USB cable"

Commit message: MCU pins, PSON power distribution, KiCad-Sharepoint, and 7 seg
Parts:
- removed U19: CP2102N-A02-GQFN24, Package_DFN_QFN:QFN-24-1EP_4x4mm_P0.5mm_EP2.6x2.6mm, symbol Interface_USB:CP2102N-A01-GQFN24
- added C43: 4.7uF, Capacitor_SMD:C_0805_2012Metric, symbol Device:C
- added C44: 0.1uF, Capacitor_SMD:C_0805_2012Metric, symbol Device:C
- added U7: CP2102N-Axx-xQFN24, UTSVT_ICs:CP2102N-A02-GQFN24, symbol UTSVT-ICs:CP2102N-Axx-xQFN24
- D8: symbol utsvt-chips:SP0503BAHT-Power_Protection -> UTSVT-ICs:SP0503BAH
- J6: footprint Connector_USB:USB_C_Receptacle_GCT_USB4105-xx-A_16P_TopMnt_Horizontal -> UTSVT_ICs:USB_C_Receptacle_GCT_USB4105-xx-A_16P_TopMnt_Horizontal; symbol Connector:USB_C_Receptacle_USB2.0_16P -> UTSVT-Connectors:USB_C_Receptacle_USB2.0_16P
Connections:
- net +3V3: now also C43.1, C44.1, U7.5 (VIO), U7.6 (VDD), U7.7 (VREGIN)
- net CHIP_RX: now also U7.21 (TXD)
- net CHIP_TX: now also U7.20 (RXD)
- net D+: now also U7.4 (D-)
- net D-: now also U7.3 (D+)
- net GND: now also C25.1, J6.S2 (Shield), J6.S3 (Shield), J6.S4 (Shield), C43.2, C44.2; no longer C25.2
- net VBUS: now also C25.2; no longer C25.1
- net at R45.1, R46.1: now also U7.8 (VBUS)
- net at R47.2: now also U7.9 (~{RST})
- net vbus_in renamed VBUS_IN
- new net: U7.2 (GND), U7.25 (GND)
Other:
- note added: "UART_TX -> MCU_RX UART_RX <- MCU_TX"
- note added: "USB <-> UART"
- note added: "USB Protection"
- note added: "USB-C Port"
- note added: "VDD Bypass"
- note added: "VREGIN Bypass"
- moved on the sheet: C25, C41, C42, D11, D8, JP3, R35, R39, R45, R46, R47

Commit message: net class fixes and ERC
Connections:
- net GND: now also U7.2 (GND), U7.25 (GND)
Changed lines of the file:
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@@
+	)
+	(junction
+		(at 74.295 35.56)
+		(diameter 0)
+		(color 0 0 0 0)
 	)
 	(junction
@@
 	)
 	(symbol
+		(lib_id "power:PWR_FLAG")
+		(at 74.295 35.56 270)
+		(unit 1)
+		(exclude_from_sim no)
+		(in_bom yes)
+		(on_board yes)
+		(dnp no)
+		(fields_autoplaced yes)
+		(property "Reference" "#FLG011"
+			(at 76.2 35.56 0)
+			(effects
+				(font
+					(size 1.27 1.27)
+				)
+				(hide yes)
+			)
+		)
+		(property "Value" "PWR_FLAG"
+			(at 77.47 35.56 90)
+			(effects
+				(font
+					(size 1.27 1.27)
+				)
+				(justify left)
+			)
+		)
+		(property "Footprint" ""
+			(at 74.295 35.56 0)
+			(effects
+				(font
+					(size 1.27 1.27)
+				)
+				(hide yes)
+			)
+		)
+		(property "Datasheet" "~"
+			(at 74.295 35.56 0)
+			(effects
+				(font
+					(size 1.27 1.27)
+				)
+				(hide yes)
+			)
+		)
+		(property "Description" "Special symbol for telling ERC where power comes from"
+			(at 74.295 35.56 0)
+			(effects
+				(font
+					(size 1.27 1.27)
+				)
+				(hide yes)
+			)
+		)
+		(pin "1"
+		)
+		(instances
+			(project "LeaderSOM"
+				(path "/192d0c36-944e-4927-949b-263b8c85a7ca/5bc03b31-fe77-4b0c-be7c-10fb7ad1c047"
+					(reference "#FLG011")
+					(unit 1)
+				)
+			)
+		)
+	)
+	(symbol
 		(lib_id "Device:R")
 		(at 130.81 36.195 0)
@@
 					(unit 1)
 				)
+			)
+		)
+	)
+	(symbol
+		(lib_id "power:GND")
+		(at 147.32 90.805 0)
+		(unit 1)
+		(exclude_from_sim no)
+		(in_bom yes)
+		(on_board yes)
+		(dnp no)
+		(property "Reference" "#PWR0123"
+			(at 147.32 97.155 0)
+			(effects
+				(font
+					(size 1.27 1.27)
+				)
+				(hide yes)
+			)
+		)
+		(property "Value" "GND"
+			(at 147.447 95.1992 0)
+			(effects
+				(font
+					(size 1.27 1.27)
+				)
+			)
+		)
+		(property "Footprint" ""
+			(at 147.32 90.805 0)
+			(effects
+				(font
+					(size 1.27 1.27)
+				)
+				(hide yes)
+			)
+		)
+		(property "Datasheet" ""
+			(at 147.32 90.805 0)
+			(effects
+				(font
+					(size 1.27 1.27)
+				)
+				(hide yes)
+			)
+		)
+		(property "Description" "Power symbol creates a global label with name \"GND\" , ground"
+			(at 147.32 90.805 0)
+			(effects
+				(font
+					(size 1.27 1.27)
+				)
+				(hide yes)
+			)
+		)
+		(pin "1"
+		)
+		(instances
+			(project "LeaderSOM"
+				(path "/192d0c36-944e-4927-949b-263b8c85a7ca/5bc03b31-fe77-4b0c-be7c-10fb7ad1c047"
+					(reference "#PWR0123")
+					(unit 1)
+				)

Commit message: workday for review
Parts:
- J6: footprint UTSVT_ICs:USB_C_Receptacle_GCT_USB4105-xx-A_16P_TopMnt_Horizontal -> UTSVT_Connectors:USB_C_Receptacle_GCT_USB4105-xx-A_16P_TopMnt_Horizontal
Changed lines of the file:
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@@
 			)
 		)
-		(property "Footprint" "UTSVT_ICs:USB_C_Receptacle_GCT_USB4105-xx-A_16P_TopMnt_Horizontal"
+		(property "Footprint" "UTSVT_Connectors:USB_C_Receptacle_GCT_USB4105-xx-A_16P_TopMnt_Horizontal"
 			(at 44.45 50.8 0)
 			(effects

Commit message: macbook hater
Connections:
- net D+: no longer U7.4 (D-)
- net D-: no longer U7.3 (D+)
Changed lines of the file:
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@@
 		)
 	)
-	(label "D-"
-		(at 130.81 57.785 0)
+	(label "CC2"
+		(at 67.31 72.39 0)
 		(effects
 			(font
@@
 		)
 	)
-	(label "CC2"
-		(at 67.31 72.39 0)
+	(label "D-"
+		(at 130.81 48.26 0)
 		(effects
 			(font
@@
 	)
 	(label "D+"
-		(at 131.445 55.245 0)
+		(at 130.81 50.8 0)
 		(effects
 			(font

Commit message: review council
Connections:
- net D+: now also U7.3 (D+)
- net D-: now also U7.4 (D-)
Changed lines of the file:
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@@
 	(wire
 		(pts
-			(xy 130.81 57.785) (xy 134.62 57.785)
+			(xy 131.445 57.785) (xy 134.62 57.785)
 		)
 		(stroke
@@
 		)
 	)
-	(label "D-"
-		(at 130.81 48.26 0)
-		(effects
-			(font
-				(size 1.27 1.27)
-			)
-			(justify left bottom)
-		)
-	)
 	(label "CC2"
 		(at 60.96 43.18 180)
@@
 	)
 	(label "D+"
-		(at 130.81 50.8 0)
+		(at 131.445 57.785 0)
 		(effects
 			(font
@@
 		)
 	)
+	(label "D-"
+		(at 131.445 55.245 0)
+		(effects
+			(font
+				(size 1.27 1.27)
+			)
+			(justify left bottom)
+		)
+	)

Commit message: crazy? i used to be crazy
Parts:
- C4: renamed from C41; footprint Capacitor_SMD:C_0805_2012Metric -> Capacitor_SMD:C_0603_1608Metric
- C5: renamed from C43; footprint Capacitor_SMD:C_0805_2012Metric -> Capacitor_SMD:C_0603_1608Metric
- C6: renamed from C42; footprint Capacitor_SMD:C_0805_2012Metric -> Capacitor_SMD:C_0603_1608Metric
- C7: renamed from C44; footprint Capacitor_SMD:C_0805_2012Metric -> Capacitor_SMD:C_0603_1608Metric
- R4: renamed from R35; footprint Resistor_SMD:R_0805_2012Metric -> Resistor_SMD:R_0603_1608Metric
- R5: renamed from R39; footprint Resistor_SMD:R_0805_2012Metric -> Resistor_SMD:R_0603_1608Metric
- R6: renamed from R45; footprint Resistor_SMD:R_0805_2012Metric -> Resistor_SMD:R_0603_1608Metric
- R7: renamed from R46; footprint Resistor_SMD:R_0805_2012Metric -> Resistor_SMD:R_0603_1608Metric
- R8: renamed from R47; footprint Resistor_SMD:R_0805_2012Metric -> Resistor_SMD:R_0603_1608Metric
- renumbered C25 to C3, D11 to D1, D8 to D2, J6 to J3, JP3 to JP1, U7 to U2
Connections:
- net D+: now also D2.3 (K); no longer D2.2 (K)
- net D-: now also D2.2 (K); no longer D2.3 (K)
