File: USB.kicad_sch (KiCad schematic)
At the start: 15 parts, among them J3 USB_C_Receptacle_USB2.0_16P, U2 CP2102N-Axx-xQFN24

Commit message: workday
Parts:
- C4, C5, C6, C7: footprint Capacitor_SMD:C_0603_1608Metric -> Capacitor_SMD:C_0603_1608Metric_Pad1.08x0.95mm_HandSolder
- R4, R5, R6, R7, R8: footprint Resistor_SMD:R_0603_1608Metric -> Resistor_SMD:R_0603_1608Metric_Pad0.98x0.95mm_HandSolder
Changed lines of the file:
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@@
 			)
 		)
-		(property "Footprint" "Capacitor_SMD:C_0603_1608Metric"
+		(property "Footprint" "Capacitor_SMD:C_0603_1608Metric_Pad1.08x0.95mm_HandSolder"
 			(at 184.4802 39.37 0)
 			(effects
@@
 			)
 		)
-		(property "Footprint" "Capacitor_SMD:C_0603_1608Metric"
+		(property "Footprint" "Capacitor_SMD:C_0603_1608Metric_Pad1.08x0.95mm_HandSolder"
 			(at 197.1802 39.37 0)
 			(effects
@@
 			)
 		)
-		(property "Footprint" "Resistor_SMD:R_0603_1608Metric"
+		(property "Footprint" "Resistor_SMD:R_0603_1608Metric_Pad0.98x0.95mm_HandSolder"
 			(at 65.913 76.2 90)
 			(effects
@@
 			)
 		)
-		(property "Footprint" "Capacitor_SMD:C_0603_1608Metric"
+		(property "Footprint" "Capacitor_SMD:C_0603_1608Metric_Pad1.08x0.95mm_HandSolder"
 			(at 184.4802 62.23 0)
 			(effects
@@
 			)
 		)
-		(property "Footprint" "Resistor_SMD:R_0603_1608Metric"
+		(property "Footprint" "Resistor_SMD:R_0603_1608Metric_Pad0.98x0.95mm_HandSolder"
 			(at 129.032 36.195 90)
 			(effects
@@
 			)
 		)
-		(property "Footprint" "Resistor_SMD:R_0603_1608Metric"
+		(property "Footprint" "Resistor_SMD:R_0603_1608Metric_Pad0.98x0.95mm_HandSolder"
 			(at 120.65 50.927 90)
 			(effects
@@
 			)
 		)
-		(property "Footprint" "Capacitor_SMD:C_0603_1608Metric"
+		(property "Footprint" "Capacitor_SMD:C_0603_1608Metric_Pad1.08x0.95mm_HandSolder"
 			(at 197.1802 62.23 0)
 			(effects
@@
 			)
 		)
-		(property "Footprint" "Resistor_SMD:R_0603_1608Metric"
+		(property "Footprint" "Resistor_SMD:R_0603_1608Metric_Pad0.98x0.95mm_HandSolder"
 			(at 127.762 62.865 90)
 			(effects
@@
 			)
 		)
-		(property "Footprint" "Resistor_SMD:R_0603_1608Metric"
+		(property "Footprint" "Resistor_SMD:R_0603_1608Metric_Pad0.98x0.95mm_HandSolder"
 			(at 74.168 76.2 90)
 			(effects

Commit message: lock in
Parts:
- removed JP1: CC_TX_RX, Connector_PinHeader_2.54mm:PinHeader_1x02_P2.54mm_Vertical, symbol Jumper:Jumper_2_Open
- C4, C5: footprint Capacitor_SMD:C_0603_1608Metric_Pad1.08x0.95mm_HandSolder -> Capacitor_SMD:C_0805_2012Metric
Changed lines of the file:
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@@
-	(wire
-		(pts
-			(xy 196.215 77.47) (xy 196.215 79.375)
-		)
-		(stroke
-			(width 0)
-			(type default)
-		)
-	)
 	(wire
 		(pts
@@
 	(wire
 		(pts
-			(xy 196.215 89.535) (xy 196.215 91.44)
-		)
-		(stroke
-			(width 0)
-			(type default)
-		)
-	)
-	(wire
-		(pts
 			(xy 124.46 52.705) (xy 129.54 52.705)
 		)
@@
 	(wire
 		(pts
-			(xy 192.405 91.44) (xy 196.215 91.44)
-		)
-		(stroke
-			(width 0)
-			(type default)
-		)
-	)
-	(wire
-		(pts
 			(xy 131.445 57.785) (xy 134.62 57.785)
 		)
@@
 		(pts
 			(xy 130.81 32.385) (xy 139.7 32.385)
-		)
-		(stroke
-			(width 0)
-			(type default)
-		)
-	)
-	(wire
-		(pts
-			(xy 192.405 77.47) (xy 196.215 77.47)
 		)
 		(stroke
@@
 			)
 			(justify right bottom)
-		)
-	)
-	(hierarchical_label "CHIP_TX"
-		(shape output)
-		(at 192.405 77.47 180)
-		(effects
-			(font
-				(size 1.27 1.27)
-			)
-			(justify right)
 		)
 	)
@@
 			)
 			(justify left)
-		)
-	)
-	(hierarchical_label "CHIP_RX"
-		(shape input)
-		(at 192.405 91.44 180)
-		(effects
-			(font
-				(size 1.27 1.27)
-			)
-			(justify right)
 		)
 	)
@@
 			)
 		)
-		(property "Footprint" "Capacitor_SMD:C_0603_1608Metric_Pad1.08x0.95mm_HandSolder"
+		(property "Footprint" "Capacitor_SMD:C_0805_2012Metric"
 			(at 184.4802 39.37 0)
 			(effects
@@
 			)
 		)
-		(property "Footprint" "Capacitor_SMD:C_0603_1608Metric_Pad1.08x0.95mm_HandSolder"
+		(property "Footprint" "Capacitor_SMD:C_0805_2012Metric"
 			(at 184.4802 62.23 0)
 			(effects
@@
 					(unit 1)
 				)
-			)
-		)
-	)
-	(symbol
-		(lib_id "Jumper:Jumper_2_Open")
-		(at 196.215 84.455 90)
-		(unit 1)
-		(exclude_from_sim yes)
-		(in_bom yes)
-		(on_board yes)
-		(dnp no)
-		(property "Reference" "JP1"
-			(at 198.247 84.582 0)
-			(effects
-				(font
-					(size 1.27 1.27)
-				)
-			)
-		)
-		(property "Value" "CC_TX_RX"
-			(at 200.787 84.582 0)
-			(effects
-				(font
-					(size 1.27 1.27)
-				)
-			)
-		)
-		(property "Footprint" "Connector_PinHeader_2.54mm:PinHeader_1x02_P2.54mm_Vertical"
-			(at 196.215 84.455 0)
-			(effects
-				(font
-					(size 1.27 1.27)
-				)
-				(hide yes)
-			)
-		)
-		(property "Datasheet" "~"
-			(at 196.215 84.455 0)
-			(effects
-				(font
-					(size 1.27 1.27)
-				)
-				(hide yes)
-			)
-		)
-		(property "Description" "Jumper, 2-pole, open"
-			(at 196.215 84.455 0)
-			(effects
-				(font
-					(size 1.27 1.27)
-				)
-				(hide yes)
-			)
-		)
-		(property "PN" ""
-			(at 196.215 84.455 0)
-			(effects
-				(font
-					(size 1.27 1.27)
-				)
-				(hide yes)
-			)
-		)
-		(property "p/n" ""
-			(at 196.215 84.455 0)
-			(effects
-				(font
-					(size 1.27 1.27)
-				)
-				(hide yes)
-			)
-		)
-		(pin "2"
-		)
-		(pin "1"
-		)
-		(instances
-			(project "LeaderSOM"
-				(path "/192d0c36-944e-4927-949b-263b8c85a7ca/5bc03b31-fe77-4b0c-be7c-10fb7ad1c047"
-					(reference "JP1")
-					(unit 1)
-				)

Commit message: JLCPCB BOM and gerbers
Parts:
- D1: footprint Diode_SMD:D_SOD-323_HandSoldering -> Diode_SMD:D_SOD-123
Changed lines of the file:
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@@
 			)
 		)
-		(property "Footprint" "Diode_SMD:D_SOD-323_HandSoldering"
+		(property "Footprint" "Diode_SMD:D_SOD-123"
 			(at 67.31 35.56 0)
 			(effects

Commit message: bom
Parts:
- C3: Mouser Part Number 581-22201C106KAT2A -> GRM21BR61H106KE43K
- C4, C5: Mouser Part Number 81-GRM219R6YA475KA3D -> 08055D475KAT4A
- C6, C7: Mouser Part Number 80-C0805C104M5R -> MLASH168SB7104KTNA01
- D1: Mouser Part Number (none) -> 1N5819HW-7-F
- J3: Mouser Part Number (none) -> 640-USB4105-GF-A
- R4, R5: Mouser Part Number (none) -> CRCW06035K10FKEC
- R6: Mouser Part Number 71-CRCW0805-22.1K-E3 -> CRCW060322K1FKEBC
- R7: Mouser Part Number 71-CRCW0805-47.5K-E3 -> CRCW060347K5FKEAHP
- R8: Mouser Part Number 71-CRCW08051K00FKEAC -> CRCW06031K00FKEI
- U2: Mouser Part Number (none) -> CP2102N-A02-GQFN24
Changed lines of the file:
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@@
 			)
 		)
-		(property "Mouser Part Number" "81-GRM219R6YA475KA3D"
+		(property "Mouser Part Number" "08055D475KAT4A"
 			(at 183.515 35.56 0)
 			(effects
@@
 			)
 		)
-		(property "Mouser Part Number" "80-C0805C104M5R"
+		(property "Mouser Part Number" "MLASH168SB7104KTNA01"
 			(at 196.215 35.56 0)
 			(effects
@@
 			)
 		)
+		(property "Mouser Part Number" "CRCW06035K10FKEC "
+			(at 64.135 76.2 0)
+			(effects
+				(font
+					(size 1.27 1.27)
+				)
+			)
+		)
 		(pin "1"
 		)
@@
 			)
 		)
-		(property "Mouser Part Number" "81-GRM219R6YA475KA3D"
+		(property "Mouser Part Number" "08055D475KAT4A"
 			(at 183.515 58.42 0)
 			(effects
@@
 			)
 		)
+		(property "Mouser Part Number" "CP2102N-A02-GQFN24"
+			(at 147.32 62.865 0)
+			(effects
+				(font
+					(size 1.27 1.27)
+				)
+			)
+		)
 		(pin "3"
 		)
@@
 			)
 		)
-		(property "Mouser Part Number" "71-CRCW08051K00FKEAC"
+		(property "Mouser Part Number" "CRCW06031K00FKEI "
 			(at 130.81 36.195 0)
 			(effects
@@
 			)
 		)
-		(property "Mouser Part Number" "581-22201C106KAT2A"
+		(property "Mouser Part Number" "GRM21BR61H106KE43K"
 			(at 71.12 41.275 0)
 			(effects
@@
 			)
 		)
-		(property "Mouser Part Number" "71-CRCW0805-22.1K-E3"
+		(property "Mouser Part Number" "CRCW060322K1FKEBC "
 			(at 120.65 52.705 0)
 			(effects
@@
 			)
 		)
-		(property "Mouser Part Number" "80-C0805C104M5R"
+		(property "Mouser Part Number" "MLASH168SB7104KTNA01"
 			(at 196.215 58.42 0)
 			(effects
@@
 			)
 		)
-		(property "Mouser Part Number" "71-CRCW0805-47.5K-E3"
+		(property "Mouser Part Number" "CRCW060347K5FKEAHP "
 			(at 129.54 62.865 0)
 			(effects
@@
 			)
 		)
+		(property "Mouser Part Number" "1N5819HW-7-F"
+			(at 67.31 35.56 0)
+			(effects
+				(font
+					(size 1.27 1.27)
+				)
+			)
+		)
 		(pin "2"
 		)
@@
 		)
 		(property "Vf" ""
+			(at 72.39 76.2 0)
+			(effects
+				(font
+					(size 1.27 1.27)
+				)
+			)
+		)
+		(property "Mouser Part Number" "CRCW06035K10FKEC "
 			(at 72.39 76.2 0)
 			(effects
@@
 			(at 40.64 50.8 0)
 			(effects
+				(font
+					(size 1.27 1.27)
+				)
+			)
+		)
+		(property "Mouser Part Number" "640-USB4105-GF-A"
+			(at 40.64 50.8 0)
+			(effects

Commit message: revB for assembly stuff
Parts:
- renumbered C5 to C4, C7 to C5, C4 to C6, C6 to C7
Changed lines of the file:
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@@
 		(on_board yes)
 		(dnp no)
-		(property "Reference" "C4"
+		(property "Reference" "C6"
 			(at 186.436 34.3916 0)
 			(effects
@@
 			(project "LeaderSOM"
 				(path "/192d0c36-944e-4927-949b-263b8c85a7ca/5bc03b31-fe77-4b0c-be7c-10fb7ad1c047"
-					(reference "C4")
+					(reference "C6")
 					(unit 1)
 				)
@@
 		(on_board yes)
 		(dnp no)
-		(property "Reference" "C6"
+		(property "Reference" "C7"
 			(at 199.136 34.3916 0)
 			(effects
@@
 			(project "LeaderSOM"
 				(path "/192d0c36-944e-4927-949b-263b8c85a7ca/5bc03b31-fe77-4b0c-be7c-10fb7ad1c047"
-					(reference "C6")
+					(reference "C7")
 					(unit 1)
 				)
@@
 		(on_board yes)
 		(dnp no)
-		(property "Reference" "C5"
+		(property "Reference" "C4"
 			(at 186.436 57.2516 0)
 			(effects
@@
 			(project "LeaderSOM"
 				(path "/192d0c36-944e-4927-949b-263b8c85a7ca/5bc03b31-fe77-4b0c-be7c-10fb7ad1c047"
-					(reference "C5")
+					(reference "C4")
 					(unit 1)
 				)
@@
 		(on_board yes)
 		(dnp no)
-		(property "Reference" "C7"
+		(property "Reference" "C5"
 			(at 199.136 57.2516 0)
 			(effects
@@
 			(project "LeaderSOM"
 				(path "/192d0c36-944e-4927-949b-263b8c85a7ca/5bc03b31-fe77-4b0c-be7c-10fb7ad1c047"
-					(reference "C7")
+					(reference "C5")
 					(unit 1)
 				)

Commit message: updated pins
Parts:
- removed C4, C6: 4.7uF, Capacitor_SMD:C_0805_2012Metric, symbol Device:C
- removed C5, C7: 0.1uF, Capacitor_SMD:C_0603_1608Metric_Pad1.08x0.95mm_HandSolder, symbol Device:C
- removed R6: 22.1k, Resistor_SMD:R_0603_1608Metric_Pad0.98x0.95mm_HandSolder, symbol Device:R
- removed R7: 47.5k, Resistor_SMD:R_0603_1608Metric_Pad0.98x0.95mm_HandSolder, symbol Device:R
- removed R8: 1k, Resistor_SMD:R_0603_1608Metric_Pad0.98x0.95mm_HandSolder, symbol Device:R
- removed U2: CP2102N-Axx-xQFN24, UTSVT_ICs:CP2102N-A02-GQFN24, symbol UTSVT-ICs:CP2102N-Axx-xQFN24
Connections:
- net D+ renamed USB_D+
- net D- renamed USB_D-
- no-connect marks 14 -> 2
Other:
- note removed: "UART_TX -> MCU_RX UART_RX <- MCU_TX"
- note removed: "USB <-> UART"
- note removed: "VDD Bypass"
- note removed: "VREGIN Bypass"
- moved on the sheet: C3, D2, R4
