File: Power_Protection.kicad_sch (KiCad schematic)
At the start: 19 parts, among them IC3 LM76202QPWPRQ1

Commit message: ahahahahsaofiwqihfwqof
Parts:
- 24V2: now left out of the parts list

Commit message: JLCPCB BOM and gerbers
Parts:
- GND1: now left out of the parts list

Commit message: bom
Parts:
- C42, C45: value 10u -> 10uF; Mouser Part Number (none) -> GRM21BR61H106KE43K
- C43, C46: value 1u -> 1uF; Mouser Part Number (none) -> MLASU168SB5105KTNA01
- C44: value 100nF -> 0.1uF; Mouser Part Number 80-C0805C104M5R -> MLASH168SB7104KTNA01
- D18: Mouser Part Number (none) -> MP01EA06
- R24: Mouser Part Number (none) -> CRCW060345K3FKEAHP
- R25: Mouser Part Number (none) -> CRCW0603590RFKEA
- R26: Mouser Part Number (none) -> CRCW06032K10FKEA
- R27: Mouser Part Number (none) -> CRCW0603402KFKEAC
- R28, R30: Mouser Part Number 71-CRCW080510K0FKEAC -> CRCW060310K0FKEI
- R29: Mouser Part Number 71-CRCW0805100KFKEAC -> CRCW060310K0FKEI
- R31: Mouser Part Number (none) -> CRCW060320K0FKEA
