File: Power_Protection.kicad_sch (KiCad schematic)
At the start: 19 parts, among them IC3 LM76202QPWPRQ1

Commit message: revB for assembly stuff
Parts:
- removed D18: TVS, Diode_SMD:D_SOD-123F, symbol Device:D_Zener
- removed R28: 10K, Resistor_SMD:R_0603_1608Metric_Pad0.98x0.95mm_HandSolder, symbol Device:R
- removed R32: 100k, Resistor_SMD:R_0603_1608Metric_Pad0.98x0.95mm_HandSolder, symbol Device:R
- R31: Mouser Part Number CRCW060320K0FKEA -> (none); P/N WFCP0603R0240FE66 -> (none)
Connections:
- no-connect marks 2 -> 3
Other:
- note added: "Got rid of current monitoring for an onboard led just leaving it here in case"
- note removed: "Current Monitoring"
- note removed: "DNP until validated"
- note removed: "Typical gain: 78.28 uA/A Vout @ 1.5A = 2.231v R(imon) = 19 kΩ"
