File: MISC.kicad_sch (KiCad schematic)
At the start: 16 parts, among them IC2 SN74AHC1G32TDBVRQ1, SW1 SW_SPDT

Commit message: mcu sheet
Parts:
- removed SWD1: SWD, Connector_PinHeader_2.54mm:PinHeader_1x04_P2.54mm_Vertical, symbol Connector_Generic:Conn_01x04
Other:
- note removed: "SWD Connector"

Commit message: macbook hater
Parts:
- added J1: ~, symbol UTSVT-Connectors:LSOM_DaughterConn
Connections:
- new net: J1.1 (+3.3V), J1.2 (+3.3V), J1.3 (+3.3V), J1.4 (+3.3V), J1.45 (+3.3V), J1.46 (+3.3V), J1.47 (+3.3V), J1.48 (+3.3V)
- new net: J1.21 (24VExt), J1.22 (24VExt), J1.23 (24VExt), J1.24 (24VExt)
- new net: J1.25 (GND), J1.26 (GND), J1.27 (GND), J1.28 (GND)
- new net: J1.37 (+3.3VA), J1.39 (+3.3VA)
- new net: J1.38 (GNDA), J1.40 (GNDA)
Changed lines of the file:
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@@
+	)
+	(symbol
+		(lib_id "UTSVT-Connectors:LSOM_DaughterConn")
+		(at 161.29 31.75 0)
+		(unit 1)
+		(exclude_from_sim no)
+		(in_bom yes)
+		(on_board yes)
+		(dnp no)
+		(fields_autoplaced yes)
+		(property "Reference" "J1"
+			(at 177.4033 92.71 0)
+			(effects
+				(font
+					(size 1.27 1.27)
+				)
+				(justify left)
+			)
+		)
+		(property "Value" "~"
+			(at 177.4033 95.25 0)
+			(effects
+				(font
+					(size 1.27 1.27)
+				)
+				(justify left)
+			)
+		)
+		(property "Footprint" ""
+			(at 161.29 31.75 0)
+			(effects
+				(font
+					(size 1.27 1.27)
+				)
+				(hide yes)
+			)
+		)
+		(property "Datasheet" "https://www.molex.com/en-us/products/part-detail/533072471"
+			(at 161.544 26.924 0)
+			(effects
+				(font
+					(size 1.27 1.27)
+				)
+				(hide yes)
+			)
+		)
+		(property "Description" "Symbol for both board-to-board connectors from the LeaderSOM"
+			(at 161.544 24.13 0)
+			(effects
+				(font
+					(size 1.27 1.27)
+				)
+				(hide yes)
+			)
+		)
+		(pin "16"
+		)
+		(pin "25"
+		)
+		(pin "37"
+		)
+		(pin "18"
+		)
+		(pin "34"
+		)
+		(pin "9"
+		)
+		(pin "11"
+		)
+		(pin "13"
+		)
+		(pin "7"
+		)
+		(pin "31"
+		)
+		(pin "29"
+		)
+		(pin "41"
+		)
+		(pin "35"
+		)
+		(pin "33"
+		)
+		(pin "44"
+		)
+		(pin "42"
+		)
+		(pin "36"
+		)
+		(pin "1"
+		)
+		(pin "38"
+		)
+		(pin "21"
+		)
+		(pin "22"
+		)
+		(pin "14"
+		)
+		(pin "23"
+		)
+		(pin "2"
+		)
+		(pin "27"
+		)
+		(pin "24"
+		)
+		(pin "15"
+		)
+		(pin "17"
+		)
+		(pin "12"
+		)
+		(pin "43"
+		)
+		(pin "10"
+		)
+		(pin "48"
+		)
+		(pin "8"
+		)
+		(pin "6"
+		)
+		(pin "32"
+		)
+		(pin "30"
+		)
+		(pin "40"
+		)
+		(pin "46"
+		)
+		(pin "47"
+		)
+		(pin "3"
+		)
+		(pin "4"
+		)
+		(pin "45"
+		)
+		(pin "19"
+		)
+		(pin "5"
+		)
+		(pin "26"
+		)
+		(pin "20"
+		)
+		(pin "39"
+		)
+		(pin "28"
+		)
+		(instances
+			(project ""
+				(path "/192d0c36-944e-4927-949b-263b8c85a7ca/4a7189ca-6f29-418f-88ee-cfefc930b205"
+					(reference "J1")
+					(unit 1)
+				)
+			)
+		)
 	)
 	(symbol

Commit message: review council
Parts:
- removed C15: 100nF, Capacitor_SMD:C_0805_2012Metric, symbol Device:C
- removed C29: C, Capacitor_SMD:C_0603_1608Metric, symbol Device:C
- removed D2: D_TVS, Diode_SMD:D_SOD-323, symbol Device:D_TVS
- removed IC2: SN74AHC1G32TDBVRQ1, OR_Gate:SOT95P280X145-5N, symbol OR-Gate:SN74AHC1G32TDBVRQ1
- removed R4: 10k, Resistor_SMD:R_0603_1608Metric, symbol Device:R_US
- removed Reset1: Reset, Button_Switch_SMD:SW_SPST_B3SL-1002P, symbol Switch:SW_Push
- removed SW1: SW_SPDT, UTSVT_Special:SW_SPST_B3SL-1002P, symbol Switch:SW_SPDT
- added C45, C46, C47, C48: 100nF, Capacitor_SMD:C_0603_1608Metric_Pad1.08x0.95mm_HandSolder, symbol Device:C
- added D15, D18, D19, D7: WS2812B-2020, LED_SMD:LED_WS2812B-2020_PLCC4_2.0x2.0mm, symbol LED:WS2812B-2020
- added J?: 53307-2471, UTSVT_Connectors:PeripheralSOM, symbol UTSVT-Connectors:PeripheralSOMConnector
Connections:
- net GND: now also C45.2, C46.2, C47.2, C48.2, D15.2 (VSS), D18.2 (VSS), D19.2 (VSS), D7.2 (VSS)
- net at D17.1 (DOUT): now also D7.3 (DIN)
- net +3V3 renamed +5V
- net +5V: now also C45.1, C46.1, C47.1, C48.1, D15.4 (VDD), D18.4 (VDD), D19.4 (VDD), D7.4 (VDD)
- new net: D15.3 (DIN), D7.1 (DOUT)
- new net: D18.1 (DOUT), D19.3 (DIN)
- new net: D15.1 (DOUT), D18.3 (DIN)
- no-connect marks 1 -> 0
Other:
- note removed: "Boot Switch"
- note removed: "Buttons & Stuff"
- note removed: "Reset Button"

Commit message: review council stuff
Parts:
- removed J1: ~, symbol UTSVT-Connectors:LSOM_DaughterConn
- removed J?: 53307-2471, UTSVT_Connectors:PeripheralSOM, symbol UTSVT-Connectors:PeripheralSOMConnector
- added C49, C50, C51, C52, C53, C54, C55, C56: 100nF, Capacitor_SMD:C_0603_1608Metric_Pad1.08x0.95mm_HandSolder, symbol Device:C
- added D20, D21, D22, D23, D24, D25, D26, D27: WS2812B-2020, LED_SMD:LED_WS2812B-2020_PLCC4_2.0x2.0mm, symbol LED:WS2812B-2020
Connections:
- net +5V: now also C49.1, C50.1, C51.1, C52.1, C53.1, C54.1, C55.1, C56.1, D20.4 (VDD), D21.4 (VDD), D22.4 (VDD), D23.4 (VDD), D24.4 (VDD), D25.4 (VDD), D26.4 (VDD), D27.4 (VDD)
- net GND: now also C49.2, C50.2, C51.2, C52.2, C53.2, C54.2, C55.2, C56.2, D20.2 (VSS), D21.2 (VSS), D22.2 (VSS), D23.2 (VSS), D24.2 (VSS), D25.2 (VSS), D26.2 (VSS), D27.2 (VSS)
- net AdressableData: now reaches D19.1 (DOUT)
- net AdressableData: now also D20.3 (DIN)
- new net: D22.1 (DOUT), D23.3 (DIN)
- new net: D21.1 (DOUT), D22.3 (DIN)
- new net: D25.1 (DOUT), D26.3 (DIN)
- new net: D24.1 (DOUT), D25.3 (DIN)
- new net: D20.1 (DOUT), D21.3 (DIN)
- new net: D23.1 (DOUT), D24.3 (DIN)
- new net: D26.1 (DOUT), D27.3 (DIN)
- no-connect marks 0 -> 1
Other:
- moved on the sheet: C45, C46, C47, C48, D15, D18, D19, D7

Commit message: crazy? i used to be crazy
Parts:
- removed C49, C50, C51, C52, C53, C54, C55, C56: 100nF, Capacitor_SMD:C_0603_1608Metric_Pad1.08x0.95mm_HandSolder, symbol Device:C
- removed D20, D21, D22, D23, D24, D25, D26, D27: WS2812B-2020, LED_SMD:LED_WS2812B-2020_PLCC4_2.0x2.0mm, symbol LED:WS2812B-2020
- renumbered C32 to C23, C38 to C24, C39 to C25, C40 to C26, C45 to C27, C46 to C28, C47 to C29, C48 to C30, D16 to D10, D17 to D11, D7 to D12, D15 to D13, D18 to D14, D19 to D15, D4 to D8, D6 to D9
Connections:
- net AdressableData: no longer names the net of D15.1 (DOUT)

Commit message: workday
Parts:
- D10, D11, D12, D13, D14, D15, D8, D9: footprint LED_SMD:LED_WS2812B-2020_PLCC4_2.0x2.0mm -> UTSVT_Passive:WS2812B-2020
Changed lines of the file:
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@@
 			)
 		)
-		(property "Footprint" "LED_SMD:LED_WS2812B-2020_PLCC4_2.0x2.0mm"
+		(property "Footprint" "UTSVT_Passive:WS2812B-2020"
 			(at 103.505 46.99 0)
 			(effects
@@
 			)
 		)
-		(property "Footprint" "LED_SMD:LED_WS2812B-2020_PLCC4_2.0x2.0mm"
+		(property "Footprint" "UTSVT_Passive:WS2812B-2020"
 			(at 122.555 46.99 0)
 			(effects
@@
 			)
 		)
-		(property "Footprint" "LED_SMD:LED_WS2812B-2020_PLCC4_2.0x2.0mm"
+		(property "Footprint" "UTSVT_Passive:WS2812B-2020"
 			(at 180.34 46.99 0)
 			(effects
@@
 			)
 		)
-		(property "Footprint" "LED_SMD:LED_WS2812B-2020_PLCC4_2.0x2.0mm"
+		(property "Footprint" "UTSVT_Passive:WS2812B-2020"
 			(at 45.72 46.99 0)
 			(effects
@@
 			)
 		)
-		(property "Footprint" "LED_SMD:LED_WS2812B-2020_PLCC4_2.0x2.0mm"
+		(property "Footprint" "UTSVT_Passive:WS2812B-2020"
 			(at 83.82 46.99 0)
 			(effects
@@
 			)
 		)
-		(property "Footprint" "LED_SMD:LED_WS2812B-2020_PLCC4_2.0x2.0mm"
+		(property "Footprint" "UTSVT_Passive:WS2812B-2020"
 			(at 141.605 46.99 0)
 			(effects
@@
 			)
 		)
-		(property "Footprint" "LED_SMD:LED_WS2812B-2020_PLCC4_2.0x2.0mm"
+		(property "Footprint" "UTSVT_Passive:WS2812B-2020"
 			(at 64.77 46.99 0)
 			(effects
@@
 			)
 		)
-		(property "Footprint" "LED_SMD:LED_WS2812B-2020_PLCC4_2.0x2.0mm"
+		(property "Footprint" "UTSVT_Passive:WS2812B-2020"
 			(at 160.655 46.99 0)
 			(effects

Commit message: bom
Parts:
- C23, C24, C25, C26, C27, C28, C29, C30: value 100nF -> 0.1uF; Mouser Part Number (none) -> MLASH168SB7104KTNA01
- D10, D11, D12, D13, D14, D15, D8, D9: Mouser Part Number (none) -> WS2812-2020
Changed lines of the file:
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@@
 			)
 		)
+		(property "Mouser Part Number" "WS2812-2020"
+			(at 102.235 39.37 0)
+			(effects
+				(font
+					(size 1.27 1.27)
+				)
+			)
+		)
 		(pin "3"
 		)
@@
 		(fields_autoplaced yes)
 		(property "Reference" "C28"
-			(at 151.765 24.765 0)
+			(at 152.4 22.8599 0)
 			(effects
 				(font
@@
 			)
 		)
-		(property "Value" "100nF"
-			(at 151.765 27.305 0)
+		(property "Value" "0.1uF"
+			(at 152.4 25.3999 0)
 			(effects
 				(font
@@
 			)
 		)
+		(property "Mouser Part Number" "MLASH168SB7104KTNA01"
+			(at 152.4 27.9399 0)
+			(effects
+				(font
+					(size 1.27 1.27)
+				)
+				(justify left)
+			)
+		)
 		(pin "1"
 		)
@@
 			)
 		)
+		(property "Mouser Part Number" "WS2812-2020"
+			(at 121.285 39.37 0)
+			(effects
+				(font
+					(size 1.27 1.27)
+				)
+			)
+		)
 		(pin "3"
 		)
@@
 			)
 		)
+		(property "Mouser Part Number" "WS2812-2020"
+			(at 179.07 39.37 0)
+			(effects
+				(font
+					(size 1.27 1.27)
+				)
+			)
+		)
 		(pin "3"
 		)
@@
 			)
 		)
+		(property "Mouser Part Number" "WS2812-2020"
+			(at 44.45 39.37 0)
+			(effects
+				(font
+					(size 1.27 1.27)
+				)
+			)
+		)
 		(pin "3"
 		)
@@
 			)
 		)
+		(property "Mouser Part Number" "WS2812-2020"
+			(at 82.55 39.37 0)
+			(effects
+				(font
+					(size 1.27 1.27)
+				)
+			)
+		)
 		(pin "3"
 		)
@@
 			)
 		)
+		(property "Mouser Part Number" "WS2812-2020"
+			(at 140.335 39.37 0)
+			(effects
+				(font
+					(size 1.27 1.27)
+				)
+			)
+		)
 		(pin "3"
 		)
@@
 		(fields_autoplaced yes)
 		(property "Reference" "C26"
-			(at 113.665 25.4 0)
+			(at 114.3 23.4949 0)
 			(effects
 				(font
@@
 			)
 		)
-		(property "Value" "100nF"
-			(at 113.665 27.94 0)
+		(property "Value" "0.1uF"
+			(at 114.3 26.0349 0)
 			(effects
 				(font
@@
 			)
 		)
+		(property "Mouser Part Number" "MLASH168SB7104KTNA01"
+			(at 114.3 28.5749 0)
+			(effects
+				(font
+					(size 1.27 1.27)
+				)
+				(justify left)
+			)
+		)
 		(pin "1"
 		)
@@
 		(fields_autoplaced yes)
 		(property "Reference" "C25"
-			(at 93.98 24.765 0)
+			(at 93.98 22.8599 0)
 			(effects
 				(font
@@
 			)
 		)
-		(property "Value" "100nF"
-			(at 93.98 27.305 0)
+		(property "Value" "0.1uF"
+			(at 93.98 25.3999 0)
 			(effects
 				(font
@@
 			)
 		)
+		(property "Mouser Part Number" "MLASH168SB7104KTNA01"
+			(at 93.98 27.9399 0)
+			(effects
+				(font
+					(size 1.27 1.27)
+				)
+				(justify left)
+			)
+		)
 		(pin "1"
 		)
@@
 		(fields_autoplaced yes)
 		(property "Reference" "C29"
-			(at 170.815 24.765 0)
+			(at 171.45 22.8599 0)
 			(effects
 				(font
@@
 			)
 		)
-		(property "Value" "100nF"
-			(at 170.815 27.305 0)
+		(property "Value" "0.1uF"
+			(at 171.45 25.3999 0)
 			(effects
 				(font
@@
 			)
 		)
+		(property "Mouser Part Number" "MLASH168SB7104KTNA01"
+			(at 171.45 27.9399 0)
+			(effects
+				(font
+					(size 1.27 1.27)
+				)
+				(justify left)
+			)
+		)
 		(pin "1"
 		)
@@
 			)
 		)
+		(property "Mouser Part Number" "WS2812-2020"
+			(at 63.5 39.37 0)
+			(effects
+				(font
+					(size 1.27 1.27)
+				)
+			)
+		)
 		(pin "3"
 		)
@@
 		(fields_autoplaced yes)
 		(property "Reference" "C27"
-			(at 132.715 24.765 0)
+			(at 133.35 22.8599 0)
 			(effects
 				(font
@@
 			)
 		)
-		(property "Value" "100nF"
-			(at 132.715 27.305 0)
+		(property "Value" "0.1uF"
+			(at 133.35 25.3999 0)
 			(effects
 				(font
@@
 			)
 		)
+		(property "Mouser Part Number" "MLASH168SB7104KTNA01"
+			(at 133.35 27.9399 0)
+			(effects
+				(font
+					(size 1.27 1.27)
+				)
+				(justify left)
+			)
+		)
 		(pin "1"
 		)
@@
 		(fields_autoplaced yes)
 		(property "Reference" "C30"
-			(at 190.5 25.4 0)
+			(at 190.5 23.4949 0)
 			(effects
 				(font
@@
 			)
 		)
-		(property "Value" "100nF"
-			(at 190.5 27.94 0)
+		(property "Value" "0.1uF"
+			(at 190.5 26.0349 0)
 			(effects
 				(font
@@
 			)
 		)
+		(property "Mouser Part Number" "MLASH168SB7104KTNA01"
+			(at 190.5 28.5749 0)
+			(effects
+				(font
+					(size 1.27 1.27)
+				)
+				(justify left)
+			)
+		)
 		(pin "1"
 		)
@@
 		(fields_autoplaced yes)
 		(property "Reference" "C24"
-			(at 74.93 24.765 0)
+			(at 74.93 22.8599 0)
 			(effects
 				(font
@@
 			)
 		)
-		(property "Value" "100nF"
-			(at 74.93 27.305 0)
+		(property "Value" "0.1uF"
+			(at 74.93 25.3999 0)
 			(effects
 				(font
@@
 			)
 		)
+		(property "Mouser Part Number" "MLASH168SB7104KTNA01"
+			(at 74.93 27.9399 0)
+			(effects
+				(font
+					(size 1.27 1.27)
+				)
+				(justify left)
+			)
+		)
 		(pin "1"
 		)
@@
 			)
 		)
+		(property "Mouser Part Number" "WS2812-2020"
+			(at 159.385 39.37 0)
+			(effects
+				(font
+					(size 1.27 1.27)
+				)
+			)
+		)
 		(pin "3"
 		)
@@
 		(fields_autoplaced yes)
 		(property "Reference" "C23"
-			(at 55.88 24.765 0)
+			(at 55.88 22.8599 0)
 			(effects
 				(font
@@
 			)
 		)
-		(property "Value" "100nF"
-			(at 55.88 27.305 0)
+		(property "Value" "0.1uF"
+			(at 55.88 25.3999 0)
 			(effects
 				(font
@@
 			)
 		)
+		(property "Mouser Part Number" "MLASH168SB7104KTNA01"
+			(at 55.88 27.9399 0)
+			(effects
+				(font
+					(size 1.27 1.27)
+				)
+				(justify left)
+			)
+		)
