File: MISC.kicad_sch (KiCad schematic)
At the start: 16 parts

Commit message: updated pins
Parts:
- renumbered C23 to C19, C24 to C20, C25 to C21, C26 to C22, C27 to C23, C28 to C24, C29 to C25, C30 to C26, D8 to D10, D9 to D11, D10 to D12, D11 to D13, D12 to D14, D13 to D15, D14 to D16, D15 to D17
