File: MCU.kicad_sch (KiCad schematic)
At the start: 24 parts, among them SW1 SW_SPDT, U7 STM32G473RETx, U8 74AHC1G32, Y1 8M

Commit message: JLCPCB BOM and gerbers
Parts:
- FB1, FB2: footprint Inductor_SMD:L_0805_2012Metric -> Inductor_SMD:L_0603_1608Metric_Pad1.05x0.95mm_HandSolder
Changed lines of the file:
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@@
 			"AAAAAAAAAAAAAAAAAAAAAAAAAAAAAAAAAAAAAAAAAAAAAAAAAAAAAAAAAAAAAAAAAAAAAAAAAAAA"
 			"AAAAAAAAAAAAAAAAAAAAAAAAAAAAAAAAAAAAAAAAAAAAAAAAAAAAAAAAAAAAAAAAAAAAAAAAAAAA"
+			"AAAAAAAAAAAAAAAAAAAAAAAAAAAAAAAAAAAAAAAAAAAAAAAAAAAAAAAAAAAAAAAAAAAAAAAAAAAA"
+			"AAAAAAAAAAAAAAAAAAAAAAAAAAAAAAAAAAAAAAAAAAAAAAAAAAAAAAAAAAAAAAAAAAAAAAAAAAAA"
+			"AAAAAAAAAAAAAAAAAAAAAAAAAAAAAAAAAAAAAAAAAAAAAAAAAAAAAAAAAAAAAAAAAAAAAAAAAAAA"
+			"AAAAAAAAAAAAAAAAAAAAAAAAAAAAAAAAAAAAAAAAAAAAAAAAAAAAAAAAAAAAAAAAAAAAAAAAAAAA"
+			"AAAAAAAAAAAAAAAAAAAAAAAAAAAAAAAAAAAAAAAAAAAAAAAAAAAAAAAAAAAAAAAAAAAAAAAAAAAA"
+			"AAAAAAAAAAAAAAAAAAAAAAAAAAAAAAAAAAAAAAAAAAAAAAAAAAAAAAAAAAAAAAAAAAAAAAAAAAAA"
+			"AAAAAAAAAAAAAAAAAAAAAAAAAAAAAAAAAAAAAAAAAAAAAAAAAAAAAAAAAAAAAAAAAAAAAAAAAAAA"
+			"AAAAAAAAAAAAAAAAAAAAAAAAAAAAAAAAAAAAAAAAAAAAAAAAAAAAAAAAAAAAAAAAAAAAAAAAAAAA"
+			"AAAAAAAAAAAAAAAAAAAAAAAAAAAAAAAAAAAAAAAAAAAAAAAAAAAAAAAAAAAAAAAAAAAAAAAAAAAA"
+			"AAAAAAAAAAAAAAAAAAAAAAAAAAAAAAAAAAAAAAAAAAAAAAAAAAAAAAAAAAAAAAAAAAAAAAAAAAAA"
+			"AAAAAAAAAAAAAAAAAAAAAAAAAAAAAAAAAAAAAAAAAAAAAAAAAAAAAAAAAAAAAAAAAAAAAAAAAAAA"
+			"AAAAAAAAAAAAAAAAAAAAAAAAAAAAAAAAAAAAAAAAAAAAAAAAAAAAAAAAAAAAAAAAAAAAAAAAAAAA"
+			"AAAAAAAAAAAAAAAAAAAAAAAAAAAAAAAAAAAAAAAAAAAAAAAAAAAAAAAAAAAAAAAAAAAAAAAAAAAA"
+			"AAAAAAAAAAAAAAAAAAAAAAAAAAAAAAAAAAAAAAAAAAAAAAAAAAAAAAAAAAAAAAAAAAAAAAAAAAAA"
+			"AAAAAAAAAAAAAAAAAAAAAAAAAAAAAAAAAAAAAAAAAAAAAAAAAAAAAAAAAAAAAAAAAAAAAAAAAAAA"
+			"AAAAAAAAAAAAAAAAAAAAAAAAAAAAAAAAAAAAAAAAAAAAAAAAAAAAAAAAAAAAAAAAAAAAAAAAAAAA"
+			"AAAAAAAAAAAAAAAAAAAAAAAAAAAAAAAAAAAAAAAAAAAAAAAAAAAAAAAAAAAAAAAAAAAAAAAAAAAA"
+			"AAAAAAAAAAAAAAAAAAAAAAAAAAAAAAAAAAAAAAAAAAAAAAAAAAAAAAAAAAAAAAAAAAAAAAAAAAAA"
 			"AAAAAAAAAAAAAAAAAAAAAAAAAAAAAAAAAAAAAAAAAAAAAAAAAAAAAA=="
 		)
@@
 			"AAAAAAAAAAAAAAAAAAAAAAAAAAAAAAAAAAAAAAAAAAAAAAAAAAAAAAAAAAAAAAAAAAAAAAAAAAAA"
 			"AAAAAAAAAAAAAAAAAAAAAAAAAAAAAAAAAAAAAAAAAAAAAAAAAAAAAAAAAAAAAAAAAAAAAAAAAAAA"
-			"AAAAAAAAAAAAAAAAAAAAAAAAAAAAAAAAAAAAAAAAAAAAAAAAAAAAAAAAAAAAAA=="
+			"AAAAAAAAAAAAAAAAAAAAAAAAAAAAAAAAAAAAAAAAAAAAAAAAAAAAAAAAAAAAAHJJZVBueVlrWkZS"
+			"VUZEQTUvT0ZRbUg5K3ZWcjFhb2xGb3NOS1hqcTFLa3paODRJQklLS0ZTczZPRGdvbGNvN2QrNGtK"
+			"aVpLcFZLMVdpMFNpU3BWcXRTc1dUTUR6NkNIaDRjZk9YSWtMUzFOclZhN3VMaElKQkw2aVV4WldW"
+			"bjBwWFpDb2JCNTgrYmUzdDdZMVFLRHNGMkF4U0dGZ0UySWk0dExUVTJWeVdUSnljbHF0Vm9pa2Nq"
+			"bDhwU1VGSmxNcGxhckNTRVVSZG5iMnh1K0w2T1BNQXVGd3BpWUdQcGp4OVBTMHJLenM1VktKZjF4"
+			"MVh3KzM4SEJ3ZkRoWldabTV1Zm52Mzc5T2o4L1h5UVNTYVhTdExTMGdvSUNRb2hhcmFZb3lzbkpD"
+			"UWVjZ1ZuWUxzRGk4T3hVc0FuMHpZZkp5Y2xTcVZRbWsyVmxaV1ZtWnViazVPVG01aFlVRk9UbDVm"
+			"SDVmQjZQVjY5ZXZhcFZxeHBTOFBuejUvSHg4VmxaV1FVRkJkbloyUmtaR2RuWjJibTV1VEtaakQ1"
+			"V3pPZnpuWjJkVzdkdWJlRHduajE3bHA2ZW5wK2ZMNVZLTXpNek16TXpjM056cFZKcFFVR0JUQ1lU"
+			"Q29VY0RxZEZpeFlHL2hFSllBaHNGMkJ4U0NGZ0UxeGNYRGdjVGtwS1NscGFta3dtS3lnb2tMOG5s"
+			"VW9KSVk2T2puSzV2Rm16Wm5YcjFqV2tvRUFna0VxbHIxKy9sa3FsY3JtOG9LQ0FycG1YbDZkVUtr"
+			"VWlrVUFnRUlsRVBYcjBNSEI0Q29VaU1UR1Ivc3RQTXp6NkNRMWNMdGZaMlRrM043ZHIxNjZlbnA0"
+			"bWZTTUF0R0M3QUl2RGdTenJ4T0JIT2xFVXhkcHFwU3JJNS9NOVBUMGRIUjBMQ3dzVkNvVlNxVlNw"
+			"VkFxRlFxVlN1YnE2dXJpNEVFS1VTcVdCMWJoY3JvT0RnNWVYRjBWUlNxV1NycU5VS3BWS3BVUWlj"
+			"WEp5RW92RlNxVlNyVlliK0RnbWdVQkFmNllHUFNwNmVQUnhiRWRIUjFkWFYvcFBTZXY0V1Zpa0dz"
+			"RjJvWXQxYkJkRi9yMzAyUjhPaDRNUHQyTS9wQkNyUmNsdW0xNkVZeDlnam1wbkx0ODB2Um9oSkto"
+			"ZHkzZFR0N3Q4dExPS2tMZTVoYXA3aFI2WEZkd25XZEszS1FxNVFxbFVDb1ZDQndjSEp5ZW5uSndj"
+			"cFZKSkNDRzMzbGVqS0tJbVJFMFJQb2R3T0VScmg2WW1KRmRKS1Y0cGE1eWpSQStreVFsSitmbjU5"
+			"S01oUlNLUm82T2pTQ1JTcTlYMENleDNCU21LVUlTb0tjTGhFQzRoM0EvMmowcA=="
 		)
 	)
@@
 			)
 		)
-		(property "Footprint" "Inductor_SMD:L_0805_2012Metric"
+		(property "Footprint" "Inductor_SMD:L_0603_1608Metric_Pad1.05x0.95mm_HandSolder"
 			(at 26.035 180.848 90)
 			(effects
@@
 			)
 		)
-		(property "Footprint" "Inductor_SMD:L_0805_2012Metric"
+		(property "Footprint" "Inductor_SMD:L_0603_1608Metric_Pad1.05x0.95mm_HandSolder"
 			(at 20.955 184.912 90)
 			(effects

Commit message: bom
Parts:
- C31, C33: Mouser Part Number (none) -> 0603N270F500CT
- C32: Mouser Part Number 80-C0805C104M5R -> MLASH168SB7104KTNA01
- C34: Mouser Part Number 81-GRM219R6YA475KA3D -> 08055D475KAT4A
- C35, C36, C37, C38, C39, C40: value 100nF -> 0.1uF; Mouser Part Number 80-C0805C104M5R -> MLASH168SB7104KTNA01
- C41: value 0.1u -> 0.1uF; Mouser Part Number (none) -> MLASH168SB7104KTNA01
- D16: Mouser Part Number (none) -> 771-PESD15VL1BA-T/R
- R22, R23: Mouser Part Number (none) -> CRCW060310K0FKEI
- SW1: Mouser Part Number (none) -> CJS-1200TA
- SWD1: Mouser Part Number (none) -> 105309-1104
- U7: Mouser Part Number (none) -> STM32G473RET6
- U8: Mouser Part Number (none) -> SN74AHC1G32TDBVRQ1
- Y1: Mouser Part Number (none) -> ABM3-8.000MHZ-D2Y-T

Commit message: fuckery
Parts:
- added R33: 10k, Resistor_SMD:R_0603_1608Metric_Pad0.98x0.95mm_HandSolder, symbol Device:R_US
- C32: value 100nF -> 0.1uF
Connections:
- net +3V3: now also R33.2
- net NRST: now also R33.1
Changed lines of the file:
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@@
 	(text "Reset Button"
 		(exclude_from_sim no)
-		(at 180.975 107.315 0)
+		(at 185.928 127 0)
 		(effects
 			(font
@@
 	)
 	(junction
+		(at 181.61 109.855)
+		(diameter 0)
+		(color 0 0 0 0)
+	)
+	(junction
 		(at 34.925 179.07)
 		(diameter 0)
@@
 	(wire
 		(pts
+			(xy 181.61 109.855) (xy 181.61 112.395)
+		)
+		(stroke
+			(width 0)
+			(type default)
+		)
+	)
+	(wire
+		(pts
 			(xy 56.515 147.32) (xy 58.42 147.32)
 		)
@@
 	(wire
 		(pts
-			(xy 181.61 109.855) (xy 181.61 112.395)
-		)
-		(stroke
-			(width 0)
-			(type default)
-		)
-	)
-	(wire
-		(pts
 			(xy 167.64 58.42) (xy 199.39 58.42)
 		)
@@
 		)
 	)
+	(wire
+		(pts
+			(xy 181.61 109.22) (xy 181.61 109.855)
+		)
+		(stroke
+			(width 0)
+			(type default)
+		)
+	)
 	(image
 		(at -59.055 80.01)
@@
 	)
 	(symbol
+		(lib_id "Device:R_US")
+		(at 181.61 105.41 180)
+		(unit 1)
+		(exclude_from_sim no)
+		(in_bom yes)
+		(on_board yes)
+		(dnp no)
+		(fields_autoplaced yes)
+		(property "Reference" "R33"
+			(at 183.515 104.1399 0)
+			(effects
+				(font
+					(size 1.27 1.27)
+				)
+				(justify right)
+			)
+		)
+		(property "Value" "10k"
+			(at 183.515 106.6799 0)
+			(effects
+				(font
+					(size 1.27 1.27)
+				)
+				(justify right)
+			)
+		)
+		(property "Footprint" "Resistor_SMD:R_0603_1608Metric_Pad0.98x0.95mm_HandSolder"
+			(at 180.594 105.156 90)
+			(effects
+				(font
+					(size 1.27 1.27)
+				)
+				(hide yes)
+			)
+		)
+		(property "Datasheet" "~"
+			(at 181.61 105.41 0)
+			(effects
+				(font
+					(size 1.27 1.27)
+				)
+				(hide yes)
+			)
+		)
+		(property "Description" "Resistor, US symbol"
+			(at 181.61 105.41 0)
+			(effects
+				(font
+					(size 1.27 1.27)
+				)
+				(hide yes)
+			)
+		)
+		(property "Color" ""
+			(at 181.61 105.41 0)
+			(effects
+				(font
+					(size 1.27 1.27)
+				)
+			)
+		)
+		(property "If" ""
+			(at 181.61 105.41 0)
+			(effects
+				(font
+					(size 1.27 1.27)
+				)
+			)
+		)
+		(property "Mfg" ""
+			(at 181.61 105.41 0)
+			(effects
+				(font
+					(size 1.27 1.27)
+				)
+			)
+		)
+		(property "Vf" ""
+			(at 181.61 105.41 0)
+			(effects
+				(font
+					(size 1.27 1.27)
+				)
+			)
+		)
+		(property "Mouser Part Number" "CRCW060310K0FKEI "
+			(at 181.61 105.41 0)
+			(effects
+				(font
+					(size 1.27 1.27)
+				)
+			)
+		)
+		(pin "1"
+		)
+		(pin "2"
+		)
+		(instances
+			(project "LeaderSOM"
+				(path "/192d0c36-944e-4927-949b-263b8c85a7ca/97cc3b6d-03de-444a-9e7b-201a12c14f47"
+					(reference "R33")
+					(unit 1)
+				)
+			)
+		)
+	)
+	(symbol
 		(lib_id "MCU_ST_STM32G4:STM32G473RETx")
 		(at 73.66 72.39 0)
@@
 		(fields_autoplaced yes)
 		(property "Reference" "C32"
-			(at 33.02 182.245 0)
+			(at 33.02 181.6099 0)
 			(effects
 				(font
@@
 			)
 		)
-		(property "Value" "100nF"
-			(at 33.02 184.785 0)
+		(property "Value" "0.1uF"
+			(at 33.02 184.1499 0)
 			(effects
 				(font
@@
 					(unit 1)
 				)
+			)
+		)
+	)
+	(symbol
+		(lib_id "power:+3.3V")
+		(at 181.61 101.6 0)
+		(unit 1)
+		(exclude_from_sim no)
+		(in_bom yes)
+		(on_board yes)
+		(dnp no)
+		(property "Reference" "#PWR0119"
+			(at 181.61 105.41 0)
+			(effects
+				(font
+					(size 1.27 1.27)
+				)
+				(hide yes)
+			)
+		)
+		(property "Value" "+3V3"
+			(at 181.991 97.2058 0)
+			(effects
+				(font
+					(size 1.27 1.27)
+				)
+			)
+		)
+		(property "Footprint" ""
+			(at 181.61 101.6 0)
+			(effects
+				(font
+					(size 1.27 1.27)
+				)
+				(hide yes)
+			)
+		)
+		(property "Datasheet" ""
+			(at 181.61 101.6 0)
+			(effects
+				(font
+					(size 1.27 1.27)
+				)
+				(hide yes)
+			)
+		)
+		(property "Description" "Power symbol creates a global label with name \"+3.3V\""
+			(at 181.61 101.6 0)
+			(effects
+				(font
+					(size 1.27 1.27)
+				)
+				(hide yes)
+			)
+		)
+		(pin "1"
+		)
+		(instances
+			(project "LeaderSOM"
+				(path "/192d0c36-944e-4927-949b-263b8c85a7ca/97cc3b6d-03de-444a-9e7b-201a12c14f47"
+					(reference "#PWR0119")
+					(unit 1)
+				)

Commit message: revB for assembly stuff
Parts:
- added D21: 3V3, LED_SMD:LED_0603_1608Metric_Pad1.05x0.95mm_HandSolder, symbol Device:LED
- added R35: 120, Resistor_SMD:R_0603_1608Metric_Pad0.98x0.95mm_HandSolder, symbol Device:R
- Reset1: Mouser Part Number 653-B3SL-1002P -> 612-TL3365AF180QG; P/N B3SL-1002P -> TL3365AF180QG
Connections:
- net GND: now also D21.1 (K)
- net IMON renamed Onboard_LED
- net Onboard_LED: now also R35.1
- new net: D21.2 (A), R35.2

Commit message: the emptiness machine - linkin park
Connections:
- net UART4_RX/TIM8_CH2N renamed USART3_RX/TIM8_CH2N
- net UART4_TX/TIM8_CH1N renamed USART3_TX/TIM8_CH1N
- net USART3_RX/ADC1_IN14/TIM2_CH4 renamed LPUART1_TX/ADC1_IN14/TIM2_CH4
- net USART3_TX/OPAMP3_VINM/TIM2_CH3 renamed LPUART1_RX/TIM2_CH3/OPAMP3_VINM

Commit message: revc start
Connections:
- net UART5_RX is gone; now on net AddressableLED: U7.55 (PD2)
- net AddressableLED: no longer U7.59 (PB6)
- net SPI3_MISO/TIM3_CH1/USART2_RX: no longer U7.57 (PB4)
- net SPI3_MOSI/TIM3_CH2/TIM17_CH1: no longer U7.58 (PB5)
- net SPI3_SCK/TIM2_CH2/USART2_TX: no longer U7.56 (PB3)
- net USART1_RX renamed USART1_RX/ADC2_IN11
- net USART1_TX renamed USART1_TX/ADC2_IN5
- new net FDCAN2_RX: U7.58 (PB5)
- new net FDCAN2_TX: U7.59 (PB6)
Other:
- moved on the sheet: C32, C33, C40, C41, D16, D21, FB1, FB2, R22, R23, R35, Reset1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

Commit message: updated pins
Parts:
- renumbered C31 to C27, C32 to C28, C33 to C29, C34 to C30, C35 to C31, C36 to C32, C37 to C33, C38 to C34, C39 to C35, C40 to C36, C41 to C37, CR3 to CR2, CR2 to CR3, D16 to D18, D21 to D19, R33 to R21, R35 to R24, U7 to U6, U8 to U7
Connections:
- net FDCAN1_RX is gone; now on net USB_D-: U6.45 (PA11)
- net FDCAN1_TX is gone; now on net USB_D+: U6.46 (PA12)
- net OPAMP5_VINM/ADC1_IN4/TIM2_CH4 is gone; now on net ADC1_IN4/TIM2_CH4/OPAMP5_VINM: U6.17 (PA3)
- net SPI2_SCK/OPAMP3_VINP/FDCAN2_TX is gone; now on net SPI2_SCK/OPAMP3_VINP/ADC3_IN5: CR3.4, U6.35 (PB13)
- net SPI3_MISO/TIM3_CH1/USART2_RX is gone; now on net SPI3_MISO/TIM8_CH2N/UART4_RX: CR2.3
- net SPI3_MOSI/TIM3_CH2/TIM17_CH1 is gone; now on net SPI3_MOSI/TIM5_CH2: CR2.6
- net SPI3_SCK/TIM2_CH2/USART2_TX is gone; now on net SPI3_SCK/TIM8_CH1N/UART4_TX: CR2.4
- net UART5_TX/TIM5_CH2 is gone; now on net SPI3_MOSI/TIM5_CH2: U6.54 (PC12)
- net USART3_RX/TIM8_CH2N is gone; now on net SPI3_MISO/TIM8_CH2N/UART4_RX: U6.53 (PC11)
- net USART3_TX/TIM8_CH1N is gone; now on net SPI3_SCK/TIM8_CH1N/UART4_TX: U6.52 (PC10)
- net ADC1_IN9/OPAMP5_VINP/TIM1_CH4: now also U6.11 (PC3)
- net ADC5_IN2/TIM1_CH2/COMP5_OUT: now also U6.43 (PA9)
- net FDCAN3_RX: now also U6.56 (PB3); no longer U6.42 (PA8)
- net FDCAN3_TX: now also U6.57 (PB4); no longer U6.51 (PA15)
- net Onboard_LED: now also U6.42 (PA8); no longer U6.11 (PC3)
- net SDC_DET: now also U6.44 (PA10); no longer U6.43 (PA9)
- net SPI3_NSS: now also CR2.1, U6.51 (PA15)
- removed net SPI3_NSS/TIM1_CH3/COMP6_OUT: CR2.1, U6.44 (PA10)
