File: PowerMUX/PowerMUX.kicad_sch (KiCad schematic)
At the start: 26 parts, among them J1 Conn_01x02_Pin, J2 UJ31-CH-G2-SMT-TR, U1 FT230XS-R, U2 LM2596S-5, U3 TPS2115APW, U4 LM3940IMP-3.3

Commit message: power negotiation fix
Parts:
- added R6, R7: 5.1k, symbol Device:R
Connections:
- net GND: now also R6.2, R7.2
- net at J2.A5 (CC1): now also R6.1
- net at J2.B5 (CC2): now also R7.1
- no-connect marks 24 -> 22

Commit message: changed old THT buck converter to SMD buck converter from LSOM
Parts:
- added C11: 10uF, Capacitor_SMD:C_0805_2012Metric, symbol Device:C
- added C12: 0.1uF, Capacitor_SMD:C_0805_2012Metric, symbol Device:C
- added C13: 47uF, Capacitor_SMD:C_0805_2012Metric, symbol Device:C
- added L2: 3.3uH, Inductor_SMD:L_0805_2012Metric_Pad1.15x1.40mm_HandSolder, symbol Device:L
- added R8: 56k, Resistor_SMD:R_0805_2012Metric, symbol Device:R
- added R9: 10k, Resistor_SMD:R_0805_2012Metric, symbol Device:R
- added U5: TPS562231DRLR, Package_TO_SOT_SMD:SOT-563, symbol utsvt-power-regulators:TPS562231DRLR
Connections:
- net 5v: now also C13.1, L2.2, R8.1; no longer C8.1, L1.1, U2.4 (FB)
- net GND: now also C11.2, C13.2, R9.2, U5.3 (GND)
- net at C7.1, U2.1 (VIN): no longer TP2.1
- new net: R8.2, R9.1, U5.6 (FB)
- new net: C11.1, TP2.1, U5.1 (VIN), U5.5 (EN)
- new net: C8.1, L1.1, U2.4 (FB)
- new net BST: C12.1, U5.4 (BST)
- new net SW: C12.2, L2.1, U5.2 (SW)
Other:
- note added: "+12v -> +5v"
- moved on the sheet: C7, C8, D2, L1, TP1, TP2, U2

Commit message: added testpoints
Parts:
- removed D2: D_Schottky, symbol Device:D_Schottky
- removed L1: 33uH, symbol Device:L
- removed U2: LM2596S-5, Package_TO_SOT_SMD:TO-263-5_TabPin3, symbol Regulator_Switching:LM2596S-5
- removed U4: LM3940IMP-3.3, MP04A, symbol LM3940:LM3940IMP-3.3
- added J3: Conn_01x04_Pin, symbol Connector:Conn_01x04_Pin
- added J4: Conn_01x02_Pin, symbol Connector:Conn_01x02_Pin
- added J5: Conn_01x01_Pin, symbol Connector:Conn_01x01_Pin
- added TP3: TestPoint, symbol Connector:TestPoint
- added U2: TLV70130DBVR, DBV5, symbol 2025-01-18_20-51-31:TLV70130DBVR
- C7: value 680uF -> 0.1uf
- C8: value 220uF -> 1uf
Connections:
- net +3.3V: now also C8.1, U2.1 (OUT)
- net 5Vmux: now also C7.1, J5.1 (Pin_1), U2.3 (IN)
- net 5v: now also J4.2 (Pin_2)
- net D+: now also J3.3 (Pin_3)
- net D-: now also J3.2 (Pin_2)
- net GND: now also J3.1 (Pin_1), TP3.1, U2.2 (GND)
- net vbus: now also J3.4 (Pin_4), J4.1 (Pin_1)
- no-connect marks 22 -> 24
Other:
- note added: "+5v -> 3.3v LDO"
- note added: "Ground"
- note added: "MUX out"
- note added: "Testpoints"
- note added: "USB input"
- note added: "power MUX input"
- moved on the sheet: C1, C10, C2, C3, C5, C9, R5, U3

Commit message: finished PCB layout
Parts:
- added C14: 0.1uF, Capacitor_SMD:C_0805_2012Metric, symbol Device:C
- C10, C7, C8, C9: footprint (none) -> Capacitor_SMD:C_0805_2012Metric
- J1, J4: footprint (none) -> Connector_PinHeader_1.00mm:PinHeader_1x02_P1.00mm_Vertical
- J2: footprint UJ31-CH-G2-SMT-TR:CUI_UJ31-CH-G2-SMT-TR -> UTSVT_Connectors:CUI_UJ31-CH-G2-SMT-TR
- J3: footprint (none) -> Connector_PinHeader_1.00mm:PinHeader_1x04_P1.00mm_Vertical
- J5: footprint (none) -> Connector_PinHeader_1.00mm:PinHeader_1x01_P1.00mm_Vertical
- R5, R6, R7: footprint (none) -> Resistor_SMD:R_0805_2012Metric
- R8: value 56k -> 73k
- TP1, TP2: footprint (none) -> TestPoint:TestPoint_Plated_Hole_D2.0mm
- TP3: value TestPoint -> TestpointGND; footprint (none) -> TestPoint:TestPoint_Plated_Hole_D2.0mm
- U2: footprint DBV5 -> TLV70130DBVR:DBV5-L
- U3: footprint PW8 -> TPS2115APW:PW8
Connections:
- net 5Vmux: now also C14.1
- net GND: now also C14.2
Other:
- moved on the sheet: TP3

Commit message: commit messages are so boring
Parts:
- added J6, J7: Conn_01x01_Pin, Connector_PinHeader_2.54mm:PinHeader_1x01_P2.54mm_Vertical, symbol Connector:Conn_01x01_Pin
- J1: footprint Connector_PinHeader_1.00mm:PinHeader_1x02_P1.00mm_Vertical -> Connector_PinSocket_2.54mm:PinSocket_1x02_P2.54mm_Vertical
- J3: footprint Connector_PinHeader_1.00mm:PinHeader_1x04_P1.00mm_Vertical -> Connector_PinHeader_2.54mm:PinHeader_1x04_P2.54mm_Vertical
- J4: footprint Connector_PinHeader_1.00mm:PinHeader_1x02_P1.00mm_Vertical -> Connector_PinHeader_2.54mm:PinHeader_1x02_P2.54mm_Vertical
- J5: footprint Connector_PinHeader_1.00mm:PinHeader_1x01_P1.00mm_Vertical -> Connector_PinHeader_2.54mm:PinHeader_1x01_P2.54mm_Vertical
Connections:
- net CC1: now reaches J2.A5 (CC1), R6.1
- net CC1: now also J6.1 (Pin_1)
- net CC2: now reaches J2.B5 (CC2), R7.1
- net CC2: now also J7.1 (Pin_1)
