File: PowerMUX/PowerMUX.kicad_pcb (KiCad board)
At the start: 2 copper layers, 63.6 x 24.1 mm, 37 parts, among them J1 Conn_01x02_Pin, J2 UJ31-CH-G2-SMT-TR, J3 Conn_01x04_Pin, J4 Conn_01x02_Pin, J5 Conn_01x01_Pin, U1 FT230XS-R, U2 TLV70130DBVR, U3 TPS2115APW, U5 TPS562231DRLR

Commit message: fix trace width ts ong
Parts:
- moved C5 2.67 mm to (156.2, 107.5)
- moved C3 1.40 mm to (158.2, 107.5)
- moved C1 1.14 mm to (162.3, 107.5)
- moved C14 0.13 mm to (182.8, 97.4)
- moved C2 0.13 mm to (160.3, 107.5)
- moved R2 0.13 mm to (153.9, 101.2)
- moved R4 0.10 mm to (153.9, 97.8)
Routing:
- net vbus: track 128.9 -> 95.5 mm
- net GND: track 147.3 -> 128.7 mm, vias 12 -> 15
- net +3.3V: track 58.0 -> 51.5 mm
- net Net-(U1-CBUS3): track 10.2 -> 10.9 mm
- net 5Vmux: track 49.2 -> 48.5 mm
- net Net-(J2-CC1): track 4.79 -> 4.14 mm
- net 5v: track 61.4 -> 62.0 mm

Commit message: fix traces fr on god
Parts:
- moved R5 4.18 mm to (171.2, 97.0), turned to 90 degrees
Routing:
- net GND: track 128.7 -> 38.6 mm, vias 15 -> 17
- net D+: track 48.5 -> 45.1 mm, vias 2 -> 3
- net +3.3V: track 51.5 -> 49.5 mm
- net D-: track 30.8 -> 29.2 mm
- net Net-(U3-ILIM): track 2.84 -> 2.16 mm

Commit message: commit messages are so boring
Parts:
- added CC1: Conn_01x01_Pin, Connector_PinHeader_2.54mm:PinHeader_1x01_P2.54mm_Vertical, F.Cu at (135.8, 114.2)
- added CC2: Conn_01x01_Pin, Connector_PinHeader_2.54mm:PinHeader_1x01_P2.54mm_Vertical, F.Cu at (139.7, 114.2)
- USB out: renamed from J3; footprint Connector_PinHeader_1.00mm:PinHeader_1x04_P1.00mm_Vertical -> Connector_PinHeader_2.54mm:PinHeader_1x04_P2.54mm_Vertical
- [Tx, Rx]: renamed from J1; footprint Connector_PinHeader_1.00mm:PinHeader_1x02_P1.00mm_Vertical -> Connector_PinSocket_2.54mm:PinSocket_1x02_P2.54mm_Vertical
- [Vbus, 5V]: renamed from J4; footprint Connector_PinHeader_1.00mm:PinHeader_1x02_P1.00mm_Vertical -> Connector_PinHeader_2.54mm:PinHeader_1x02_P2.54mm_Vertical
- mux: renamed from J5; footprint Connector_PinHeader_1.00mm:PinHeader_1x01_P1.00mm_Vertical -> Connector_PinHeader_2.54mm:PinHeader_1x01_P2.54mm_Vertical
- moved mux 17.5 mm to (185.3, 103.6), turned to -90 degrees
- moved GND 9.68 mm to (143.9, 114.2)
- moved USB out 9.19 mm to (155.8, 114.2)
- moved C12 8.73 mm to (172.5, 104.4), turned to 0 degrees
- moved C13 7.43 mm to (177.3, 109.4)
- moved L2 7.42 mm to (174.8, 109.6)
- moved U5 7.38 mm to (172.7, 106.5)
- moved U2 7.38 mm to (182.9, 94.8)
- moved C10 7.38 mm to (175.4, 99.7)
- moved C11 7.38 mm to (175.9, 106.5)
- moved C14 7.38 mm to (175.4, 97.0)
- moved C7 7.38 mm to (184.5, 99.0)
- moved C8 7.38 mm to (181.2, 99.0)
- moved C9 7.38 mm to (175.4, 94.6)
- moved R5 7.38 mm to (163.8, 96.6)
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- renumbered TP2 to 12V+, TP1 to 12V-, TP3 to GND
Connections:
- net Net-(J2-CC1) renamed CC1
- net Net-(J2-CC2) renamed CC2
Routing:
- net 5Vmux: track 48.5 -> 24.2 mm, vias 1 -> 0
- net CC1: track 3.98 -> 22.0 mm, vias 2 -> 3
- net /BST: track 18.0 -> 1.84 mm
- net CC2: track 10.7 -> 25.2 mm
- net vbus: track 95.3 -> 83.5 mm, vias 2 -> 4
- net GND: track 38.6 -> 29.1 mm
- net +3.3V: track 49.5 -> 42.3 mm
- net 5v: track 62.3 -> 56.5 mm
- net Net-(J1-Pin_1): track 15.7 -> 12.3 mm
- net /SW: track 11.1 -> 8.41 mm
- net Net-(J1-Pin_2): track 14.7 -> 12.1 mm
- net D+: track 45.1 -> 43.1 mm
- net Net-(U5-FB): track 7.40 -> 6.11 mm
- net D-: track 29.2 -> 28.0 mm, vias 1 -> 0
- net Net-(U5-EN): track 18.4 -> 17.5 mm
Other:
- board size 63.6 x 24.1 mm -> 56.3 x 24.1 mm

Commit message: buck SW inductor closer to pad, USBc clearance
Parts:
- [Vbus, D+, D-, GND]: renamed from USB out
- moved GND 23.7 mm to (167.6, 114.3)
- moved [Vbus, 5V] 21.7 mm to (158.2, 95.1)
- moved C13 7.19 mm to (176.0, 102.4), turned to 0 degrees
- moved L2 5.38 mm to (176.1, 104.4), turned to 0 degrees
- moved CC1 4.19 mm to (140.0, 114.2)
- moved CC2 4.19 mm to (143.9, 114.2)
- moved R3 1.91 mm to (155.1, 97.7)
- moved R8 1.42 mm to (169.5, 108.0)
- moved R9 1.27 mm to (169.5, 105.2)
- moved R4 0.90 mm to (153.0, 97.7)
Routing:
- net 5v: track 56.5 -> 39.0 mm, vias 3 -> 0
- net vbus: track 83.5 -> 66.4 mm
- net /SW: track 8.41 -> 4.61 mm
- net CC2: track 25.2 -> 22.8 mm
- net Net-(U5-FB): track 6.11 -> 4.14 mm
- net CC1: track 22.0 -> 20.3 mm
- net Net-(U5-EN): track 17.5 -> 16.8 mm
- net 5Vmux: track 24.2 -> 23.7 mm
Other:
- board size 56.3 x 24.1 mm -> 54.2 x 24.1 mm
